File: 2016/PT_2016_PB_MAIN_Rev1.sch (EAGLE design)
At the start: 136 parts, among them M1+ ANDERSON_POWERPOLEPP45_PCB_HO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, M1- ANDERSON_POWERPOLEPP45_PCB_HO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, M2+ ANDERSON_POWERPOLEPP45_PCB_HO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, M2- ANDERSON_POWERPOLEPP45_PCB_HO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, M3+ ANDERSON_POWERPOLEPP45_PCB_HO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, M3- ANDERSON_POWERPOLEPP45_PCB_HO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, M4+ ANDERSON_POWERPOLEPP45_PCB_HO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, M4- ANDERSON_POWERPOLEPP45_PCB_HO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, M5+ ANDERSON_POWERPOLEPP45_PCB_HO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, M5- ANDERSON_POWERPOLEPP45_PCB_HO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

Commit message: New Layout Idea
Parts:
- removed U$45: APP_2POS_CONFIG5V_VERT, MRDT-Connectors:APP_2POS_CONFIG5V_VERT
- removed U$46: APP_2POS_CONFIG12V_VERT, MRDT-Connectors:APP_2POS_CONFIG12V_VERT
- added M2-1, M2-2, M2-3, M2-4: ANDERSON_POWERPOLEPP45_PCB_HORIZ_RIGHT, MRDT-Connectors:ANDERSON_POWERPOLEPP45_PCB_HORIZ_RIGHT
- added U$25: APP_MOUTING_WINGHORIZ, MRDT-Connectors:APP_MOUTING_WINGHORIZ
Connections:
- net 12V-AUX: now also M2-2.P$1; no longer U$46VCC.P$1
- net 12V-SIG: now also U$4.PN3; no longer U$4.PP2
- net 5V-AUX: now also M2-4.P$1; no longer U$45VCC.P$1
- net 5V-SIG: now also U$4.PP2; no longer U$4.PN3
- net GND: now also M2-1.P$1, M2-3.P$1; no longer U$45GND.P$1, U$46GND.P$1
- net RX1: now also U$24.R0; no longer U$12.R0
- net RX2: now also U$12.R0; no longer U$24.R0
- net TX1: now also U$24.DI; no longer U$12.DI
- net TX2: now also U$12.DI; no longer U$24.DI
Changed lines of the file:
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@@
 <?xml version="1.0" encoding="utf-8"?>
 <!DOCTYPE eagle SYSTEM "eagle.dtd">
-<eagle version="6.5.0">
+<eagle version="7.3.0">
 <drawing>
 <settings>
@@
 <part name="M2-" library="MRDT-Connectors" deviceset="ANDERSON_POWERPOLE" device="PP45_PCB_HORIZ_RIGHT"/>
 <part name="M1+" library="MRDT-Connectors" deviceset="ANDERSON_POWERPOLE" device="PP45_PCB_HORIZ_RIGHT"/>
-<part name="U$45" library="MRDT-Connectors" deviceset="APP_2POS_CONFIG" device="5V_VERT"/>
-<part name="U$46" library="MRDT-Connectors" deviceset="APP_2POS_CONFIG" device="12V_VERT"/>
 <part name="U$41" library="MRDT-Connectors" deviceset="APP_MOUTING_WING" device="HORIZ"/>
 <part name="U$42" library="MRDT-Connectors" deviceset="APP_MOUTING_WING" device="HORIZ"/>
+<part name="M2-1" library="MRDT-Connectors" deviceset="ANDERSON_POWERPOLE" device="PP45_PCB_HORIZ_RIGHT"/>
+<part name="M2-2" library="MRDT-Connectors" deviceset="ANDERSON_POWERPOLE" device="PP45_PCB_HORIZ_RIGHT"/>
+<part name="M2-3" library="MRDT-Connectors" deviceset="ANDERSON_POWERPOLE" device="PP45_PCB_HORIZ_RIGHT"/>
+<part name="M2-4" library="MRDT-Connectors" deviceset="ANDERSON_POWERPOLE" device="PP45_PCB_HORIZ_RIGHT"/>
+<part name="U$25" library="MRDT-Connectors" deviceset="APP_MOUTING_WING" device="HORIZ"/>
 </parts>
 <sheets>
@@
 <instance part="M2-" gate="G$1" x="-205.74" y="15.24" rot="R270"/>
 <instance part="M1+" gate="G$1" x="-198.12" y="15.24" rot="R270"/>
-<instance part="U$45" gate="GND" x="116.84" y="-96.52" rot="R270"/>
-<instance part="U$45" gate="VCC" x="127" y="-96.52" rot="R270"/>
-<instance part="U$46" gate="GND" x="53.34" y="-96.52" rot="R270"/>
-<instance part="U$46" gate="VCC" x="63.5" y="-96.52" rot="R270"/>
 <instance part="U$41" gate="G$1" x="-607.06" y="160.02"/>
 <instance part="U$42" gate="G$1" x="-607.06" y="152.4"/>
+<instance part="M2-1" gate="G$1" x="53.34" y="-96.52" rot="R270"/>
+<instance part="M2-2" gate="G$1" x="63.5" y="-96.52" rot="R270"/>
+<instance part="M2-3" gate="G$1" x="116.84" y="-96.52" rot="R270"/>
+<instance part="M2-4" gate="G$1" x="127" y="-96.52" rot="R270"/>
+<instance part="U$25" gate="G$1" x="-607.06" y="142.24"/>
 </instances>
 <busses>
@@
 <wire x1="45.72" y1="-88.9" x2="45.72" y2="-93.98" width="0.1524" layer="91"/>
 <wire x1="45.72" y1="-88.9" x2="53.34" y2="-88.9" width="0.1524" layer="91"/>
-<pinref part="U$46" gate="GND" pin="P$1"/>
+<pinref part="M2-1" gate="G$1" pin="P$1"/>
 </segment>
 <segment>
@@
 <wire x1="109.22" y1="-88.9" x2="109.22" y2="-93.98" width="0.1524" layer="91"/>
 <wire x1="109.22" y1="-88.9" x2="116.84" y2="-88.9" width="0.1524" layer="91"/>
-<pinref part="U$45" gate="GND" pin="P$1"/>
+<pinref part="M2-3" gate="G$1" pin="P$1"/>
 </segment>
 <segment>
@@
 <junction x="73.66" y="-86.36"/>
 <wire x1="63.5" y1="-88.9" x2="73.66" y2="-88.9" width="0.1524" layer="91"/>
-<pinref part="U$46" gate="VCC" pin="P$1"/>
+<pinref part="M2-2" gate="G$1" pin="P$1"/>
 </segment>
 </net>
@@
 </segment>
 <segment>
-<pinref part="U$4" gate="G$1" pin="PP2"/>
-<wire x1="-167.64" y1="-137.16" x2="-172.72" y2="-137.16" width="0.1524" layer="91"/>
-<label x="-180.34" y="-137.16" size="1.778" layer="95"/>
+<pinref part="U$4" gate="G$1" pin="PN3"/>
+<wire x1="-132.08" y1="-127" x2="-127" y2="-127" width="0.1524" layer="91"/>
+<label x="-127" y="-127" size="1.778" layer="95"/>
 </segment>
 </net>
@@
 <net name="RX1" class="0">
 <segment>
-<wire x1="-373.38" y1="-55.88" x2="-393.7" y2="-55.88" width="0.1524" layer="91"/>
-<pinref part="U$12" gate="G$1" pin="R0"/>
-<label x="-373.38" y="-55.88" size="1.778" layer="95"/>
-</segment>
-<segment>
 <pinref part="U$4" gate="G$1" pin="PC4"/>
 <wire x1="-167.64" y1="-50.8" x2="-172.72" y2="-50.8" width="0.1524" layer="91"/>
 <label x="-177.8" y="-50.8" size="1.778" layer="95"/>
+</segment>
+<segment>
+<wire x1="-373.38" y1="-91.44" x2="-393.7" y2="-91.44" width="0.1524" layer="91"/>
+<pinref part="U$24" gate="G$1" pin="R0"/>
+<label x="-373.38" y="-91.44" size="1.778" layer="95"/>
 </segment>
 </net>
@@
 <net name="TX1" class="0">
 <segment>
+<pinref part="U$4" gate="G$1" pin="PC5"/>
+<wire x1="-167.64" y1="-53.34" x2="-172.72" y2="-53.34" width="0.1524" layer="91"/>
+<label x="-177.8" y="-53.34" size="1.778" layer="95"/>
+</segment>
+<segment>
+<wire x1="-393.7" y1="-86.36" x2="-373.38" y2="-86.36" width="0.1524" layer="91"/>
+<pinref part="U$24" gate="G$1" pin="DI"/>
+<label x="-373.38" y="-86.36" size="1.778" layer="95"/>
+</segment>
+</net>
+<net name="RX2" class="0">
+<segment>
+<pinref part="U$4" gate="G$1" pin="PP0"/>
+<wire x1="-167.64" y1="-132.08" x2="-172.72" y2="-132.08" width="0.1524" layer="91"/>
+<label x="-177.8" y="-132.08" size="1.778" layer="95"/>
+</segment>
+<segment>
+<wire x1="-373.38" y1="-55.88" x2="-393.7" y2="-55.88" width="0.1524" layer="91"/>
+<pinref part="U$12" gate="G$1" pin="R0"/>
+<label x="-373.38" y="-55.88" size="1.778" layer="95"/>
+</segment>
+</net>
+<net name="TX2" class="0">
+<segment>
+<pinref part="U$4" gate="G$1" pin="PP1"/>
+<wire x1="-167.64" y1="-134.62" x2="-172.72" y2="-134.62" width="0.1524" layer="91"/>
+<label x="-177.8" y="-134.62" size="1.778" layer="95"/>
+</segment>
+<segment>
 <wire x1="-393.7" y1="-50.8" x2="-373.38" y2="-50.8" width="0.1524" layer="91"/>
 <pinref part="U$12" gate="G$1" pin="DI"/>
 <label x="-373.38" y="-50.8" size="1.778" layer="95"/>
-</segment>
-<segment>
-<pinref part="U$4" gate="G$1" pin="PC5"/>
-<wire x1="-167.64" y1="-53.34" x2="-172.72" y2="-53.34" width="0.1524" layer="91"/>
-<label x="-177.8" y="-53.34" size="1.778" layer="95"/>
-</segment>
-</net>
-<net name="RX2" class="0">
-<segment>
-<wire x1="-373.38" y1="-91.44" x2="-393.7" y2="-91.44" width="0.1524" layer="91"/>
-<pinref part="U$24" gate="G$1" pin="R0"/>
-<label x="-373.38" y="-91.44" size="1.778" layer="95"/>
-</segment>
-<segment>
-<pinref part="U$4" gate="G$1" pin="PP0"/>
-<wire x1="-167.64" y1="-132.08" x2="-172.72" y2="-132.08" width="0.1524" layer="91"/>
-<label x="-177.8" y="-132.08" size="1.778" layer="95"/>
-</segment>
-</net>
-<net name="TX2" class="0">
-<segment>
-<wire x1="-393.7" y1="-86.36" x2="-373.38" y2="-86.36" width="0.1524" layer="91"/>
-<pinref part="U$24" gate="G$1" pin="DI"/>
-<label x="-373.38" y="-86.36" size="1.778" layer="95"/>
-</segment>
-<segment>
-<pinref part="U$4" gate="G$1" pin="PP1"/>
-<wire x1="-167.64" y1="-134.62" x2="-172.72" y2="-134.62" width="0.1524" layer="91"/>
-<label x="-177.8" y="-134.62" size="1.778" layer="95"/>
 </segment>
 </net>
@@
 <junction x="137.16" y="-86.36"/>
 <wire x1="127" y1="-88.9" x2="137.16" y2="-88.9" width="0.1524" layer="91"/>
-<pinref part="U$45" gate="VCC" pin="P$1"/>
+<pinref part="M2-4" gate="G$1" pin="P$1"/>
 </segment>
 <segment>
@@
 </segment>
 <segment>
-<pinref part="U$4" gate="G$1" pin="PN3"/>
-<wire x1="-132.08" y1="-127" x2="-127" y2="-127" width="0.1524" layer="91"/>
-<label x="-127" y="-127" size="1.778" layer="95"/>
-</segment>
-</net>
+<pinref part="U$4" gate="G$1" pin="PP2"/>
+<wire x1="-167.64" y1="-137.16" x2="-172.72" y2="-137.16" width="0.1524" layer="91"/>
+<label x="-180.34" y="-137.16" size="1.778" layer="95"/>
+</segment>
+</net>

Commit message: Routed new layout
Parts:
- added U$26, U$27, U$28, U$29: ANDERSON_POWERPOLEPP45_PCB_HORIZ_RIGHT_2HIGH, MRDT-Connectors:ANDERSON_POWERPOLEPP45_PCB_HORIZ_RIGHT_2HIGH
- added X1: 22-23-2041, con-molex:22-23-2041
Connections:
- new net N$11: M2-2.P$1, X1-1.S
- new net N$3: M2-3.P$1, X1-4.S
- new net N$5: M2-1.P$1, X1-3.S
- new net N$8: M2-4.P$1, X1-2.S
- net 12V-AUX: now also U$26.P$1; no longer M2-2.P$1
- net 5V-AUX: now also U$27.P$1; no longer M2-4.P$1
- net GND: now also U$28.P$1, U$29.P$1; no longer M2-1.P$1, M2-3.P$1
Other:
- moved on the sheet: M2-1, M2-2, M2-3, M2-4
Changed lines of the file:
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@@
 <part name="M2-4" library="MRDT-Connectors" deviceset="ANDERSON_POWERPOLE" device="PP45_PCB_HORIZ_RIGHT"/>
 <part name="U$25" library="MRDT-Connectors" deviceset="APP_MOUTING_WING" device="HORIZ"/>
+<part name="U$26" library="MRDT-Connectors" deviceset="ANDERSON_POWERPOLE" device="PP45_PCB_HORIZ_RIGHT_2HIGH"/>
+<part name="U$27" library="MRDT-Connectors" deviceset="ANDERSON_POWERPOLE" device="PP45_PCB_HORIZ_RIGHT_2HIGH"/>
+<part name="U$28" library="MRDT-Connectors" deviceset="ANDERSON_POWERPOLE" device="PP45_PCB_HORIZ_RIGHT_2HIGH"/>
+<part name="U$29" library="MRDT-Connectors" deviceset="ANDERSON_POWERPOLE" device="PP45_PCB_HORIZ_RIGHT_2HIGH"/>
+<part name="X1" library="con-molex" deviceset="22-23-2041" device=""/>
 </parts>
 <sheets>
@@
 <instance part="U$41" gate="G$1" x="-607.06" y="160.02"/>
 <instance part="U$42" gate="G$1" x="-607.06" y="152.4"/>
-<instance part="M2-1" gate="G$1" x="53.34" y="-96.52" rot="R270"/>
-<instance part="M2-2" gate="G$1" x="63.5" y="-96.52" rot="R270"/>
-<instance part="M2-3" gate="G$1" x="116.84" y="-96.52" rot="R270"/>
-<instance part="M2-4" gate="G$1" x="127" y="-96.52" rot="R270"/>
+<instance part="M2-1" gate="G$1" x="68.58" y="-172.72"/>
+<instance part="M2-2" gate="G$1" x="68.58" y="-198.12"/>
+<instance part="M2-3" gate="G$1" x="68.58" y="-162.56"/>
+<instance part="M2-4" gate="G$1" x="68.58" y="-185.42"/>
 <instance part="U$25" gate="G$1" x="-607.06" y="142.24"/>
+<instance part="U$26" gate="G$1" x="63.5" y="-96.52" rot="R270"/>
+<instance part="U$27" gate="G$1" x="129.54" y="-96.52" rot="R270"/>
+<instance part="U$28" gate="G$1" x="119.38" y="-96.52" rot="R270"/>
+<instance part="U$29" gate="G$1" x="55.88" y="-96.52" rot="R270"/>
+<instance part="X1" gate="-1" x="25.4" y="-182.88" rot="R180"/>
+<instance part="X1" gate="-2" x="25.4" y="-180.34" rot="R180"/>
+<instance part="X1" gate="-3" x="25.4" y="-177.8" rot="R180"/>
+<instance part="X1" gate="-4" x="25.4" y="-175.26" rot="R180"/>
 </instances>
 <busses>
@@
 <pinref part="GND32" gate="1" pin="GND"/>
 <wire x1="45.72" y1="-88.9" x2="45.72" y2="-93.98" width="0.1524" layer="91"/>
-<wire x1="45.72" y1="-88.9" x2="53.34" y2="-88.9" width="0.1524" layer="91"/>
-<pinref part="M2-1" gate="G$1" pin="P$1"/>
+<pinref part="U$29" gate="G$1" pin="P$1"/>
+<wire x1="45.72" y1="-88.9" x2="55.88" y2="-88.9" width="0.1524" layer="91"/>
 </segment>
 <segment>
@@
 <pinref part="GND20" gate="1" pin="GND"/>
 <wire x1="109.22" y1="-88.9" x2="109.22" y2="-93.98" width="0.1524" layer="91"/>
-<wire x1="109.22" y1="-88.9" x2="116.84" y2="-88.9" width="0.1524" layer="91"/>
-<pinref part="M2-3" gate="G$1" pin="P$1"/>
+<pinref part="U$28" gate="G$1" pin="P$1"/>
+<wire x1="109.22" y1="-88.9" x2="119.38" y2="-88.9" width="0.1524" layer="91"/>
 </segment>
 <segment>
@@
 <wire x1="78.74" y1="-86.36" x2="73.66" y2="-86.36" width="0.1524" layer="91"/>
 <junction x="73.66" y="-86.36"/>
+<pinref part="U$26" gate="G$1" pin="P$1"/>
 <wire x1="63.5" y1="-88.9" x2="73.66" y2="-88.9" width="0.1524" layer="91"/>
-<pinref part="M2-2" gate="G$1" pin="P$1"/>
 </segment>
 </net>
@@
 <wire x1="142.24" y1="-86.36" x2="137.16" y2="-86.36" width="0.1524" layer="91"/>
 <junction x="137.16" y="-86.36"/>
-<wire x1="127" y1="-88.9" x2="137.16" y2="-88.9" width="0.1524" layer="91"/>
-<pinref part="M2-4" gate="G$1" pin="P$1"/>
+<pinref part="U$27" gate="G$1" pin="P$1"/>
+<wire x1="137.16" y1="-88.9" x2="129.54" y2="-88.9" width="0.1524" layer="91"/>
 </segment>
 <segment>
@@
 </segment>
 </net>
+<net name="N$3" class="0">
+<segment>
+<pinref part="X1" gate="-4" pin="S"/>
+<wire x1="27.94" y1="-175.26" x2="48.26" y2="-175.26" width="0.1524" layer="91"/>
+<pinref part="M2-3" gate="G$1" pin="P$1"/>
+<wire x1="60.96" y1="-162.56" x2="48.26" y2="-162.56" width="0.1524" layer="91"/>
+<wire x1="48.26" y1="-162.56" x2="48.26" y2="-175.26" width="0.1524" layer="91"/>
+</segment>
+</net>
+<net name="N$8" class="0">
+<segment>
+<pinref part="X1" gate="-2" pin="S"/>
+<wire x1="27.94" y1="-180.34" x2="48.26" y2="-180.34" width="0.1524" layer="91"/>
+<pinref part="M2-4" gate="G$1" pin="P$1"/>
+<wire x1="60.96" y1="-185.42" x2="48.26" y2="-185.42" width="0.1524" layer="91"/>
+<wire x1="48.26" y1="-185.42" x2="48.26" y2="-180.34" width="0.1524" layer="91"/>
+</segment>
+</net>
+<net name="N$11" class="0">
+<segment>
+<pinref part="X1" gate="-1" pin="S"/>
+<wire x1="27.94" y1="-182.88" x2="45.72" y2="-182.88" width="0.1524" layer="91"/>
+<pinref part="M2-2" gate="G$1" pin="P$1"/>
+<wire x1="60.96" y1="-198.12" x2="45.72" y2="-198.12" width="0.1524" layer="91"/>
+<wire x1="45.72" y1="-198.12" x2="45.72" y2="-182.88" width="0.1524" layer="91"/>
+</segment>
+</net>
+<net name="N$5" class="0">
+<segment>
+<pinref part="M2-1" gate="G$1" pin="P$1"/>
+<wire x1="60.96" y1="-172.72" x2="50.8" y2="-172.72" width="0.1524" layer="91"/>
+<wire x1="50.8" y1="-172.72" x2="50.8" y2="-177.8" width="0.1524" layer="91"/>
+<pinref part="X1" gate="-3" pin="S"/>
+<wire x1="50.8" y1="-177.8" x2="27.94" y2="-177.8" width="0.1524" layer="91"/>
+</segment>
+</net>
