File: 2016/PT_2016_PB_4lyr_Rev2.brd (EAGLE design)
At the start: 154.7 x 201.9 mm, 143 parts, among them M1+ ANDERSON_POWERPOLEPP45_PCB_HO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, M1- ANDERSON_POWERPOLEPP45_PCB_HO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, M2+ ANDERSON_POWERPOLEPP45_PCB_HO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, M2- ANDERSON_POWERPOLEPP45_PCB_HO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, M3+ ANDERSON_POWERPOLEPP45_PCB_HO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, M3- ANDERSON_POWERPOLEPP45_PCB_HO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, M4+ ANDERSON_POWERPOLEPP45_PCB_HO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, M4- ANDERSON_POWERPOLEPP45_PCB_HO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, M5+ ANDERSON_POWERPOLEPP45_PCB_HO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, M5- ANDERSON_POWERPOLEPP45_PCB_HO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, M6+ ANDERSON_POWERPOLEPP45_PCB_HO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, M6- ANDERSON_POWERPOLEPP45_PCB_HO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, Q1 Q_IRFS7437PbF, Q11 Q_IRFS7437PbF, Q12 2N7002, Q14 Q_IRFS7437PbF, Q16 Q_IRFS7437PbF, Q2 2N7002, Q20 Q_IRFS7437PbF, Q6 Q_IRFS7437PbF, Q7 Q_IRFS7437PbF, Q9 Q_IRFS7437PbF

Commit message: Changed 5V Caps
Parts:
- removed C50, C52: 10uF, resistor:C1206
- removed C51: 1nF, resistor:C1206
- added C18: 1nF, resistor:C1206
- added C21: 10uF, resistor:C1206
- added C22: .1uF, resistor:C1206
- C49: value 1nF -> .1uF
Connections:
- net +5V: no longer C50.1, C51.1, C52.1
- net GND: now also C18.2, C21.2, C22.2; no longer C50.2, C51.2, C52.2
- net V_BATT: now also C18.1, C21.1, C22.1
Routing:
- net +5V: track 111.2 -> 108.4 mm
- net GND: track 145.2 -> 142.4 mm
Changed lines of the file:
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@@
 <element name="C47" library="resistor" package="C1206" value="1nF" x="-48.006" y="128.016"/>
 <element name="C48" library="resistor" package="C1206" value="10uF" x="-48.006" y="125.222"/>
-<element name="C49" library="resistor" package="C1206" value="1nF" x="-42.418" y="131.064" rot="R180"/>
-<element name="C50" library="resistor" package="C1206" value="10uF" x="-42.418" y="128.016" rot="R180"/>
-<element name="C51" library="resistor" package="C1206" value="1nF" x="-42.418" y="125.222" rot="R180"/>
-<element name="C52" library="resistor" package="C1206" value="10uF" x="-52.07" y="129.286" rot="R90"/>
+<element name="C49" library="resistor" package="C1206" value=".1uF" x="-42.418" y="131.064" rot="R180"/>
 <element name="Q1" library="MRDT-2015-PowerBoard" package="D2PACK" value="Q_IRFS7437PbF" x="29.21" y="125.73" rot="R270"/>
 <element name="U$1" library="Jake" package="SO8" value="LT1910" x="13.208" y="126.746" rot="R270"/>
@@
 <element name="C15" library="resistor" package="C1206" value="1nF" x="-18.796" y="-29.464"/>
 <element name="C17" library="resistor" package="C1206" value="1nF" x="-18.796" y="-35.306"/>
+<element name="C18" library="resistor" package="C1206" value="1nF" x="-48.006" y="-52.832"/>
+<element name="C21" library="resistor" package="C1206" value="10uF" x="-48.006" y="-41.148"/>
+<element name="C22" library="resistor" package="C1206" value=".1uF" x="-48.006" y="-46.99"/>
 </elements>
 <signals>
@@
 <contactref element="R13" pad="2"/>
 <contactref element="C47" pad="2"/>
-<contactref element="C52" pad="2"/>
-<contactref element="C51" pad="2"/>
-<contactref element="C50" pad="2"/>
 <contactref element="C49" pad="2"/>
 <contactref element="C48" pad="2"/>
@@
 <wire x1="29.08" y1="141.732" x2="31.115" y2="143.767" width="0.4064" layer="1"/>
 <wire x1="31.115" y1="143.767" x2="31.115" y2="144.145" width="0.4064" layer="1"/>
-<wire x1="-43.818" y1="125.222" x2="-43.818" y2="128.016" width="0.4064" layer="1"/>
 <wire x1="36.96" y1="157.226" x2="38.354" y2="157.226" width="0.4064" layer="1"/>
 <via x="38.354" y="157.226" extent="1-16" drill="0.5"/>
@@
 <wire x1="15.494" y1="160.782" x2="15.24" y2="161.036" width="0.3048" layer="16"/>
 <wire x1="15.24" y1="161.036" x2="14.986" y2="161.036" width="0.3048" layer="16"/>
+<contactref element="C18" pad="2"/>
+<contactref element="C22" pad="2"/>
+<contactref element="C21" pad="2"/>
 <wire x1="37.1445" y1="101.5395" x2="38.989" y2="104.588" width="0" layer="19" extent="1-1"/>
 <wire x1="10.608" y1="80.645" x2="15.748" y2="82.296" width="0" layer="19" extent="1-16"/>
@@
 <wire x1="-17.396" y1="-29.464" x2="-17.396" y2="-23.622" width="0" layer="19" extent="1-1"/>
 <wire x1="-17.396" y1="-35.306" x2="-17.396" y2="-29.464" width="0" layer="19" extent="1-1"/>
-<wire x1="-43.818" y1="125.222" x2="7.62" y2="125.346" width="0" layer="19" extent="1-1"/>
-<wire x1="-46.606" y1="128.016" x2="-43.818" y2="128.016" width="0" layer="19" extent="1-1"/>
-<wire x1="-46.606" y1="130.556" x2="-46.606" y2="128.016" width="0" layer="19" extent="1-1"/>
-<wire x1="-46.606" y1="125.222" x2="-43.818" y2="125.222" width="0" layer="19" extent="1-1"/>
-<wire x1="-43.818" y1="131.064" x2="-46.606" y2="130.556" width="0" layer="19" extent="1-1"/>
-<wire x1="-52.07" y1="130.686" x2="-46.606" y2="130.556" width="0" layer="19" extent="1-1"/>
+<wire x1="-46.606" y1="-41.148" x2="-17.396" y2="-35.306" width="0" layer="19" extent="1-1"/>
+<wire x1="-46.606" y1="-46.99" x2="-46.606" y2="-41.148" width="0" layer="19" extent="1-1"/>
+<wire x1="-46.606" y1="-52.832" x2="-46.606" y2="-46.99" width="0" layer="19" extent="1-1"/>
+<wire x1="-43.818" y1="131.064" x2="7.62" y2="125.346" width="0" layer="19" extent="1-1"/>
+<wire x1="-46.606" y1="130.556" x2="-43.818" y2="131.064" width="0" layer="19" extent="1-1"/>
+<wire x1="-46.606" y1="128.016" x2="-46.606" y2="130.556" width="0" layer="19" extent="1-1"/>
+<wire x1="-46.606" y1="125.222" x2="-46.606" y2="128.016" width="0" layer="19" extent="1-1"/>
 </signal>
 <signal name="V_BATT">
@@
 <wire x1="80.772" y1="128.626" x2="80.772" y2="126.746" width="0.3048" layer="1"/>
 <wire x1="80.772" y1="126.746" x2="79.756" y2="126.746" width="0.3048" layer="1"/>
+<contactref element="C18" pad="1"/>
+<contactref element="C22" pad="1"/>
+<contactref element="C21" pad="1"/>
+<wire x1="-49.406" y1="-46.99" x2="-49.406" y2="-52.832" width="0" layer="19" extent="1-1"/>
+<wire x1="-49.406" y1="-41.148" x2="-49.406" y2="-46.99" width="0" layer="19" extent="1-1"/>
+<wire x1="41.9608" y1="7.68" x2="-49.406" y2="-41.148" width="0" layer="19" extent="1-1"/>
 </signal>
 <signal name="+5V">
@@
 <contactref element="LED5" pad="A"/>
 <contactref element="C47" pad="1"/>
-<contactref element="C52" pad="1"/>
-<contactref element="C51" pad="1"/>
-<contactref element="C50" pad="1"/>
 <contactref element="C49" pad="1"/>
 <contactref element="C48" pad="1"/>
@@
 <wire x1="-49.406" y1="130.556" x2="-49.406" y2="128.016" width="0.4064" layer="1"/>
 <wire x1="-49.406" y1="128.016" x2="-49.406" y2="125.222" width="0.4064" layer="1"/>
-<wire x1="-41.018" y1="128.016" x2="-41.018" y2="125.222" width="0.4064" layer="1"/>
 <wire x1="34.985" y1="160.782" x2="34.925" y2="160.722" width="0.4064" layer="1"/>
 <wire x1="34.925" y1="160.722" x2="34.925" y2="158.245" width="0.4064" layer="1"/>
@@
 <wire x1="34.925" y1="144.974" x2="38.608" y2="144.78" width="0" layer="19" extent="1-1"/>
 <wire x1="-41.018" y1="131.064" x2="34.16" y2="141.7193" width="0" layer="19" extent="1-1"/>
-<wire x1="-41.018" y1="128.016" x2="-41.018" y2="131.064" width="0" layer="19" extent="1-1"/>
-<wire x1="-49.406" y1="128.016" x2="-41.018" y2="128.016" width="0" layer="19" extent="1-1"/>
-<wire x1="-52.07" y1="127.886" x2="-49.406" y2="128.016" width="0" layer="19" extent="1-1"/>
+<wire x1="-49.406" y1="130.556" x2="-41.018" y2="131.064" width="0" layer="19" extent="1-1"/>
 </signal>
 <signal name="N$4">

Commit message: rerouting...
Parts:
- removed C10: 1uF, resistor:C1206
- added C34, C44, C50, C51, C52, C53: 1uF, resistor:C1206
- added U$30, U$31, U$32, U$33, U$34, U$35: APP_MOUTING_WINGHORIZ, MRDT-Connectors:APP45_MOUNTING_WING_HORIZ
- C13, C14, C15, C17: value 1nF -> 1uF
- U$2: device MRDT-2015-PowerBoard:SOIC8_ACS711_SKETCH -> MRDT-2015-PowerBoard:SOIC8_ACS711
- moved C13 234.8 mm to (161.3, 132.8)
- moved C14 234.8 mm to (161.3, 127.0)
- moved C15 234.8 mm to (161.3, 121.2)
- moved C17 234.8 mm to (161.3, 115.3)
- moved AUX1+ 185.0 mm to (168.7, 93.5)
- moved AUX1- 185.0 mm to (168.7, 93.5)
- moved C23 185.0 mm to (227.2, 8.51)
- moved C27 185.0 mm to (222.9, 80.4)
- moved C28 185.0 mm to (192.0, 57.4)
- moved C36 185.0 mm to (192.5, 104.9)
- moved C38 185.0 mm to (222.9, 10.3)
- moved C41 185.0 mm to (227.7, 95.1)
- moved C5 185.0 mm to (230.6, -6.10)
- moved LED1 185.0 mm to (217.7, -5.84)
- moved LED10 185.0 mm to (217.7, 80.4)
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Connections:
- new net N$11: C51.1
- new net N$3: C34.1
- new net N$5: C44.1
- new net N$71: C52.1
- new net N$72: C53.1
- new net N$8: C50.1
- net +5V: no longer C10.1
- net AUX_P-SIG: now also U$4.PA7; no longer U$4.PQ1
- net AUX_P2-SIG: now also U$4.PP5; no longer U$4.PK7
- net GND: now also C34.2, C44.2, C50.2, C51.2, C52.2, C53.2; no longer C10.2
- net M1-SIG: now also U$4.PK7; no longer U$4.PP5
- net M2-SIG: now also U$4.PQ1; no longer U$4.PA7
- net M3-SIG: now also U$4.PK6; no longer U$4.PH0
- net M4-SIG: now also U$4.PP3; no longer U$4.PH1
- net M5-SIG: now also U$4.PH1; no longer U$4.PP3
- net M6-SIG: now also U$4.PH0; no longer U$4.PK6
Routing:
- net GND: track 142.4 -> 329.8 mm, vias 24 -> 35
- net M1-IMEAS: track 242.4 -> 427.4 mm
- net M3-IMEAS: track 211.8 -> 396.8 mm
- net M2-IMEAS: track 227.3 -> 412.3 mm
- net M4-IMEAS: track 202.2 -> 387.1 mm
- net AUX_P2-IMEAS: track 0.00 -> 128.9 mm, vias 0 -> 1
- net AUX_P2-SIG: track 0.00 -> 95.4 mm, vias 0 -> 1
- net N$33: track 190.0 -> 160.9 mm
- net N$9: track 6.54 -> 25.5 mm
- net N$10: track 0.00 -> 6.44 mm
- net N$14: track 0.00 -> 5.33 mm
- net +5V: track 108.4 -> 104.8 mm
- net N$16: track 3.63 -> 2.45 mm
- added copper zone on layer 1, net +5V
- added copper zone on layer 1, net GND
- removed copper zone on layer 1, net N$28
- removed copper zone on layer 1, net N$40
- removed copper zone on layer 1, net N$44
- removed copper zone on layer 1, net N$54
- removed copper zone on layer 1, net N$60
- removed copper zone on layer 1, net N$66
- removed copper zone on layer 1, net N$78

Commit message: Routing
Parts:
- removed AUX1+, M1+, M2+, M3+, M4+, M5+, M6+: ANDERSON_POWERPOLEPP45_PCB_HORIZ_RIGHT_2HIGH, MRDT-Connectors:APP45_PCB_HORIZ_RIGHT_2HIGH
- removed AUX1-, M1-, M2-, M3-, M4-, M5-, M6-: ANDERSON_POWERPOLEPP45_PCB_HORIZ_RIGHT, MRDT-Connectors:APP45_PCB_HORIZ_RIGHT
- removed C16, C23, C24, C25, C26, C28, C29, C30, C32, C33, C36, C39, C41, C5: .1µF, resistor:C1206
- removed C27, C31, C35, C37, C38, C40, C42: 1nF, resistor:C1206
- removed LED1, LED10, LED11, LED12, LED6, LED7, LED8, LED9: (no value), SparkFun-LED:LED-1206
- removed Q11, Q14, Q16, Q20, Q6, Q7, Q9: Q_IRFS7437PbF, MRDT-2015-PowerBoard:D2PACK
- removed R16, R18, R20, R22, R24, R28, R5, R9: 5kΩ, SparkFun-Passives:1206
- removed U$10, U$11, U$13, U$6, U$7, U$8, U$9: LT1910, Jake:SO8
- removed U$14, U$15, U$16, U$17, U$18, U$19, U$20: ACS714LLCTR-50A-T, MRDT-2015-PowerBoard:SOIC8_ACS711_SKETCH
- added ACS714-M1, ACS714-M2, ACS714-M3, ACS714-M4, ACS714-M5, ACS714-M6, ACS714-M7, ACS714-M8: ACS714LLCTR-50A-T, MRDT-2015-PowerBoard:SOIC8_ACS711
- added ACS714CAP-M1, ACS714CAP-M2, ACS714CAP-M3, ACS714CAP-M4, ACS714CAP-M5, ACS714CAP-M6, ACS714CAP-M7, LT1910CAP-M1, LT1910CAP-M2, LT1910CAP-M3, LT1910CAP-M4, LT1910CAP-M5, LT1910CAP-M6, LT1910CAP-M7: .1µF, resistor:C1206
- added BOTAPP-M1, BOTAPP-M2, BOTAPP-M3, BOTAPP-M4, BOTAPP-M5, BOTAPP-M6, BOTAPP-M7: ANDERSON_POWERPOLEPP45_PCB_HORIZ_RIGHT, MRDT-Connectors:APP45_PCB_HORIZ_RIGHT
- added FET-M1, FET-M2, FET-M3, FET-M4, FET-M5, FET-M6, FET-M7: Q_IRFS7437PbF, MRDT-2015-PowerBoard:D2PACK
- added FILTERCAP-M1, FILTERCAP-M2, FILTERCAP-M3, FILTERCAP-M4, FILTERCAP-M5, FILTERCAP-M6, FILTERCAP-M7: 1nF, resistor:C1206
- added LED-M1, LED-M2, LED-M3, LED-M4, LED-M5, LED-M6, LED-M7, LED-M8: (no value), SparkFun-LED:LED-1206
- added LEDRES-M1, LEDRES-M2, LEDRES-M3, LEDRES-M4, LEDRES-M5, LEDRES-M6, LEDRES-M7, LEDRES-M8: 5kΩ, SparkFun-Passives:1206
- added LT1910-M1, LT1910-M2, LT1910-M3, LT1910-M4, LT1910-M5, LT1910-M6, LT1910-M7, LT1910-M8: LT1910, Jake:SO8
- added TOPAPP-M1, TOPAPP-M2, TOPAPP-M3, TOPAPP-M4, TOPAPP-M5, TOPAPP-M6, TOPAPP-M7: ANDERSON_POWERPOLEPP45_PCB_HORIZ_RIGHT_2HIGH, MRDT-Connectors:APP45_PCB_HORIZ_RIGHT_2HIGH
- U$1: value LT1910 -> TIVA-C-CONNECTED; device Jake:SO8 -> MRDT-2015-General:TIVA-C-CONNECTED
- U$2: value ACS714LLCTR-50A-T -> APP_MOUTING_WINGHORIZ; device MRDT-2015-PowerBoard:SOIC8_ACS711 -> MRDT-Connectors:APP45_MOUNTING_WING_HORIZ
- U$4: value TIVA-C-CONNECTED -> APP_MOUTING_WINGHORIZ; device MRDT-2015-General:TIVA-C-CONNECTED -> MRDT-Connectors:APP45_MOUNTING_WING_HORIZ
- moved U$42 197.2 mm to (8.38, 67.6)
- moved U$32 192.3 mm to (8.38, 99.1)
- moved U$30 188.6 mm to (8.38, 51.8)
- moved U$31 185.0 mm to (8.38, 36.1)
- moved U$34 110.2 mm to (8.38, 20.3)
- moved C44 109.0 mm to (69.3, 162.3), turned to 90 degrees
- moved C51 101.8 mm to (77.0, 162.3), turned to 90 degrees
- moved C52 101.7 mm to (71.9, 162.3), turned to 90 degrees
- moved C34 101.0 mm to (79.5, 162.3), turned to 90 degrees
- moved C50 94.8 mm to (82.0, 162.3), turned to 90 degrees
- moved C14 93.8 mm to (74.4, 162.3), turned to 90 degrees
- moved U$33 93.1 mm to (8.38, 4.57)
- moved C17 87.8 mm to (87.1, 162.3), turned to 90 degrees
- moved C15 87.0 mm to (84.6, 162.3), turned to 90 degrees
- moved U$35 85.9 mm to (8.38, 83.3), flipped to the bottom, turned to 180 degrees
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- renumbered AUX2+ to TOPAPP-M8, AUX2- to BOTAPP-M8, C7 to LT1910CAP-M8, C8 to ACS714CAP-M8, C9 to FILTERCAP-M8, Q1 to FET-M8
Connections:
- removed net AUX_P-IMEAS: U$20.7, U$4.PB4
- removed net AUX_P-SIG: U$13.4, U$4.PA7
- removed net AUX_P2-IMEAS: U$2.7, U$4.PD2
- removed net AUX_P2-SIG: U$1.4, U$4.PP5
- removed net M1-IMEAS: U$14.7, U$4.PK3
- removed net M1-SIG: U$4.PK7, U$6.4
- removed net M2-IMEAS: U$15.7, U$4.PK2
- removed net M2-SIG: U$4.PQ1, U$7.4
- removed net M3-IMEAS: U$19.7, U$4.PK1
- removed net M3-SIG: U$4.PK6, U$8.4
- removed net M4-IMEAS: U$18.7, U$4.PD4
- removed net M4-SIG: U$4.PP3, U$9.4
- removed net M5-IMEAS: U$17.7, U$4.PK0
- removed net M5-SIG: U$10.4, U$4.PH1
- removed net M6-IMEAS: U$16.7, U$4.PB5
- removed net M6-SIG: U$11.4, U$4.PH0
- removed net N$1: C37.1, U$14.6
- removed net N$10: FET-M8.2, R5.1, TOPAPP-M8.P$2
- removed net N$11: C51.1
- removed net N$14: FET-M8.1, U$1.5
- removed net N$15: LED11.A, R5.2
- removed net N$16: FILTERCAP-M8.1, U$2.6
- removed net N$17: C27.1, U$16.6
- removed net N$18: C14.1
- removed net N$19: C15.1
- removed net N$2: C38.1, U$15.6
- removed net N$20: C17.1
- removed net N$22: C31.1, U$17.6
- removed net N$23: C35.1, U$18.6
- removed net N$24: C40.1, U$19.6
- removed net N$25: C42.1, U$20.6
- removed net N$28: C24.2, Q7.TAB, U$15.4, U$7.6, U$7.8
- removed net N$29: M2+.P$2, Q7.2, R16.1
- removed net N$3: C34.1
- removed net N$30: Q7.1, U$7.5
- removed net N$31: LED6.A, R16.2
- removed net N$39: LED1.A, R9.2
- removed net N$40: C16.2, Q6.TAB, U$14.4, U$6.6, U$6.8
- removed net N$41: M1+.P$2, Q6.2, R9.1
- removed net N$42: Q6.1, U$6.5
- removed net N$44: C26.2, Q9.TAB, U$19.4, U$8.6, U$8.8
- removed net N$45: M3+.P$2, Q9.2, R18.1
- removed net N$47: Q9.1, U$8.5
- removed net N$49: LED7.A, R18.2
- removed net N$5: C44.1
- removed net N$54: C28.2, Q11.TAB, U$18.4, U$9.6, U$9.8
- removed net N$55: M4+.P$2, Q11.2, R20.1
- removed net N$56: Q11.1, U$9.5
- removed net N$57: LED8.A, R20.2
- removed net N$60: C30.2, Q14.TAB, U$10.6, U$10.8, U$17.4
- removed net N$61: M5+.P$2, Q14.2, R22.1
- removed net N$62: Q14.1, U$10.5
- removed net N$63: LED9.A, R22.2
- removed net N$66: C32.2, Q16.TAB, U$11.6, U$11.8, U$16.4
- removed net N$67: M6+.P$2, Q16.2, R24.1
- removed net N$68: Q16.1, U$11.5
- removed net N$69: LED10.A, R24.2
- removed net N$7: C13.1, REY-5V.P$6, REY-5V.P$7, U$3.1
- removed net N$72: C53.1
- removed net N$78: C36.2, Q20.TAB, U$13.6, U$13.8, U$20.4
- removed net N$79: AUX1+.P$2, Q20.2, R28.1
- removed net N$8: C50.1
- removed net N$80: Q20.1, U$13.5
- removed net N$81: LED12.A, R28.2
- removed net N$9: FET-M8.TAB, LT1910CAP-M8.2, U$1.6, U$1.8, U$2.4
- new net DRAIN-M1: ACS714-M1.4, FET-M1.TAB, LT1910-M1.6, LT1910-M1.8, LT1910CAP-M1.2
- new net DRAIN-M2: ACS714-M2.4, FET-M2.TAB, LT1910-M2.6, LT1910-M2.8, LT1910CAP-M2.2
- new net DRAIN-M3: ACS714-M3.4, FET-M3.TAB, LT1910-M3.6, LT1910-M3.8, LT1910CAP-M3.2
- new net DRAIN-M4: ACS714-M4.4, FET-M4.TAB, LT1910-M4.6, LT1910-M4.8, LT1910CAP-M4.2
- new net DRAIN-M5: ACS714-M5.4, FET-M5.TAB, LT1910-M5.6, LT1910-M5.8, LT1910CAP-M5.2
- new net DRAIN-M6: ACS714-M6.4, FET-M6.TAB, LT1910-M6.6, LT1910-M6.8, LT1910CAP-M6.2
- new net DRAIN-M7: ACS714-M7.4, FET-M7.TAB, LT1910-M7.6, LT1910-M7.8, LT1910CAP-M7.2
- new net DRAIN-M8: ACS714-M8.4, FET-M8.TAB, LT1910-M8.6, LT1910-M8.8, LT1910CAP-M8.2
- new net FILTER-M1: ACS714-M1.6, FILTERCAP-M1.1
- new net FILTER-M2: ACS714-M2.6, FILTERCAP-M2.1
- new net FILTER-M3: ACS714-M3.6, FILTERCAP-M3.1
- new net FILTER-M4: ACS714-M4.6, FILTERCAP-M4.1
- new net FILTER-M5: ACS714-M5.6, FILTERCAP-M5.1
- new net FILTER-M6: ACS714-M6.6, FILTERCAP-M6.1
- new net FILTER-M7: ACS714-M7.6, FILTERCAP-M7.1
- new net FILTER-M8: ACS714-M8.6, FILTERCAP-M8.1
- new net GATE-M1: FET-M1.1, LT1910-M1.5
- new net GATE-M2: FET-M2.1, LT1910-M2.5
- new net GATE-M3: FET-M3.1, LT1910-M3.5
- new net GATE-M4: FET-M4.1, LT1910-M4.5
- new net GATE-M5: FET-M5.1, LT1910-M5.5
- new net GATE-M6: FET-M6.1, LT1910-M6.5
- new net GATE-M7: FET-M7.1, LT1910-M7.5
- new net GATE-M8: FET-M8.1, LT1910-M8.5
- new net IMEAS-M1: ACS714-M1.7, U$1.PK3
- new net IMEAS-M2: ACS714-M2.7, U$1.PK2
- new net IMEAS-M3: ACS714-M3.7, U$1.PK1
- new net IMEAS-M4: ACS714-M4.7, U$1.PD4
- new net IMEAS-M5: ACS714-M5.7, U$1.PK0
- new net IMEAS-M6: ACS714-M6.7, U$1.PB5
- new net IMEAS-M7: ACS714-M7.7, U$1.PB4
- new net IMEAS-M8: ACS714-M8.7, U$1.PD2
- new net LEDLINE-M1: LED-M1.A, LEDRES-M1.2
- new net LEDLINE-M2: LED-M2.A, LEDRES-M2.2
- new net LEDLINE-M3: LED-M3.A, LEDRES-M3.2
- new net LEDLINE-M4: LED-M4.A, LEDRES-M4.2
- new net LEDLINE-M5: LED-M5.A, LEDRES-M5.2
- new net LEDLINE-M6: LED-M6.A, LEDRES-M6.2
- new net LEDLINE-M7: LED-M7.A, LEDRES-M7.2
- new net LEDLINE-M8: LED-M8.A, LEDRES-M8.2
- new net SIG-M1: LT1910-M1.4, U$1.PK7
- new net SIG-M2: LT1910-M2.4, U$1.PQ1
- new net SIG-M3: LT1910-M3.4, U$1.PK6
- new net SIG-M4: LT1910-M4.4, U$1.PP3
- new net SIG-M5: LT1910-M5.4, U$1.PH1
- new net SIG-M6: LT1910-M6.4, U$1.PH0
- new net SIG-M7: LT1910-M7.4, U$1.PA7
- new net SIG-M8: LT1910-M8.4, U$1.PP5
- new net SOURCE-M1: FET-M1.2, LEDRES-M1.1, TOPAPP-M1.P$2
- new net SOURCE-M2: FET-M2.2, LEDRES-M2.1, TOPAPP-M2.P$2
- new net SOURCE-M3: FET-M3.2, LEDRES-M3.1, TOPAPP-M3.P$2
- new net SOURCE-M4: FET-M4.2, LEDRES-M4.1, TOPAPP-M4.P$2
- new net SOURCE-M5: FET-M5.2, LEDRES-M5.1, TOPAPP-M5.P$2
- new net SOURCE-M6: FET-M6.2, LEDRES-M6.1, TOPAPP-M6.P$2
- new net SOURCE-M7: FET-M7.2, LEDRES-M7.1, TOPAPP-M7.P$2
- new net SOURCE-M8: FET-M8.2, LEDRES-M8.1, TOPAPP-M8.P$2
- net +5V: now also ACS714-M1.8, ACS714-M2.8, ACS714-M3.8, ACS714-M4.8, ACS714-M5.8, ACS714-M6.8, ACS714-M7.8, ACS714-M8.8, ACS714CAP-M1.2, ACS714CAP-M2.2, ACS714CAP-M3.2, ACS714CAP-M4.2, ACS714CAP-M5.2, ACS714CAP-M6.2, ACS714CAP-M7.2, U$1.+5V_1, U$1.+5V_2; no longer C23.2, C25.2, C29.2, C33.2, C39.2, C41.2, C5.2, U$14.8, U$15.8, U$16.8, U$17.8, U$18.8, U$19.8, U$2.8, U$20.8, U$4.+5V_1, U$4.+5V_2
- net 12V-IMEAS: now also U$1.PD1; no longer U$4.PD1
- net 12V-SIG: now also U$1.PN3; no longer U$4.PN3
- net 5V-IMEAS: now also U$1.PD0; no longer U$4.PD0
- net 5V-SIG: now also U$1.PP2; no longer U$4.PP2
- net GND: now also ACS714-M1.5, ACS714-M2.5, ACS714-M3.5, ACS714-M4.5, ACS714-M5.5, ACS714-M6.5, ACS714-M7.5, ACS714-M8.5, ACS714CAP-M1.1, ACS714CAP-M2.1, ACS714CAP-M3.1, ACS714CAP-M4.1, ACS714CAP-M5.1, ACS714CAP-M6.1, ACS714CAP-M7.1, BOTAPP-M1.P$1, BOTAPP-M2.P$1, BOTAPP-M3.P$1, BOTAPP-M4.P$1, BOTAPP-M5.P$1, BOTAPP-M6.P$1, BOTAPP-M7.P$1, FILTERCAP-M1.2, FILTERCAP-M2.2, FILTERCAP-M3.2, FILTERCAP-M4.2, FILTERCAP-M5.2, FILTERCAP-M6.2, FILTERCAP-M7.2, LED-M1.C, LED-M2.C, LED-M3.C, LED-M4.C, LED-M5.C, LED-M6.C, LED-M7.C, LED-M8.C, LT1910-M1.1, LT1910-M2.1, LT1910-M3.1, LT1910-M4.1, LT1910-M5.1, LT1910-M6.1, LT1910-M7.1, LT1910-M8.1, LT1910CAP-M1.1, LT1910CAP-M2.1, LT1910CAP-M3.1, LT1910CAP-M4.1, LT1910CAP-M5.1, LT1910CAP-M6.1, LT1910CAP-M7.1, U$1.GND_1, U$1.GND_2, U$1.GND_3, U$1.GND_4; no longer AUX1-.P$1, C16.1, C23.1, C24.1, C25.1, C26.1, C27.2, C28.1, C29.1, C30.1, C31.2, C32.1, C33.1, C35.2, C36.1, C37.2, C38.2, C39.1, C40.2, C41.1, C42.2, C5.1, LED1.C, LED10.C, LED11.C, LED12.C, LED6.C, LED7.C, LED8.C, LED9.C, M1-.P$1, M2-.P$1, M3-.P$1, M4-.P$1, M5-.P$1, M6-.P$1, U$1.1, U$10.1, U$11.1, U$13.1, U$14.5, U$15.5, U$16.5, U$17.5, U$18.5, U$19.5, U$2.5, U$20.5, U$4.GND_1, U$4.GND_2, U$4.GND_3, U$4.GND_4, U$6.1, U$7.1, U$8.1, U$9.1
- net N$100: now also U$1.RST1, U$1.RST_2; no longer U$4.RST1, U$4.RST_2
- net N$101: now also U$1.PB2; no longer U$4.PB2
- net N$102: now also U$1.PB3; no longer U$4.PB3
- net N$108: now also U$1.PD3; no longer U$4.PD3
- net N$110: now also U$1.PD5; no longer U$4.PD5
- net N$112: now also U$1.PE0; no longer U$4.PE0
- net N$113: now also U$1.PE1; no longer U$4.PE1
- net N$115: now also U$1.PE2; no longer U$4.PE2
- net N$116: now also U$1.PE3; no longer U$4.PE3
- net N$117: now also U$1.PE4; no longer U$4.PE4
- net N$118: now also U$1.PE5; no longer U$4.PE5
- net N$119: now also U$1.PG0; no longer U$4.PG0
- net N$120: now also U$1.PG1; no longer U$4.PG1
- net N$121: now also U$1.PL0; no longer U$4.PL0
- net N$122: now also U$1.PL1; no longer U$4.PL1
- net N$123: now also U$1.PL2; no longer U$4.PL2
- net N$124: now also U$1.PL3; no longer U$4.PL3
- net N$125: now also U$1.PL4; no longer U$4.PL4
- net N$129: now also U$1.PN4; no longer U$4.PN4
- net N$130: now also U$1.PN5; no longer U$4.PN5
- net N$131: now also U$1.PQ0; no longer U$4.PQ0
- net N$133: now also U$1.PQ2/PA3; no longer U$4.PQ2/PA3
- net N$134: now also U$1.PQ3/PA2; no longer U$4.PQ3/PA2
- net N$21: now also U$1.PH3; no longer U$4.PH3
- net N$35: now also U$1.PA4; no longer U$4.PA4
- net N$36: now also U$1.PA5; no longer U$4.PA5
- net N$37: now also U$1.PA6; no longer U$4.PA6
- net N$50: now also U$1.PC6; no longer U$4.PC6
- net N$51: now also U$1.PC7; no longer U$4.PC7
- net N$52: now also U$1.PF1; no longer U$4.PF1
- net N$53: now also U$1.PF2; no longer U$4.PF2
- net N$58: now also U$1.PF3; no longer U$4.PF3
- net N$70: now also U$1.PH2; no longer U$4.PH2
- net N$71: now also C13.1, C14.1, C15.1, C17.1, C34.1, C44.1, C50.1, C51.1, C53.1, REY-5V.P$6, REY-5V.P$7, U$3.1
- net N$75: now also U$1.PK4; no longer U$4.PK4
- net N$82: now also U$1.PK5; no longer U$4.PK5
- net N$83: now also U$1.PM0; no longer U$4.PM0
- net N$84: now also U$1.PM1; no longer U$4.PM1
- net N$85: now also U$1.PM2; no longer U$4.PM2
- net N$86: now also U$1.PM3; no longer U$4.PM3
- net N$87: now also U$1.PM4; no longer U$4.PM4
- net N$88: now also U$1.PM5; no longer U$4.PM5
- net N$89: now also U$1.PM6; no longer U$4.PM6
- net N$90: now also U$1.PM7; no longer U$4.PM7
- net N$93: now also U$1.PP4; no longer U$4.PP4
- net N$96: now also U$1.PN2; no longer U$4.PN2
- net N$98: now also U$1.+3V3_1, U$1.+3V3_2; no longer U$4.+3V3_1, U$4.+3V3_2
- net N$99: now also U$1.PL5; no longer U$4.PL5
- net PRIMARY-VMEAS: now also U$1.PD7; no longer U$4.PD7
- net RX1: now also U$1.PC4; no longer U$4.PC4
- net RX2: now also U$1.PP0; no longer U$4.PP0
- net TX1: now also U$1.PC5; no longer U$4.PC5
- net TX2: now also U$1.PP1; no longer U$4.PP1
- net V_BATT: now also ACS714-M1.1, ACS714-M2.1, ACS714-M3.1, ACS714-M4.1, ACS714-M5.1, ACS714-M6.1, ACS714-M7.1, ACS714-M8.1; no longer U$14.1, U$15.1, U$16.1, U$17.1, U$18.1, U$19.1, U$2.1, U$20.1
Routing:
- net M2-IMEAS: track 412.3 -> 212.1 mm, vias 1 -> 0
- net M3-IMEAS: track 396.8 -> 197.0 mm, vias 1 -> 0
- net M1-IMEAS: track 427.4 -> 227.9 mm, vias 1 -> 0
- net M4-IMEAS: track 387.1 -> 200.1 mm, vias 1 -> 0
- net SIG-M1: track 0.00 -> 183.2 mm, vias 0 -> 1
- net SIG-M2: track 0.00 -> 172.4 mm, vias 0 -> 1
- net GND: track 329.8 -> 170.2 mm, vias 35 -> 36
- net SIG-M3: track 0.00 -> 155.0 mm, vias 0 -> 1
- net SIG-M4: track 0.00 -> 145.1 mm, vias 0 -> 1
- net 12V-IMEAS: track 135.9 -> 0.00 mm, vias 3 -> 0
- net AUX_P2-IMEAS: track 128.9 -> 0.00 mm, vias 1 -> 0
- net SIG-M5: track 0.00 -> 128.5 mm, vias 0 -> 1
- net N$7: track 120.9 -> 0.00 mm
- net 5V-IMEAS: track 119.1 -> 0.00 mm, vias 3 -> 0
- net SIG-M6: track 0.00 -> 115.5 mm, vias 0 -> 1
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- added copper zone on layer 1, net DRAIN-M1
- added copper zone on layer 1, net DRAIN-M2
- added copper zone on layer 1, net DRAIN-M3
- added copper zone on layer 1, net DRAIN-M4
- added copper zone on layer 1, net DRAIN-M5
- added copper zone on layer 1, net DRAIN-M6
- added copper zone on layer 1, net DRAIN-M7
- added copper zone on layer 1, net DRAIN-M8
- added copper zone on layer 1, net N$72
- added copper zone on layer 1, net SOURCE-M1
- added copper zone on layer 1, net SOURCE-M2
- added copper zone on layer 1, net SOURCE-M3
- added copper zone on layer 1, net SOURCE-M4
- added copper zone on layer 1, net SOURCE-M5
- added copper zone on layer 1, net SOURCE-M6
- added copper zone on layer 1, net SOURCE-M7
- added copper zone on layer 1, net SOURCE-M8
- removed copper zone on layer 1, net N$10
- removed copper zone on layer 1, net N$7
- removed copper zone on layer 1, net N$9
