File: 2016/Rev2/PT_2016_PB_4lyr_Rev2.brd (EAGLE design)
At the start: 153.9 x 200.4 mm, 156 parts, among them Q12 2N7002, Q2 2N7002

Commit message: github is stupid. i changed some stuff. this is final rev2
Parts:
- added U$10, U$11, U$8: MOUNTING_HOLE#8, MRDT-Hardware:#8_SCREW
- moved U$22 6.48 mm to (125.0, 15.2)
- moved LT1910-M8 6.15 mm to (18.8, 130.3)
- moved LT1910-M4 6.15 mm to (18.8, 67.3)
- moved C13 6.15 mm to (97.0, 166.1)
- moved C14 6.15 mm to (79.2, 166.1)
- moved C15 6.15 mm to (89.4, 166.1)
- moved C34 6.15 mm to (84.3, 166.1)
- moved C44 6.15 mm to (74.2, 166.1)
- moved Q2 6.15 mm to (124.2, 150.9)
- moved R1 6.15 mm to (114.0, 178.3)
- moved R11 6.15 mm to (129.3, 150.1)
- moved R4 6.15 mm to (88.1, 133.9)
- moved R7 6.15 mm to (119.1, 178.3)
- moved U$12 6.15 mm to (111.8, 183.6)
- moved LT1910-M3 6.15 mm to (18.8, 51.5)
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Connections:
- net 12V-SIG renamed SIG-12V
- net 5V-SIG renamed SIG-5V
- removed net 12V-IMEAS: U$1.PD3, U$21.7
- removed net 5V-IMEAS: U$1.PE5, U$3.7
- removed net N$112: U$1.PE0
- removed net N$113: U$1.PE1
- removed net N$115: U$1.PE2
- removed net N$116: U$1.PE3
- removed net N$117: U$1.PE4
- removed net N$119: U$1.PG0
- removed net N$120: U$1.PG1
- removed net N$121: U$1.PL0
- removed net N$122: U$1.PL1
- removed net N$123: U$1.PL2
- removed net N$124: U$1.PL3
- removed net N$125: U$1.PL4
- removed net N$129: U$1.PN4
- removed net N$130: U$1.PN5
- removed net N$131: U$1.PQ0
- removed net N$133: U$1.PQ2/PA3
- removed net N$134: U$1.PQ3/PA2
- removed net N$21: U$1.PH3
- removed net N$35: U$1.PA4
- removed net N$36: U$1.PA5
- removed net N$37: U$1.PA6
- removed net N$50: U$1.PC6
- removed net N$51: U$1.PC7
- removed net N$52: U$1.PF1
- removed net N$53: U$1.PF2
- removed net N$58: U$1.PF3
- removed net N$70: U$1.PH2
- removed net N$75: U$1.PK4
- removed net N$82: U$1.PK5
- removed net N$83: U$1.PM0
- removed net N$84: U$1.PM1
- removed net N$85: U$1.PM2
- removed net N$86: U$1.PM3
- removed net N$87: U$1.PM4
- removed net N$88: U$1.PM5
- removed net N$89: U$1.PM6
- removed net N$90: U$1.PM7
- removed net N$93: U$1.PP4
- removed net N$96: U$1.PN2
- removed net N$99: U$1.PL5
- removed net PRIMARY-VMEAS: R3.1, R4.2, U$1.PD7
- new net IMEAS-12V: U$1.PD7, U$21.7
- new net IMEAS-5V: U$1.PE2, U$3.7
- new net VMEAS-VBATT: R3.1, R4.2, U$1.PE3
Routing:
- net VMEAS-VBATT: track 0.00 -> 201.3 mm, vias 0 -> 1
- net PRIMARY-VMEAS: track 197.9 -> 0.00 mm, vias 1 -> 0
- net 12V-IMEAS: track 155.4 -> 0.00 mm, vias 1 -> 0
- net IMEAS-12V: track 0.00 -> 153.0 mm, vias 0 -> 1
- net 5V-IMEAS: track 138.3 -> 0.00 mm, vias 1 -> 0
- net IMEAS-5V: track 0.00 -> 137.4 mm, vias 0 -> 1
- net +5V: track 70.1 -> 53.2 mm
- net SIG-M6: track 115.5 -> 120.2 mm
- net SIG-M8: track 96.9 -> 101.4 mm
- net SIG-M7: track 110.1 -> 114.7 mm
- net SIG-M5: track 128.5 -> 133.0 mm
- net SIG-M4: track 145.1 -> 149.7 mm
- net SIG-M3: track 155.0 -> 159.5 mm
- net SIG-M2: track 172.4 -> 177.0 mm
- net SIG-M1: track 183.2 -> 187.7 mm
Other:
- board text added: "Missouri S&T Mars Rover Cameron Nichols Power Board 2016"
- board text removed: "MORE MOUNTING HOLES?"
- board text removed: "Missouri S&T Mars Rover Design Team Power Board 2016"
