File: 2016/Rev2/PT_2016_PB_4lyr_Rev2.sch (EAGLE design)
At the start: 155 parts, among them Q12 2N7002, Q2 2N7002

Commit message: github is stupid. i changed some stuff. this is final rev2
Parts:
- added U$10, U$11, U$8: MOUNTING_HOLE#8, MRDT-Hardware:MOUNTING_HOLE#8
Connections:
- net 12V-SIG renamed SIG-12V
- net 5V-SIG renamed SIG-5V
- removed net 12V-IMEAS: U$1.PD3, U$21.VIOUT
- removed net 5V-IMEAS: U$1.PE5, U$3.VIOUT
- removed net N$112: U$1.PE0
- removed net N$113: U$1.PE1
- removed net N$115: U$1.PE2
- removed net N$116: U$1.PE3
- removed net N$117: U$1.PE4
- removed net N$119: U$1.PG0
- removed net N$120: U$1.PG1
- removed net N$121: U$1.PL0
- removed net N$122: U$1.PL1
- removed net N$123: U$1.PL2
- removed net N$124: U$1.PL3
- removed net N$125: U$1.PL4
- removed net N$129: U$1.PN4
- removed net N$130: U$1.PN5
- removed net N$131: U$1.PQ0
- removed net N$133: U$1.PQ2/PA3
- removed net N$134: U$1.PQ3/PA2
- removed net N$21: U$1.PH3
- removed net N$35: U$1.PA4
- removed net N$36: U$1.PA5
- removed net N$37: U$1.PA6
- removed net N$50: U$1.PC6
- removed net N$51: U$1.PC7
- removed net N$52: U$1.PF1
- removed net N$53: U$1.PF2
- removed net N$58: U$1.PF3
- removed net N$70: U$1.PH2
- removed net N$75: U$1.PK4
- removed net N$82: U$1.PK5
- removed net N$83: U$1.PM0
- removed net N$84: U$1.PM1
- removed net N$85: U$1.PM2
- removed net N$86: U$1.PM3
- removed net N$87: U$1.PM4
- removed net N$88: U$1.PM5
- removed net N$89: U$1.PM6
- removed net N$90: U$1.PM7
- removed net N$93: U$1.PP4
- removed net N$96: U$1.PN2
- removed net N$99: U$1.PL5
- removed net PRIMARY-VMEAS: R3.1, R4.2, U$1.PD7
- new net IMEAS-12V: U$1.PD7, U$21.VIOUT
- new net IMEAS-5V: U$1.PE2, U$3.VIOUT
- new net VMEAS-VBATT: R3.1, R4.2, U$1.PE3
