File: PowerBoard_Hardware/PowerBoard_Hardware/PowerBoard_Hardware.kicad_pcb (KiCad board)
At the start: 2 copper layers, 74 parts, among them Q1 Q_NMOS_DGS, Q2 Q_NMOS_DGS, Q3 Q_NMOS_DGS, Q4 Q_NMOS_DGS, Q5 Q_NMOS_DGS, Q6 Q_NMOS_DGS, Q7 Q_NMOS_DGS, U1 LT1910, U10 LT1910, U11 LT1910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

Commit message: Pass 1.6
*Pins were rearranged on the schematic appropriately
*Layout has been cleaned up and generalized for PDR
*Problems still persist with Conn15-PVDD
Parts:
- Conn2, Conn3: footprint MRDT_Connectors:MOLEX_SL_10_Horizontal -> MRDT_Connectors:MOLEX_SL_10_Vertical
- moved Conn4 357.8 mm to (198.1, 47.0), turned to 180 degrees
- moved F5 262.2 mm to (158.8, 69.8)
- moved Conn3 261.5 mm to (142.2, 36.8)
- moved F1 246.7 mm to (158.8, 38.1)
- moved Conn1 244.3 mm to (129.5, 144.8)
- moved Conn15 237.7 mm to (149.9, 144.8)
- moved Conn9 233.1 mm to (81.3, 61.0)
- moved F4 232.0 mm to (160.0, 100.3)
- moved Conn2 228.9 mm to (114.3, 36.8)
- moved Conn10 228.7 mm to (81.3, 94.0)
- moved F2 228.6 mm to (160.0, 133.3)
- moved Conn7 228.4 mm to (198.1, 108.0)
- moved Conn8 228.3 mm to (198.0, 79.9)
- moved Conn6 228.1 mm to (81.3, 127.0)
- moved Conn5 225.4 mm to (198.1, 141.0)
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Connections:
- U10 pad 4: PE_0 -> PE_3
- U11 pad 4: PE_0 -> PC_4
- U2 pad 4: PE_0 -> PE_2
- U3 pad 4: PE_0 -> PE_4
- U4 pad 4: PE_0 -> PC_5
- U9 pad 4: PE_0 -> PE_1

Commit message: Pass 1.7
Parts:
- moved Conn15 71.8 mm to (200.7, 195.6), turned to 180 degrees
- moved Conn1 51.1 mm to (106.7, 190.5)
- moved C10 33.0 mm to (174.0, 186.7)
- moved C2 33.0 mm to (162.6, 186.7)
- moved C6 33.0 mm to (168.0, 186.7)
- moved Conn5 33.0 mm to (198.1, 174.0)
- moved F2 33.0 mm to (160.0, 166.4)
- moved Q2 33.0 mm to (168.9, 174.0)
- moved R2 33.0 mm to (184.2, 186.7)
- moved R6 33.0 mm to (179.9, 186.7)
- moved U2 33.0 mm to (182.9, 170.2)
- moved U6 33.0 mm to (182.9, 179.1)
- moved C3 32.1 mm to (128.3, 148.6)
- moved Conn6 32.1 mm to (111.8, 137.2)
- moved R7 32.1 mm to (148.6, 148.6)
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