File: Hardware/PackVoltage_2021_Rev1/Power_IN.sch (KiCad schematic (older format))
At the start: 8 parts

Commit message: Annotated Sheet, added Busses, Moved Andersons
Autocompleted annotations for sheet
Duplicated bus for Motor 1 to all other busses, split "Busses" sheet into "Motor Busses" and "Other Busses" for space.
Moved andersons from bus sheets to top level sheet.
Parts:
- gave numbers to parts that had none: 2
- renumbered C1 to C15, C2 to C16, D1 to D11, D2 to D12
Other:
- moved on the sheet: C?, D?, GND?, V?
Changed lines of the file:
@@
 $Descr A4 11693 8268
 encoding utf-8
-Sheet 5 5
+Sheet 5 6
 Title ""
 Date ""
@@
 L MRDT_Drill_Holes:BATT_PWR_VIA V1
 U 1 1 5F83ED6F
-P 2200 2400
-F 0 "V1" H 2328 2420 60  0000 L CNN
-F 1 "BATT_PWR_VIA" H 2328 2314 60  0000 L CNN
-F 2 "" H 2200 2400 60  0001 C CNN
-F 3 "" H 2200 2400 60  0001 C CNN
-	1    2200 2400
+P 1000 1150
+F 0 "V?" H 1128 1170 60  0000 L CNN
+F 1 "BATT_PWR_VIA" H 1128 1064 60  0000 L CNN
+F 2 "" H 1000 1150 60  0001 C CNN
+F 3 "" H 1000 1150 60  0001 C CNN
+	1    1000 1150
 	1    0    0    -1
 $EndComp
 $Comp
-L Device:CP1 C1
+L Device:CP1 C15
 U 1 1 5F83FC51
-P 2350 2850
-F 0 "C1" H 2465 2896 50  0000 L CNN
-F 1 "470uF" H 2465 2805 50  0000 L CNN
-F 2 "" H 2350 2850 50  0001 C CNN
-F 3 "~" H 2350 2850 50  0001 C CNN
-	1    2350 2850
+P 1150 1600
+F 0 "C?" H 1265 1646 50  0000 L CNN
+F 1 "470uF" H 1265 1555 50  0000 L CNN
+F 2 "" H 1150 1600 50  0001 C CNN
+F 3 "~" H 1150 1600 50  0001 C CNN
+	1    1150 1600
 	1    0    0    -1
 $EndComp
 $Comp
-L Device:CP1 C2
+L Device:CP1 C16
 U 1 1 5F840D70
-P 2750 2850
-F 0 "C2" H 2865 2896 50  0000 L CNN
-F 1 "470uF" H 2865 2805 50  0000 L CNN
-F 2 "" H 2750 2850 50  0001 C CNN
-F 3 "~" H 2750 2850 50  0001 C CNN
-	1    2750 2850
+P 1550 1600
+F 0 "C?" H 1665 1646 50  0000 L CNN
+F 1 "470uF" H 1665 1555 50  0000 L CNN
+F 2 "" H 1550 1600 50  0001 C CNN
+F 3 "~" H 1550 1600 50  0001 C CNN
+	1    1550 1600
 	1    0    0    -1
 $EndComp
 $Comp
-L Device:CP1 C?
+L Device:CP1 C17
 U 1 1 5F8410A5
-P 3150 2850
-F 0 "C?" H 3265 2896 50  0000 L CNN
-F 1 "CP1" H 3265 2805 50  0000 L CNN
-F 2 "" H 3150 2850 50  0001 C CNN
-F 3 "~" H 3150 2850 50  0001 C CNN
-	1    3150 2850
+P 1950 1600
+F 0 "C?" H 2065 1646 50  0000 L CNN
+F 1 "CP1" H 2065 1555 50  0000 L CNN
+F 2 "" H 1950 1600 50  0001 C CNN
+F 3 "~" H 1950 1600 50  0001 C CNN
+	1    1950 1600
 	1    0    0    -1
 $EndComp
 $Comp
-L Device:CP1 C?
+L Device:CP1 C18
 U 1 1 5F8414AB
-P 3550 2850
-F 0 "C?" H 3665 2896 50  0000 L CNN
-F 1 "CP1" H 3665 2805 50  0000 L CNN
-F 2 "" H 3550 2850 50  0001 C CNN
-F 3 "~" H 3550 2850 50  0001 C CNN
-	1    3550 2850
+P 2350 1600
+F 0 "C?" H 2465 1646 50  0000 L CNN
+F 1 "CP1" H 2465 1555 50  0000 L CNN
+F 2 "" H 2350 1600 50  0001 C CNN
+F 3 "~" H 2350 1600 50  0001 C CNN
+	1    2350 1600
 	1    0    0    -1
 $EndComp
 Wire Wire Line
-	2200 2600 2200 2700
+	1000 1350 1000 1450
 Wire Wire Line
-	2200 2700 2350 2700
+	1000 1450 1150 1450
 Wire Wire Line
-	2350 2700 2750 2700
-Connection ~ 2350 2700
-Connection ~ 2750 2700
+	1150 1450 1550 1450
+Connection ~ 1150 1450
+Connection ~ 1550 1450
 Wire Wire Line
-	2750 2700 3150 2700
-Connection ~ 3150 2700
+	1550 1450 1950 1450
+Connection ~ 1950 1450
 Wire Wire Line
-	3150 2700 3550 2700
+	1950 1450 2350 1450
 Wire Wire Line
-	2350 3000 2750 3000
-Connection ~ 2750 3000
+	1150 1750 1550 1750
+Connection ~ 1550 1750
 Wire Wire Line
-	2750 3000 3150 3000
-Connection ~ 3150 3000
+	1550 1750 1950 1750
+Connection ~ 1950 1750
 Wire Wire Line
-	3150 3000 3550 3000
-Connection ~ 3550 2700
+	1950 1750 2350 1750
+Connection ~ 2350 1450
 $Comp
-L power:GND #PWR?
+L power:GND #PWR049
 U 1 1 5F841CDF
-P 4650 3050
-F 0 "#PWR?" H 4650 2800 50  0001 C CNN
-F 1 "GND" H 4655 2877 50  0000 C CNN
-F 2 "" H 4650 3050 50  0001 C CNN
-F 3 "" H 4650 3050 50  0001 C CNN
-	1    4650 3050
+P 3450 1800
+F 0 "#PWR?" H 3450 1550 50  0001 C CNN
+F 1 "GND" H 3455 1627 50  0000 C CNN
+F 2 "" H 3450 1800 50  0001 C CNN
+F 3 "" H 3450 1800 50  0001 C CNN
+	1    3450 1800
 	1    0    0    -1
 $EndComp
 Wire Wire Line
-	4650 3000 4650 3050
+	3450 1750 3450 1800
 $Comp
 L MRDT_Drill_Holes:Via GND1
 U 1 1 5F842285
-P 2200 3350
-F 0 "GND1" H 2428 3408 60  0000 L CNN
-F 1 "Via" H 2428 3302 60  0000 L CNN
-F 2 "" H 2200 3350 60  0001 C CNN
-F 3 "" H 2200 3350 60  0001 C CNN
-	1    2200 3350
+P 1000 2100
+F 0 "GND?" H 1228 2158 60  0000 L CNN
+F 1 "Via" H 1228 2052 60  0000 L CNN
+F 2 "" H 1000 2100 60  0001 C CNN
+F 3 "" H 1000 2100 60  0001 C CNN
+	1    1000 2100
 	1    0    0    -1
 $EndComp
 $Comp
-L power:GND #PWR?
+L power:GND #PWR048
 U 1 1 5F8427B7
-P 2350 3600
-F 0 "#PWR?" H 2350 3350 50  0001 C CNN
-F 1 "GND" H 2355 3427 50  0000 C CNN
-F 2 "" H 2350 3600 50  0001 C CNN
-F 3 "" H 2350 3600 50  0001 C CNN
-	1    2350 3600
+P 1150 2350
+F 0 "#PWR?" H 1150 2100 50  0001 C CNN
+F 1 "GND" H 1155 2177 50  0000 C CNN
+F 2 "" H 1150 2350 50  0001 C CNN
+F 3 "" H 1150 2350 50  0001 C CNN
+	1    1150 2350
 	1    0    0    -1
 $EndComp
 Wire Wire Line
-	2200 3350 2350 3350
+	1000 2100 1150 2100
 Wire Wire Line
-	2350 3350 2350 3600
+	1150 2100 1150 2350
 $Comp
-L Device:D D1
+L Device:D D11
 U 1 1 5F844C01
-P 3900 2850
-F 0 "D1" V 3854 2930 50  0000 L CNN
-F 1 "D" V 3945 2930 50  0000 L CNN
-F 2 "" H 3900 2850 50  0001 C CNN
-F 3 "~" H 3900 2850 50  0001 C CNN
-	1    3900 2850
+P 2700 1600
+F 0 "D?" V 2654 1680 50  0000 L CNN
+F 1 "D" V 2745 1680 50  0000 L CNN
+F 2 "" H 2700 1600 50  0001 C CNN
+F 3 "~" H 2700 1600 50  0001 C CNN
+	1    2700 1600
 	0    1    1    0
 $EndComp
 $Comp
-L Device:D D2
+L Device:D D12
 U 1 1 5F845B68
-P 4350 2850
-F 0 "D2" V 4304 2930 50  0000 L CNN
-F 1 "D" V 4395 2930 50  0000 L CNN
-F 2 "" H 4350 2850 50  0001 C CNN
-F 3 "~" H 4350 2850 50  0001 C CNN
-	1    4350 2850
+P 3150 1600
+F 0 "D?" V 3104 1680 50  0000 L CNN
+F 1 "D" V 3195 1680 50  0000 L CNN
+F 2 "" H 3150 1600 50  0001 C CNN
+F 3 "~" H 3150 1600 50  0001 C CNN
+	1    3150 1600
 	0    1    1    0
 $EndComp
 Wire Wire Line
-	3550 2700 3900 2700
+	2350 1450 2700 1450
 Wire Wire Line
-	4450 2600 4450 2700
-Connection ~ 3900 2700
+	3250 1350 3250 1450
+Connection ~ 2700 1450
 Wire Wire Line
-	3900 2700 4350 2700
-Connection ~ 4350 2700
+	2700 1450 3150 1450
+Connection ~ 3150 1450
 Wire Wire Line
-	4350 2700 4450 2700
+	3150 1450 3250 1450
 Wire Wire Line
-	3550 3000 3900 3000
-Connection ~ 3550 3000
-Connection ~ 3900 3000
+	2350 1750 2700 1750
+Connection ~ 2350 1750
+Connection ~ 2700 1750
 Wire Wire Line
-	3900 3000 4350 3000
-Connection ~ 4350 3000
+	2700 1750 3150 1750
+Connection ~ 3150 1750
 Wire Wire Line
-	4350 3000 4650 3000
-Text HLabel 4450 2600 1    50   Output ~ 0
+	3150 1750 3450 1750
+Text HLabel 3250 1350 1    50   Output ~ 0
 PV
 $EndSCHEMATC
