File: Hardware/PackVoltage_2021_Rev1/PackVoltage_2021_Rev1.sch (KiCad schematic (older format))
At the start: 20 parts

Commit message: Renamed Andersons
Parts:
- Conn1: value AndersonPP -> Motor 1
- Conn10: value AndersonPP -> Driveboard
- Conn11: value AndersonPP -> Auxiliary
- Conn12: value AndersonPP -> Spare
- Conn2: value AndersonPP -> Rockets
- Conn3: value AndersonPP -> Motor 2
- Conn4: value AndersonPP -> 12 V
- Conn7: value AndersonPP -> Motor 3
- Conn8: value AndersonPP -> Vaccum
- Conn9: value AndersonPP -> Motor 4
Changed lines of the file:
@@
 AR Path="/5F94335D" Ref="Conn1"  Part="4"
 F 0 "Conn1" H 4758 5087 60  0000 C CNN
-F 1 "AndersonPP" H 4758 4981 60  0000 C CNN
+F 1 "Motor 1" H 4758 4981 60  0000 C CNN
 F 2 "MRDT_Connectors:Anderson_2_Horizontal_Side_by_Side" H 4400 4150 60  0001 C CNN
 F 3 "" H 4400 4150 60  0001 C CNN
@@
 AR Path="/5F943363" Ref="Conn1"  Part="1"
 F 0 "Conn1" H 4900 5500 60  0000 R CNN
-F 1 "AndersonPP" H 5050 5400 60  0000 R CNN
+F 1 "Motor 1" H 5050 5400 60  0000 R CNN
 F 2 "MRDT_Connectors:Anderson_2_Horizontal_Side_by_Side" H 4400 4600 60  0001 C CNN
 F 3 "" H 4400 4600 60  0001 C CNN
@@
 AR Path="/5F943377" Ref="Conn7"  Part="4"
 F 0 "Conn7" H 7058 5087 60  0000 C CNN
-F 1 "AndersonPP" H 7058 4981 60  0000 C CNN
+F 1 "Motor 3" H 7058 4981 60  0000 C CNN
 F 2 "MRDT_Connectors:Anderson_2_Horizontal_Side_by_Side" H 6700 4150 60  0001 C CNN
 F 3 "" H 6700 4150 60  0001 C CNN
@@
 AR Path="/5F94337D" Ref="Conn7"  Part="1"
 F 0 "Conn7" H 7200 5500 60  0000 R CNN
-F 1 "AndersonPP" H 7350 5400 60  0000 R CNN
+F 1 "Motor 3" H 7350 5400 60  0000 R CNN
 F 2 "MRDT_Connectors:Anderson_2_Horizontal_Side_by_Side" H 6700 4600 60  0001 C CNN
 F 3 "" H 6700 4600 60  0001 C CNN
@@
 AR Path="/5F94338B" Ref="Conn9"  Part="4"
 F 0 "Conn9" H 8208 5087 60  0000 C CNN
-F 1 "AndersonPP" H 8208 4981 60  0000 C CNN
+F 1 "Motor 4" H 8208 4981 60  0000 C CNN
 F 2 "MRDT_Connectors:Anderson_2_Horizontal_Side_by_Side" H 7850 4150 60  0001 C CNN
 F 3 "" H 7850 4150 60  0001 C CNN
@@
 AR Path="/5F943391" Ref="Conn9"  Part="1"
 F 0 "Conn9" H 8350 5500 60  0000 R CNN
-F 1 "AndersonPP" H 8500 5400 60  0000 R CNN
+F 1 "Motor 4" H 8500 5400 60  0000 R CNN
 F 2 "MRDT_Connectors:Anderson_2_Horizontal_Side_by_Side" H 7850 4600 60  0001 C CNN
 F 3 "" H 7850 4600 60  0001 C CNN
@@
 AR Path="/5F943399" Ref="Conn3"  Part="1"
 F 0 "Conn3" H 6050 5500 60  0000 R CNN
-F 1 "AndersonPP" H 6200 5400 60  0000 R CNN
+F 1 "Motor 2" H 6200 5400 60  0000 R CNN
 F 2 "MRDT_Connectors:Anderson_2_Horizontal_Side_by_Side" H 5550 4600 60  0001 C CNN
 F 3 "" H 5550 4600 60  0001 C CNN
@@
 AR Path="/5F94339F" Ref="Conn3"  Part="4"
 F 0 "Conn3" H 5908 5087 60  0000 C CNN
-F 1 "AndersonPP" H 5908 4981 60  0000 C CNN
+F 1 "Motor 2" H 5908 4981 60  0000 C CNN
 F 2 "MRDT_Connectors:Anderson_2_Horizontal_Side_by_Side" H 5550 4150 60  0001 C CNN
 F 3 "" H 5550 4150 60  0001 C CNN
@@
 AR Path="/5F9A1793" Ref="Conn2"  Part="4"
 F 0 "Conn2" H 4758 6237 60  0000 C CNN
-F 1 "AndersonPP" H 4758 6131 60  0000 C CNN
+F 1 "Rockets" H 4758 6131 60  0000 C CNN
 F 2 "MRDT_Connectors:Anderson_2_Horizontal_Side_by_Side" H 4400 5300 60  0001 C CNN
 F 3 "" H 4400 5300 60  0001 C CNN
@@
 AR Path="/5F9A1799" Ref="Conn2"  Part="1"
 F 0 "Conn2" H 4900 6650 60  0000 R CNN
-F 1 "AndersonPP" H 5050 6550 60  0000 R CNN
+F 1 "Rockets" H 5050 6550 60  0000 R CNN
 F 2 "MRDT_Connectors:Anderson_2_Horizontal_Side_by_Side" H 4400 5750 60  0001 C CNN
 F 3 "" H 4400 5750 60  0001 C CNN
@@
 AR Path="/5F9A17A7" Ref="Conn4"  Part="4"
 F 0 "Conn4" H 5908 6237 60  0000 C CNN
-F 1 "AndersonPP" H 5908 6131 60  0000 C CNN
+F 1 "12 V" H 5908 6131 60  0000 C CNN
 F 2 "MRDT_Connectors:Anderson_2_Horizontal_Side_by_Side" H 5550 5300 60  0001 C CNN
 F 3 "" H 5550 5300 60  0001 C CNN
@@
 AR Path="/5F9A17AD" Ref="Conn4"  Part="1"
 F 0 "Conn4" H 6050 6650 60  0000 R CNN
-F 1 "AndersonPP" H 6200 6550 60  0000 R CNN
+F 1 "12 V" H 6200 6550 60  0000 R CNN
 F 2 "MRDT_Connectors:Anderson_2_Horizontal_Side_by_Side" H 5550 5750 60  0001 C CNN
 F 3 "" H 5550 5750 60  0001 C CNN
@@
 AR Path="/5F9A17BB" Ref="Conn8"  Part="4"
 F 0 "Conn8" H 7058 6237 60  0000 C CNN
-F 1 "AndersonPP" H 7058 6131 60  0000 C CNN
+F 1 "Vaccum" H 7058 6131 60  0000 C CNN
 F 2 "MRDT_Connectors:Anderson_2_Horizontal_Side_by_Side" H 6700 5300 60  0001 C CNN
 F 3 "" H 6700 5300 60  0001 C CNN
@@
 AR Path="/5F9A17C1" Ref="Conn8"  Part="1"
 F 0 "Conn8" H 7200 6650 60  0000 R CNN
-F 1 "AndersonPP" H 7350 6550 60  0000 R CNN
+F 1 "Vaccum" H 7350 6550 60  0000 R CNN
 F 2 "MRDT_Connectors:Anderson_2_Horizontal_Side_by_Side" H 6700 5750 60  0001 C CNN
 F 3 "" H 6700 5750 60  0001 C CNN
@@
 AR Path="/5F9A17CF" Ref="Conn10"  Part="4"
 F 0 "Conn10" H 8208 6237 60  0000 C CNN
-F 1 "AndersonPP" H 8208 6131 60  0000 C CNN
+F 1 "Driveboard" H 8208 6131 60  0000 C CNN
 F 2 "MRDT_Connectors:Anderson_2_Horizontal_Side_by_Side" H 7850 5300 60  0001 C CNN
 F 3 "" H 7850 5300 60  0001 C CNN
@@
 AR Path="/5F9A17D5" Ref="Conn10"  Part="1"
 F 0 "Conn10" H 8350 6650 60  0000 R CNN
-F 1 "AndersonPP" H 8500 6550 60  0000 R CNN
+F 1 "Driveboard" H 8500 6550 60  0000 R CNN
 F 2 "MRDT_Connectors:Anderson_2_Horizontal_Side_by_Side" H 7850 5750 60  0001 C CNN
 F 3 "" H 7850 5750 60  0001 C CNN
@@
 AR Path="/5F888F54" Ref="Conn12"  Part="4"
 F 0 "Conn12" H 9358 5087 60  0000 C CNN
-F 1 "AndersonPP" H 9358 4981 60  0000 C CNN
+F 1 "Spare" H 9358 4981 60  0000 C CNN
 F 2 "MRDT_Connectors:Anderson_2_Horizontal_Side_by_Side" H 9000 4150 60  0001 C CNN
 F 3 "" H 9000 4150 60  0001 C CNN
@@
 AR Path="/5F888F5A" Ref="Conn12"  Part="1"
 F 0 "Conn12" H 9500 5500 60  0000 R CNN
-F 1 "AndersonPP" H 9650 5400 60  0000 R CNN
+F 1 "Spare" H 9650 5400 60  0000 R CNN
 F 2 "MRDT_Connectors:Anderson_2_Horizontal_Side_by_Side" H 9000 4600 60  0001 C CNN
 F 3 "" H 9000 4600 60  0001 C CNN
@@
 AR Path="/5F8BC44B" Ref="Conn11"  Part="4"
 F 0 "Conn11" H 9333 6237 60  0000 C CNN
-F 1 "AndersonPP" H 9333 6131 60  0000 C CNN
+F 1 "Auxiliary" H 9333 6131 60  0000 C CNN
 F 2 "MRDT_Connectors:Anderson_2_Horizontal_Side_by_Side" H 8975 5300 60  0001 C CNN
 F 3 "" H 8975 5300 60  0001 C CNN
@@
 AR Path="/5F8BC451" Ref="Conn11"  Part="1"
 F 0 "Conn11" H 9475 6650 60  0000 R CNN
-F 1 "AndersonPP" H 9625 6550 60  0000 R CNN
+F 1 "Auxiliary" H 9625 6550 60  0000 R CNN
 F 2 "MRDT_Connectors:Anderson_2_Horizontal_Side_by_Side" H 8975 5750 60  0001 C CNN
 F 3 "" H 8975 5750 60  0001 C CNN
