File: Hardware/PackVoltage_2021_Rev1/_autosave-Buck.sch (KiCad schematic (older format))
At the start: 24 parts, among them J12V1 Test_Point, J3V1 Test_Point, J5V1 Test_Point, U11 LM2576S-12/NOPB, U12 LM2576SX-5.0/NOPB, U13 LM2576SX-3.3/NOPB

Commit message: started editing layout
Parts:
- D10, D8, D9: footprint Diode_THT:D_DO-201AD_P5.08mm_Vertical_AnodeUp -> Diode_THT:D_DO-201AD_P15.24mm_Horizontal
Changed lines of the file:
@@
 F 0 "D9" V 2429 3180 50  0000 L CNN
 F 1 "1N5822" V 2520 3180 50  0000 L CNN
-F 2 "Diode_THT:D_DO-201AD_P5.08mm_Vertical_AnodeUp" H 2475 3100 50  0001 C CNN
+F 2 "Diode_THT:D_DO-201AD_P15.24mm_Horizontal" H 2475 3100 50  0001 C CNN
 F 3 "~" H 2475 3100 50  0001 C CNN
 	1    2475 3100
@@
 F 0 "D10" V 2454 4880 50  0000 L CNN
 F 1 "1N5822" V 2545 4880 50  0000 L CNN
-F 2 "Diode_THT:D_DO-201AD_P5.08mm_Vertical_AnodeUp" H 2500 4800 50  0001 C CNN
+F 2 "Diode_THT:D_DO-201AD_P15.24mm_Horizontal" H 2500 4800 50  0001 C CNN
 F 3 "~" H 2500 4800 50  0001 C CNN
 	1    2500 4800
@@
 F 0 "D8" V 2429 1730 50  0000 L CNN
 F 1 "1N5822" V 2520 1730 50  0000 L CNN
-F 2 "Diode_THT:D_DO-201AD_P5.08mm_Vertical_AnodeUp" H 2475 1650 50  0001 C CNN
+F 2 "Diode_THT:D_DO-201AD_P15.24mm_Horizontal" H 2475 1650 50  0001 C CNN
 F 3 "~" H 2475 1650 50  0001 C CNN
 	1    2475 1650
