File: Hardware/PackVoltage_2021_Rev1/_autosave-PackVoltage_2021_Rev1.kicad_pcb (KiCad board)
At the start: 2 copper layers, 149 parts, among them J12V1 Test_Point, J3V1 Test_Point, J5V1 Test_Point, Q1 Q_NMOS_DGS, Q10 Q_NMOS_DGS, Q2 Q_NMOS_DGS, Q3 Q_NMOS_DGS, Q4 Q_NMOS_DGS, Q5 Q_NMOS_DGS, Q6 Q_NMOS_DGS, Q7 Q_NMOS_DGS, Q8 Q_NMOS_DGS, Q9 Q_NMOS_DGS, U1 LT1910, U10 INA281, U11 LM2576S-12/NOPB, U12 OKI-78SR-3.3_1.5-W36-C, U13 OKI-78SR-5_1.5-W36-C, U14 LT1910, U15 LT1910, U16 LT1910, U17 INA281, U18 INA281, U19 INA281, U2 LT1910, U20 LT1910, U21 LT1910, U22 INA281, U23 INA281, U24 TM4C129E_Launchpad, U3 LT1910, U4 INA281, U5 INA281, U6 INA281, U7 LT1910, U8 LT1910, U9 INA281

Commit message: rearranged components on layout
Parts:
- R22: moved to B.Cu
- moved R22 348.4 mm to (61.2, 82.5)
- moved R19 261.3 mm to (68.9, 88.0), turned to 90 degrees
- moved R17 212.3 mm to (94.2, 131.1), turned to 90 degrees
- moved C18 99.4 mm to (102.7, 115.6), turned to 180 degrees
- moved D8 78.6 mm to (114.7, 108.1)
- moved L1 68.3 mm to (107.2, 107.2)
- moved C15 62.3 mm to (126.0, 113.2), turned to 180 degrees
- moved R18 56.2 mm to (157.1, 131.0), turned to 90 degrees
- moved R16 47.5 mm to (125.6, 127.3)
- moved J12V1 42.9 mm to (106.7, 124.7)
- moved C21 26.8 mm to (299.8, 160.6)
- moved F6 14.7 mm to (78.1, 82.2)
- moved D2 10.5 mm to (124.1, 178.1)
