File: Hardware/PackVoltage_2021_Rev1/Other_Busses.sch (KiCad schematic (older format))
At the start: 50 parts, among them Q10 Q_NMOS_DGS, Q6 Q_NMOS_DGS, Q7 Q_NMOS_DGS, Q8 Q_NMOS_DGS, Q9 Q_NMOS_DGS, U14 LT1910, U15 LT1910, U16 LT1910, U17 INA281, U18 INA281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

Commit message: updated footprints
Parts:
- C21, C22, C23, C24, C25, C26, C27, C28, C29, C30: footprint (none) -> Capacitor_SMD:C_0603_1608Metric_Pad1.05x0.95mm_HandSolder
- D14, D15, D16, D17, D18: footprint (none) -> Diode_SMD:D_0201_0603Metric
- F10, F6, F7, F8, F9: footprint (none) -> MRDT_Passives:ATC_Fuse_Block
- R19, R20, R21, R25, R26, R27, R28, R29, R32, R33: footprint (none) -> Resistor_SMD:R_0603_1608Metric_Pad1.05x0.95mm_HandSolder
- U14, U15, U16, U20, U21: footprint (none) -> Package_SO:SOIC-8-N7_3.9x4.9mm_P1.27mm; symbol MRDT_ICs:LT1910 -> PackVoltage_2021_Rev1-rescue:LT1910-MRDT_ICs
- U17, U18, U19, U22, U23: symbol MRDT_ICs:INA281 -> PackVoltage_2021_Rev1-rescue:INA281-MRDT_ICs
Changed lines of the file:
@@
 F 0 "R21" V 850 1500 50  0000 C CNN
 F 1 "5.1k" V 950 1500 50  0000 C CNN
-F 2 "" V 880 1500 50  0001 C CNN
+F 2 "Resistor_SMD:R_0603_1608Metric_Pad1.05x0.95mm_HandSolder" V 880 1500 50  0001 C CNN
 F 3 "~" H 950 1500 50  0001 C CNN
 	1    950  1500
@@
 F 0 "C23" H 1342 2046 50  0000 L CNN
 F 1 "0.1uF" H 1342 1955 50  0000 L CNN
-F 2 "" H 1250 2000 50  0001 C CNN
+F 2 "Capacitor_SMD:C_0603_1608Metric_Pad1.05x0.95mm_HandSolder" H 1250 2000 50  0001 C CNN
 F 3 "~" H 1250 2000 50  0001 C CNN
 	1    1250 2000
@@
 F 0 "C26" H 2692 2046 50  0000 L CNN
 F 1 "10uF" H 2692 1955 50  0000 L CNN
-F 2 "" H 2600 2000 50  0001 C CNN
+F 2 "Capacitor_SMD:C_0603_1608Metric_Pad1.05x0.95mm_HandSolder" H 2600 2000 50  0001 C CNN
 F 3 "~" H 2600 2000 50  0001 C CNN
 	1    2600 2000
@@
 F 0 "D16" H 3500 2400 50  0000 C CNN
 F 1 "LED" H 3500 2500 50  0000 C CNN
-F 2 "" H 3500 2300 50  0001 C CNN
+F 2 "Diode_SMD:D_0201_0603Metric" H 3500 2300 50  0001 C CNN
 F 3 "~" H 3500 2300 50  0001 C CNN
 	1    3500 2300
@@
 F 0 "R27" V 3850 2250 50  0000 L CNN
 F 1 "3300" V 3950 2200 50  0000 L CNN
-F 2 "" V 3880 2300 50  0001 C CNN
+F 2 "Resistor_SMD:R_0603_1608Metric_Pad1.05x0.95mm_HandSolder" V 3880 2300 50  0001 C CNN
 F 3 "~" H 3950 2300 50  0001 C CNN
 	1    3950 2300
@@
 PV
 $Comp
-L MRDT_ICs:LT1910 U?
+L PackVoltage_2021_Rev1-rescue:LT1910-MRDT_ICs U?
 U 1 1 5F8E1128
 P 1450 1900
@@
 F 0 "U16" H 1825 2587 60  0000 C CNN
 F 1 "LT1910" H 1825 2481 60  0000 C CNN
-F 2 "" H 1450 1900 60  0001 C CNN
+F 2 "Package_SO:SOIC-8-N7_3.9x4.9mm_P1.27mm" H 1450 1900 60  0001 C CNN
 F 3 "" H 1450 1900 60  0001 C CNN
 	1    1450 1900
@@
 F 0 "F6" V 2350 3200 50  0000 L CNN
 F 1 "20" V 2450 3200 50  0000 L CNN
-F 2 "" V 2380 3250 50  0001 C CNN
+F 2 "MRDT_Passives:ATC_Fuse_Block" V 2380 3250 50  0001 C CNN
 F 3 "~" H 2450 3250 50  0001 C CNN
 	1    2450 3250
@@
 F 0 "R19" V 800 3500 50  0000 C CNN
 F 1 "5.1k" V 900 3500 50  0000 C CNN
-F 2 "" V 830 3500 50  0001 C CNN
+F 2 "Resistor_SMD:R_0603_1608Metric_Pad1.05x0.95mm_HandSolder" V 830 3500 50  0001 C CNN
 F 3 "~" H 900 3500 50  0001 C CNN
 	1    900  3500
@@
 F 0 "C21" H 1292 4046 50  0000 L CNN
 F 1 "0.1uF" H 1292 3955 50  0000 L CNN
-F 2 "" H 1200 4000 50  0001 C CNN
+F 2 "Capacitor_SMD:C_0603_1608Metric_Pad1.05x0.95mm_HandSolder" H 1200 4000 50  0001 C CNN
 F 3 "~" H 1200 4000 50  0001 C CNN
 	1    1200 4000
@@
 F 0 "C24" H 2642 4046 50  0000 L CNN
 F 1 "10uF" H 2642 3955 50  0000 L CNN
-F 2 "" H 2550 4000 50  0001 C CNN
+F 2 "Capacitor_SMD:C_0603_1608Metric_Pad1.05x0.95mm_HandSolder" H 2550 4000 50  0001 C CNN
 F 3 "~" H 2550 4000 50  0001 C CNN
 	1    2550 4000
@@
 F 0 "D14" H 3450 4400 50  0000 C CNN
 F 1 "LED" H 3450 4500 50  0000 C CNN
-F 2 "" H 3450 4300 50  0001 C CNN
+F 2 "Diode_SMD:D_0201_0603Metric" H 3450 4300 50  0001 C CNN
 F 3 "~" H 3450 4300 50  0001 C CNN
 	1    3450 4300
@@
 12V
 $Comp
-L MRDT_ICs:INA281 U?
+L PackVoltage_2021_Rev1-rescue:INA281-MRDT_ICs U?
 U 1 1 5F9AF79E
 P 4050 3550
@@
 $EndComp
 $Comp
-L MRDT_ICs:LT1910 U?
+L PackVoltage_2021_Rev1-rescue:LT1910-MRDT_ICs U?
 U 1 1 5F9AF79F
 P 1400 3900
@@
 F 0 "U14" H 1775 4587 60  0000 C CNN
 F 1 "LT1910" H 1775 4481 60  0000 C CNN
-F 2 "" H 1400 3900 60  0001 C CNN
+F 2 "Package_SO:SOIC-8-N7_3.9x4.9mm_P1.27mm" H 1400 3900 60  0001 C CNN
 F 3 "" H 1400 3900 60  0001 C CNN
 	1    1400 3900
@@
 F 0 "F7" V 2350 5400 50  0000 L CNN
 F 1 "10" V 2450 5400 50  0000 L CNN
-F 2 "" V 2380 5450 50  0001 C CNN
+F 2 "MRDT_Passives:ATC_Fuse_Block" V 2380 5450 50  0001 C CNN
 F 3 "~" H 2450 5450 50  0001 C CNN
 	1    2450 5450
@@
 F 0 "R20" V 800 5700 50  0000 C CNN
 F 1 "5.1k" V 900 5700 50  0000 C CNN
-F 2 "" V 830 5700 50  0001 C CNN
+F 2 "Resistor_SMD:R_0603_1608Metric_Pad1.05x0.95mm_HandSolder" V 830 5700 50  0001 C CNN
 F 3 "~" H 900 5700 50  0001 C CNN
 	1    900  5700
@@
 F 0 "C22" H 1292 6246 50  0000 L CNN
 F 1 "0.1uF" H 1292 6155 50  0000 L CNN
-F 2 "" H 1200 6200 50  0001 C CNN
+F 2 "Capacitor_SMD:C_0603_1608Metric_Pad1.05x0.95mm_HandSolder" H 1200 6200 50  0001 C CNN
 F 3 "~" H 1200 6200 50  0001 C CNN
 	1    1200 6200
@@
 F 0 "C25" H 2642 6246 50  0000 L CNN
 F 1 "10uF" H 2642 6155 50  0000 L CNN
-F 2 "" H 2550 6200 50  0001 C CNN
+F 2 "Capacitor_SMD:C_0603_1608Metric_Pad1.05x0.95mm_HandSolder" H 2550 6200 50  0001 C CNN
 F 3 "~" H 2550 6200 50  0001 C CNN
 	1    2550 6200
@@
 F 0 "D15" H 3450 6600 50  0000 C CNN
 F 1 "LED" H 3450 6700 50  0000 C CNN
-F 2 "" H 3450 6500 50  0001 C CNN
+F 2 "Diode_SMD:D_0201_0603Metric" H 3450 6500 50  0001 C CNN
 F 3 "~" H 3450 6500 50  0001 C CNN
 	1    3450 6500
@@
 PV
 $Comp
-L MRDT_ICs:INA281 U?
+L PackVoltage_2021_Rev1-rescue:INA281-MRDT_ICs U?
 U 1 1 5F9AF7AB
 P 4050 5750
@@
 $EndComp
 $Comp
-L MRDT_ICs:LT1910 U?
+L PackVoltage_2021_Rev1-rescue:LT1910-MRDT_ICs U?
 U 1 1 5F8A5A3C
 P 1400 6100
@@
 F 0 "U15" H 1775 6787 60  0000 C CNN
 F 1 "LT1910" H 1775 6681 60  0000 C CNN
-F 2 "" H 1400 6100 60  0001 C CNN
+F 2 "Package_SO:SOIC-8-N7_3.9x4.9mm_P1.27mm" H 1400 6100 60  0001 C CNN
 F 3 "" H 1400 6100 60  0001 C CNN
 	1    1400 6100
@@
 F 0 "F9" V 7750 1250 50  0000 L CNN
 F 1 "20" V 7850 1250 50  0000 L CNN
-F 2 "" V 7780 1300 50  0001 C CNN
+F 2 "MRDT_Passives:ATC_Fuse_Block" V 7780 1300 50  0001 C CNN
 F 3 "~" H 7850 1300 50  0001 C CNN
 	1    7850 1300
@@
 F 0 "R28" V 6200 1550 50  0000 C CNN
 F 1 "5.1k" V 6300 1550 50  0000 C CNN
-F 2 "" V 6230 1550 50  0001 C CNN
+F 2 "Resistor_SMD:R_0603_1608Metric_Pad1.05x0.95mm_HandSolder" V 6230 1550 50  0001 C CNN
 F 3 "~" H 6300 1550 50  0001 C CNN
 	1    6300 1550
@@
 F 0 "C27" H 6692 2096 50  0000 L CNN
 F 1 "0.1uF" H 6692 2005 50  0000 L CNN
-F 2 "" H 6600 2050 50  0001 C CNN
+F 2 "Capacitor_SMD:C_0603_1608Metric_Pad1.05x0.95mm_HandSolder" H 6600 2050 50  0001 C CNN
 F 3 "~" H 6600 2050 50  0001 C CNN
 	1    6600 2050
@@
 F 0 "C29" H 8042 2096 50  0000 L CNN
 F 1 "10uF" H 8042 2005 50  0000 L CNN
-F 2 "" H 7950 2050 50  0001 C CNN
+F 2 "Capacitor_SMD:C_0603_1608Metric_Pad1.05x0.95mm_HandSolder" H 7950 2050 50  0001 C CNN
 F 3 "~" H 7950 2050 50  0001 C CNN
 	1    7950 2050
@@
 F 0 "D17" H 8850 2450 50  0000 C CNN
 F 1 "LED" H 8850 2550 50  0000 C CNN
-F 2 "" H 8850 2350 50  0001 C CNN
+F 2 "Diode_SMD:D_0201_0603Metric" H 8850 2350 50  0001 C CNN
 F 3 "~" H 8850 2350 50  0001 C CNN
 	1    8850 2350
@@
 F 0 "R32" V 9200 2300 50  0000 L CNN
 F 1 "3300" V 9300 2250 50  0000 L CNN
-F 2 "" V 9230 2350 50  0001 C CNN
+F 2 "Resistor_SMD:R_0603_1608Metric_Pad1.05x0.95mm_HandSolder" V 9230 2350 50  0001 C CNN
 F 3 "~" H 9300 2350 50  0001 C CNN
 	1    9300 2350
@@
 PV
 $Comp
-L MRDT_ICs:INA281 U?
+L PackVoltage_2021_Rev1-rescue:INA281-MRDT_ICs U?
 U 1 1 5F9AF7B8
 P 9450 1600
@@
 $EndComp
 $Comp
-L MRDT_ICs:LT1910 U?
+L PackVoltage_2021_Rev1-rescue:LT1910-MRDT_ICs U?
 U 1 1 5F9AF7B9
 P 6800 1950
@@
 F 0 "U20" H 7175 2637 60  0000 C CNN
 F 1 "LT1910" H 7175 2531 60  0000 C CNN
-F 2 "" H 6800 1950 60  0001 C CNN
+F 2 "Package_SO:SOIC-8-N7_3.9x4.9mm_P1.27mm" H 6800 1950 60  0001 C CNN
 F 3 "" H 6800 1950 60  0001 C CNN
 	1    6800 1950
@@
 F 0 "F8" V 2400 1200 50  0000 L CNN
 F 1 "15" V 2500 1200 50  0000 L CNN
-F 2 "" V 2430 1250 50  0001 C CNN
+F 2 "MRDT_Passives:ATC_Fuse_Block" V 2430 1250 50  0001 C CNN
 F 3 "~" H 2500 1250 50  0001 C CNN
 	1    2500 1250
@@
 F 0 "F10" V 7750 3300 50  0000 L CNN
 F 1 "20" V 7850 3300 50  0000 L CNN
-F 2 "" V 7780 3350 50  0001 C CNN
+F 2 "MRDT_Passives:ATC_Fuse_Block" V 7780 3350 50  0001 C CNN
 F 3 "~" H 7850 3350 50  0001 C CNN
 	1    7850 3350
@@
 F 0 "R29" V 6200 3600 50  0000 C CNN
 F 1 "5.1k" V 6300 3600 50  0000 C CNN
-F 2 "" V 6230 3600 50  0001 C CNN
+F 2 "Resistor_SMD:R_0603_1608Metric_Pad1.05x0.95mm_HandSolder" V 6230 3600 50  0001 C CNN
 F 3 "~" H 6300 3600 50  0001 C CNN
 	1    6300 3600
@@
 F 0 "C28" H 6692 4146 50  0000 L CNN
 F 1 "0.1uF" H 6692 4055 50  0000 L CNN
-F 2 "" H 6600 4100 50  0001 C CNN
+F 2 "Capacitor_SMD:C_0603_1608Metric_Pad1.05x0.95mm_HandSolder" H 6600 4100 50  0001 C CNN
 F 3 "~" H 6600 4100 50  0001 C CNN
 	1    6600 4100
@@
 F 0 "C30" H 8042 4146 50  0000 L CNN
 F 1 "10uF" H 8042 4055 50  0000 L CNN
-F 2 "" H 7950 4100 50  0001 C CNN
+F 2 "Capacitor_SMD:C_0603_1608Metric_Pad1.05x0.95mm_HandSolder" H 7950 4100 50  0001 C CNN
 F 3 "~" H 7950 4100 50  0001 C CNN
 	1    7950 4100
@@
 F 0 "D18" H 8850 4500 50  0000 C CNN
 F 1 "LED" H 8850 4600 50  0000 C CNN
-F 2 "" H 8850 4400 50  0001 C CNN
+F 2 "Diode_SMD:D_0201_0603Metric" H 8850 4400 50  0001 C CNN
 F 3 "~" H 8850 4400 50  0001 C CNN
 	1    8850 4400
@@
 F 0 "R33" V 9200 4350 50  0000 L CNN
 F 1 "3300" V 9300 4300 50  0000 L CNN
-F 2 "" V 9230 4400 50  0001 C CNN
+F 2 "Resistor_SMD:R_0603_1608Metric_Pad1.05x0.95mm_HandSolder" V 9230 4400 50  0001 C CNN
 F 3 "~" H 9300 4400 50  0001 C CNN
 	1    9300 4400
@@
 PV
 $Comp
-L MRDT_ICs:INA281 U?
+L PackVoltage_2021_Rev1-rescue:INA281-MRDT_ICs U?
 U 1 1 5F8E4246
 P 9450 3650
@@
 $EndComp
 $Comp
-L MRDT_ICs:LT1910 U?
+L PackVoltage_2021_Rev1-rescue:LT1910-MRDT_ICs U?
 U 1 1 5F8E424C
 P 6800 4000
@@
 F 0 "U21" H 7175 4687 60  0000 C CNN
 F 1 "LT1910" H 7175 4581 60  0000 C CNN
-F 2 "" H 6800 4000 60  0001 C CNN
+F 2 "Package_SO:SOIC-8-N7_3.9x4.9mm_P1.27mm" H 6800 4000 60  0001 C CNN
 F 3 "" H 6800 4000 60  0001 C CNN
 	1    6800 4000
@@
 	3550 1450 3900 1450
 $Comp
-L MRDT_ICs:INA281 U?
+L PackVoltage_2021_Rev1-rescue:INA281-MRDT_ICs U?
 U 1 1 5F9AF7BB
 P 4100 1550
@@
 F 0 "R26" V 3800 6450 50  0000 L CNN
 F 1 "3300" V 3900 6400 50  0000 L CNN
-F 2 "" V 3830 6500 50  0001 C CNN
+F 2 "Resistor_SMD:R_0603_1608Metric_Pad1.05x0.95mm_HandSolder" V 3830 6500 50  0001 C CNN
 F 3 "~" H 3900 6500 50  0001 C CNN
 	1    3900 6500
@@
 F 0 "R25" V 3800 4250 50  0000 L CNN
 F 1 "1200" V 3900 4200 50  0000 L CNN
-F 2 "" V 3830 4300 50  0001 C CNN
+F 2 "Resistor_SMD:R_0603_1608Metric_Pad1.05x0.95mm_HandSolder" V 3830 4300 50  0001 C CNN
 F 3 "~" H 3900 4300 50  0001 C CNN
 	1    3900 4300

Commit message: Added Footprints (Still missing MOSFET)
Parts:
- R22, R23, R24, R30, R31: footprint (none) -> Package_TO_SOT_SMD:TO-263-2
- U17, U18, U19, U22, U23: footprint (none) -> Package_TO_SOT_SMD:SOT-23-5_HandSoldering
Changed lines of the file:
@@
 F 0 "R24" V 3450 1650 50  0000 L CNN
 F 1 "0.05" V 3550 1600 50  0000 L CNN
-F 2 "" V 3480 1700 50  0001 C CNN
+F 2 "Package_TO_SOT_SMD:TO-263-2" V 3480 1700 50  0001 C CNN
 F 3 "https://riedon.com/media/pdf/PFS35.pdf" H 3550 1700 50  0001 C CNN
 	1    3550 1700
@@
 F 0 "R22" V 3400 3650 50  0000 L CNN
 F 1 "0.05" V 3500 3600 50  0000 L CNN
-F 2 "" V 3430 3700 50  0001 C CNN
+F 2 "Package_TO_SOT_SMD:TO-263-2" V 3430 3700 50  0001 C CNN
 F 3 "https://riedon.com/media/pdf/PFS35.pdf" H 3500 3700 50  0001 C CNN
 	1    3500 3700
@@
 F 0 "U17" H 4150 3850 50  0000 L CNN
 F 1 "INA281" H 4100 3750 50  0000 L CNN
-F 2 "" H 4300 3750 50  0001 C CNN
+F 2 "Package_TO_SOT_SMD:SOT-23-5_HandSoldering" H 4300 3750 50  0001 C CNN
 F 3 "" H 4300 3750 50  0001 C CNN
 	1    4050 3550
@@
 F 0 "R23" V 3400 5850 50  0000 L CNN
 F 1 "0.05" V 3500 5800 50  0000 L CNN
-F 2 "" V 3430 5900 50  0001 C CNN
+F 2 "Package_TO_SOT_SMD:TO-263-2" V 3430 5900 50  0001 C CNN
 F 3 "https://riedon.com/media/pdf/PFS35.pdf" H 3500 5900 50  0001 C CNN
 	1    3500 5900
@@
 F 0 "U18" H 4150 6050 50  0000 L CNN
 F 1 "INA281" H 4100 5950 50  0000 L CNN
-F 2 "" H 4300 5950 50  0001 C CNN
+F 2 "Package_TO_SOT_SMD:SOT-23-5_HandSoldering" H 4300 5950 50  0001 C CNN
 F 3 "" H 4300 5950 50  0001 C CNN
 	1    4050 5750
@@
 F 0 "R30" V 8800 1700 50  0000 L CNN
 F 1 "0.05" V 8900 1650 50  0000 L CNN
-F 2 "" V 8830 1750 50  0001 C CNN
+F 2 "Package_TO_SOT_SMD:TO-263-2" V 8830 1750 50  0001 C CNN
 F 3 "https://riedon.com/media/pdf/PFS35.pdf" H 8900 1750 50  0001 C CNN
 	1    8900 1750
@@
 F 0 "U22" H 9550 1900 50  0000 L CNN
 F 1 "INA281" H 9500 1800 50  0000 L CNN
-F 2 "" H 9700 1800 50  0001 C CNN
+F 2 "Package_TO_SOT_SMD:SOT-23-5_HandSoldering" H 9700 1800 50  0001 C CNN
 F 3 "" H 9700 1800 50  0001 C CNN
 	1    9450 1600
@@
 F 0 "R31" V 8800 3750 50  0000 L CNN
 F 1 "0.05" V 8900 3700 50  0000 L CNN
-F 2 "" V 8830 3800 50  0001 C CNN
+F 2 "Package_TO_SOT_SMD:TO-263-2" V 8830 3800 50  0001 C CNN
 F 3 "https://riedon.com/media/pdf/PFS35.pdf" H 8900 3800 50  0001 C CNN
 	1    8900 3800
@@
 F 0 "U23" H 9550 3950 50  0000 L CNN
 F 1 "INA281" H 9500 3850 50  0000 L CNN
-F 2 "" H 9700 3850 50  0001 C CNN
+F 2 "Package_TO_SOT_SMD:SOT-23-5_HandSoldering" H 9700 3850 50  0001 C CNN
 F 3 "" H 9700 3850 50  0001 C CNN
 	1    9450 3650
@@
 F 0 "U19" H 4200 1850 50  0000 L CNN
 F 1 "INA281" H 4150 1750 50  0000 L CNN
-F 2 "" H 4350 1750 50  0001 C CNN
+F 2 "Package_TO_SOT_SMD:SOT-23-5_HandSoldering" H 4350 1750 50  0001 C CNN
 F 3 "" H 4350 1750 50  0001 C CNN
 	1    4100 1550

Commit message: added DriveCTL to MOLEX and TIVA, changed andersons to actuation
Parts:
- Q10, Q6, Q7, Q8, Q9: footprint (none) -> Package_TO_SOT_SMD:LFPAK56
Changed lines of the file:
@@
 F 0 "Q8" H 3000 1450 50  0000 C CNN
 F 1 "Q_NMOS_DGS" H 3300 1350 50  0000 C CNN
-F 2 "" H 3200 1750 50  0001 C CNN
+F 2 "Package_TO_SOT_SMD:LFPAK56" H 3200 1750 50  0001 C CNN
 F 3 "~" H 3000 1650 50  0001 C CNN
 	1    3000 1650
@@
 F 0 "Q6" H 2950 3450 50  0000 C CNN
 F 1 "Q_NMOS_DGS" H 3250 3350 50  0000 C CNN
-F 2 "" H 3150 3750 50  0001 C CNN
+F 2 "Package_TO_SOT_SMD:LFPAK56" H 3150 3750 50  0001 C CNN
 F 3 "~" H 2950 3650 50  0001 C CNN
 	1    2950 3650
@@
 F 0 "Q7" H 2950 5650 50  0000 C CNN
 F 1 "Q_NMOS_DGS" H 3250 5550 50  0000 C CNN
-F 2 "" H 3150 5950 50  0001 C CNN
+F 2 "Package_TO_SOT_SMD:LFPAK56" H 3150 5950 50  0001 C CNN
 F 3 "~" H 2950 5850 50  0001 C CNN
 	1    2950 5850
@@
 F 0 "Q9" H 8350 1500 50  0000 C CNN
 F 1 "Q_NMOS_DGS" H 8650 1400 50  0000 C CNN
-F 2 "" H 8550 1800 50  0001 C CNN
+F 2 "Package_TO_SOT_SMD:LFPAK56" H 8550 1800 50  0001 C CNN
 F 3 "~" H 8350 1700 50  0001 C CNN
 	1    8350 1700
@@
 F 0 "Q10" H 8350 3550 50  0000 C CNN
 F 1 "Q_NMOS_DGS" H 8650 3450 50  0000 C CNN
-F 2 "" H 8550 3850 50  0001 C CNN
+F 2 "Package_TO_SOT_SMD:LFPAK56" H 8550 3850 50  0001 C CNN
 F 3 "~" H 8350 3750 50  0001 C CNN
 	1    8350 3750

Commit message: Layout
Parts:
- D14, D15, D16, D17, D18: footprint Diode_SMD:D_0201_0603Metric -> LED_SMD:LED_0603_1608Metric_Pad1.05x0.95mm_HandSolder
- Q10, Q6, Q7, Q8, Q9: footprint Package_TO_SOT_SMD:LFPAK56 -> Custom:LFPAK56_MOSFET
- R22, R23, R24, R30, R31: footprint Package_TO_SOT_SMD:TO-263-2 -> Package_TO_SOT_SMD:TO-263-2_TabPin1
Changed lines of the file:
@@
 F 0 "Q8" H 3000 1450 50  0000 C CNN
 F 1 "Q_NMOS_DGS" H 3300 1350 50  0000 C CNN
-F 2 "Package_TO_SOT_SMD:LFPAK56" H 3200 1750 50  0001 C CNN
+F 2 "Custom:LFPAK56_MOSFET" H 3200 1750 50  0001 C CNN
 F 3 "~" H 3000 1650 50  0001 C CNN
 	1    3000 1650
@@
 F 0 "R24" V 3450 1650 50  0000 L CNN
 F 1 "0.05" V 3550 1600 50  0000 L CNN
-F 2 "Package_TO_SOT_SMD:TO-263-2" V 3480 1700 50  0001 C CNN
+F 2 "Package_TO_SOT_SMD:TO-263-2_TabPin1" V 3480 1700 50  0001 C CNN
 F 3 "https://riedon.com/media/pdf/PFS35.pdf" H 3550 1700 50  0001 C CNN
 	1    3550 1700
@@
 F 0 "D16" H 3500 2400 50  0000 C CNN
 F 1 "LED" H 3500 2500 50  0000 C CNN
-F 2 "Diode_SMD:D_0201_0603Metric" H 3500 2300 50  0001 C CNN
+F 2 "LED_SMD:LED_0603_1608Metric_Pad1.05x0.95mm_HandSolder" H 3500 2300 50  0001 C CNN
 F 3 "~" H 3500 2300 50  0001 C CNN
 	1    3500 2300
@@
 F 0 "Q6" H 2950 3450 50  0000 C CNN
 F 1 "Q_NMOS_DGS" H 3250 3350 50  0000 C CNN
-F 2 "Package_TO_SOT_SMD:LFPAK56" H 3150 3750 50  0001 C CNN
+F 2 "Custom:LFPAK56_MOSFET" H 3150 3750 50  0001 C CNN
 F 3 "~" H 2950 3650 50  0001 C CNN
 	1    2950 3650
@@
 F 0 "R22" V 3400 3650 50  0000 L CNN
 F 1 "0.05" V 3500 3600 50  0000 L CNN
-F 2 "Package_TO_SOT_SMD:TO-263-2" V 3430 3700 50  0001 C CNN
+F 2 "Package_TO_SOT_SMD:TO-263-2_TabPin1" V 3430 3700 50  0001 C CNN
 F 3 "https://riedon.com/media/pdf/PFS35.pdf" H 3500 3700 50  0001 C CNN
 	1    3500 3700
@@
 F 0 "D14" H 3450 4400 50  0000 C CNN
 F 1 "LED" H 3450 4500 50  0000 C CNN
-F 2 "Diode_SMD:D_0201_0603Metric" H 3450 4300 50  0001 C CNN
+F 2 "LED_SMD:LED_0603_1608Metric_Pad1.05x0.95mm_HandSolder" H 3450 4300 50  0001 C CNN
 F 3 "~" H 3450 4300 50  0001 C CNN
 	1    3450 4300
@@
 F 0 "Q7" H 2950 5650 50  0000 C CNN
 F 1 "Q_NMOS_DGS" H 3250 5550 50  0000 C CNN
-F 2 "Package_TO_SOT_SMD:LFPAK56" H 3150 5950 50  0001 C CNN
+F 2 "Custom:LFPAK56_MOSFET" H 3150 5950 50  0001 C CNN
 F 3 "~" H 2950 5850 50  0001 C CNN
 	1    2950 5850
@@
 F 0 "R23" V 3400 5850 50  0000 L CNN
 F 1 "0.05" V 3500 5800 50  0000 L CNN
-F 2 "Package_TO_SOT_SMD:TO-263-2" V 3430 5900 50  0001 C CNN
+F 2 "Package_TO_SOT_SMD:TO-263-2_TabPin1" V 3430 5900 50  0001 C CNN
 F 3 "https://riedon.com/media/pdf/PFS35.pdf" H 3500 5900 50  0001 C CNN
 	1    3500 5900
@@
 F 0 "D15" H 3450 6600 50  0000 C CNN
 F 1 "LED" H 3450 6700 50  0000 C CNN
-F 2 "Diode_SMD:D_0201_0603Metric" H 3450 6500 50  0001 C CNN
+F 2 "LED_SMD:LED_0603_1608Metric_Pad1.05x0.95mm_HandSolder" H 3450 6500 50  0001 C CNN
 F 3 "~" H 3450 6500 50  0001 C CNN
 	1    3450 6500
@@
 F 0 "Q9" H 8350 1500 50  0000 C CNN
 F 1 "Q_NMOS_DGS" H 8650 1400 50  0000 C CNN
-F 2 "Package_TO_SOT_SMD:LFPAK56" H 8550 1800 50  0001 C CNN
+F 2 "Custom:LFPAK56_MOSFET" H 8550 1800 50  0001 C CNN
 F 3 "~" H 8350 1700 50  0001 C CNN
 	1    8350 1700
@@
 F 0 "R30" V 8800 1700 50  0000 L CNN
 F 1 "0.05" V 8900 1650 50  0000 L CNN
-F 2 "Package_TO_SOT_SMD:TO-263-2" V 8830 1750 50  0001 C CNN
+F 2 "Package_TO_SOT_SMD:TO-263-2_TabPin1" V 8830 1750 50  0001 C CNN
 F 3 "https://riedon.com/media/pdf/PFS35.pdf" H 8900 1750 50  0001 C CNN
 	1    8900 1750
@@
 F 0 "D17" H 8850 2450 50  0000 C CNN
 F 1 "LED" H 8850 2550 50  0000 C CNN
-F 2 "Diode_SMD:D_0201_0603Metric" H 8850 2350 50  0001 C CNN
+F 2 "LED_SMD:LED_0603_1608Metric_Pad1.05x0.95mm_HandSolder" H 8850 2350 50  0001 C CNN
 F 3 "~" H 8850 2350 50  0001 C CNN
 	1    8850 2350
@@
 F 0 "Q10" H 8350 3550 50  0000 C CNN
 F 1 "Q_NMOS_DGS" H 8650 3450 50  0000 C CNN
-F 2 "Package_TO_SOT_SMD:LFPAK56" H 8550 3850 50  0001 C CNN
+F 2 "Custom:LFPAK56_MOSFET" H 8550 3850 50  0001 C CNN
 F 3 "~" H 8350 3750 50  0001 C CNN
 	1    8350 3750
@@
 F 0 "R31" V 8800 3750 50  0000 L CNN
 F 1 "0.05" V 8900 3700 50  0000 L CNN
-F 2 "Package_TO_SOT_SMD:TO-263-2" V 8830 3800 50  0001 C CNN
+F 2 "Package_TO_SOT_SMD:TO-263-2_TabPin1" V 8830 3800 50  0001 C CNN
 F 3 "https://riedon.com/media/pdf/PFS35.pdf" H 8900 3800 50  0001 C CNN
 	1    8900 3800
@@
 F 0 "D18" H 8850 4500 50  0000 C CNN
 F 1 "LED" H 8850 4600 50  0000 C CNN
-F 2 "Diode_SMD:D_0201_0603Metric" H 8850 4400 50  0001 C CNN
+F 2 "LED_SMD:LED_0603_1608Metric_Pad1.05x0.95mm_HandSolder" H 8850 4400 50  0001 C CNN
 F 3 "~" H 8850 4400 50  0001 C CNN
 	1    8850 4400
