File: Hardware/PackVoltage_2021/TIVA.sch (KiCad schematic (older format))
At the start: 1 part, among them U24 TM4C129E_Launchpad

Commit message: uhh more circuits
finished top circuits on layout, fixed two resistors in schematic
Connections:
- net Current_Sensor_M3: now also U24.PP0 (A2_3); no longer U24.PD2 (A2_2)
- net Driver_M3: now also U24.PD2 (A2_2); no longer U24.PP0 (A2_3)
Changed lines of the file:
@@
 Text HLabel 5350 1600 1    40   Input ~ 0
 Current_Sensor_M4
-Text HLabel 3450 1750 1    40   Input ~ 0
+Text HLabel 3350 1750 1    40   Input ~ 0
 Current_Sensor_M3
 Text HLabel 3150 1750 1    40   Input ~ 0
@@
 Text HLabel 5850 1600 1    40   Input ~ 0
 Current_Sensor_S1
-Text HLabel 3350 1750 1    40   Output ~ 0
+Text HLabel 3450 1750 1    40   Output ~ 0
 Driver_M3
 Text HLabel 3250 1750 1    40   Output ~ 0

Commit message: molexes
- changed 5 pin molex to 4 pin molex (removed buckCTL)
- started making traces from molexes to tiva
Connections:
- net Current_Sensor_M3: now also U24.PD2 (A2_2); no longer U24.PP0 (A2_3)
- net Driver_M3: now also U24.PP0 (A2_3); no longer U24.PD2 (A2_2)
- net BuckCTL: no longer names the net of U24.PG1 (C2_1)
- no-connect marks 39 -> 40
Changed lines of the file:
@@
 Comment4 ""
 $EndDescr
-Text HLabel 3750 4575 1    39   Output ~ 0
-BuckCTL
 $Comp
 L PackVoltage_2021_Rev1-rescue:TM4C129E_Launchpad-MRDT_Shields U24
@@
 	3650 4675 3650 4575
 Wire Wire Line
-	3750 4675 3750 4575
-Wire Wire Line
 	2950 2850 2950 2950
 Wire Wire Line
@@
 Text HLabel 5350 1600 1    40   Input ~ 0
 Current_Sensor_M4
-Text HLabel 3350 1750 1    40   Input ~ 0
+Text HLabel 3450 1750 1    40   Input ~ 0
 Current_Sensor_M3
 Text HLabel 3150 1750 1    40   Input ~ 0
@@
 Text HLabel 5850 1600 1    40   Input ~ 0
 Current_Sensor_S1
-Text HLabel 3450 1750 1    40   Output ~ 0
+Text HLabel 3350 1750 1    40   Output ~ 0
 Driver_M3
 Text HLabel 3250 1750 1    40   Output ~ 0
@@
 NoConn ~ 5500 4350
 NoConn ~ 5400 4350
+Wire Wire Line
+	3750 4675 3750 4575
+NoConn ~ 3750 4575
 $EndSCHEMATC

Commit message: netlist
Connections:
- net 3V3: no longer U24.+3V3 (A1_1)
- no-connect marks 40 -> 41
Other:
- moved on the sheet: U24A, U24B, U24C, U24D, U24E, U24F, U24G, U24H

Commit message: Revert "netlist"
This reverts commit 1af6446f6858f10edba603e339066d14f3a2f95b.
Connections:
- net 3V3: now also U24.+3V3 (A1_1)
- no-connect marks 41 -> 40
Other:
- moved on the sheet: U24A, U24B, U24C, U24D, U24E, U24F, U24G, U24H
