File: Hardware/PackVoltage_2022/PowerBoard_2022_Rev1/High Current Outputs.sch (KiCad schematic (older format))
At the start: 0 parts

Commit message: 12V stuff and hierarchical tags
Parts:
- added C? (x2): 0.1uF, symbol Device:C
- added C? (x2): 10uF, symbol Device:C
- added D? (x2): LED, symbol Device:LED
- added F? (x2): 20, symbol Device:Fuse
- added Q? (x2): BUK7M8R0-40EX, Package_TO_SOT_SMD:LFPAK33, symbol Transistor_FET:BUK7M8R0-40EX
- added R? (x2): 5.1k, symbol Device:R
- added R? (x2): 3300, symbol Device:R
- added R? (x2): 0.0025, symbol Device:R
- added U? (x2): LT1910, symbol MRDT_ICs:LT1910
- added U? (x2): INA281, Package_TO_SOT_SMD:SOT-23-5, symbol MRDT_ICs:INA281
Connections:
- net labels added: +5V, 12V, 12VA, 5V, Anderson_Aux, Anderson_Spare, Current_Sensor_Aux, Current_Sensor_Spare, Driver_Aux, Driver_Spare, GND
- wire segments 0 -> 68
