File: Hardware/PackVoltage_2022/PowerBoard_2022_Rev1/Low Current Out One.sch (KiCad schematic (older format))
At the start: 32 parts

Commit message: Created global tags in main sheet
Parts:
- U? (x2): symbol MRDT_ICs:LT1910 -> PowerBoard_2022_Rev1-rescue:LT1910-MRDT_ICs
- U? (x2): symbol MRDT_ICs:INA281 -> PowerBoard_2022_Rev1-rescue:INA281-MRDT_ICs
Changed lines of the file:
@@
 	850  1650 950  1650
 $Comp
-L MRDT_ICs:LT1910 U?
+L PowerBoard_2022_Rev1-rescue:LT1910-MRDT_ICs U?
 U 1 1 6189A53F
 P 2250 3750
@@
 	2700 1350 2800 1350
 $Comp
-L MRDT_ICs:INA281 U?
+L PowerBoard_2022_Rev1-rescue:INA281-MRDT_ICs U?
 U 1 1 6189A590
 P 1950 1200
@@
 	3500 1700 3600 1700
 $Comp
-L MRDT_ICs:LT1910 U?
+L PowerBoard_2022_Rev1-rescue:LT1910-MRDT_ICs U?
 U 1 1 618AAA5E
 P 4900 3800
@@
 	5350 1400 5450 1400
 $Comp
-L MRDT_ICs:INA281 U?
+L PowerBoard_2022_Rev1-rescue:INA281-MRDT_ICs U?
 U 1 1 618AAAAF
 P 4600 1250
