File: Hardware/PackVoltage_2022/PowerBoard_2022_Rev1/PowerBoard_2022_Rev1.sch (KiCad schematic (older format))
At the start: 7 parts

Commit message: Minor changes with Powerboard PDF
Parts:
- gave numbers to parts that had none: 7
Changed lines of the file:
@@
 	1550 6800 1650 6800
 $Comp
-L power:GND #PWR?
+L power:GND #PWR0101
 U 1 1 61881341
 P 3850 7250
-F 0 "#PWR?" H 3850 7000 50  0001 C CNN
+F 0 "#PWR0101" H 3850 7000 50  0001 C CNN
 F 1 "GND" H 3855 7077 50  0000 C CNN
 F 2 "" H 3850 7250 50  0001 C CNN
@@
 $EndComp
 $Comp
-L Device:D D?
+L Device:D D2
 U 1 1 61880E02
 P 3650 6950
-F 0 "D?" H 3500 7100 50  0000 L CNN
+F 0 "D2" H 3500 7100 50  0000 L CNN
 F 1 "1.5kE36A+" H 3350 7200 50  0000 L CNN
 F 2 "" H 3650 6950 50  0001 C CNN
@@
 $EndComp
 $Comp
-L Device:D D?
+L Device:D D1
 U 1 1 618805D4
 P 3400 6950
-F 0 "D?" V 3600 7000 50  0000 L CNN
+F 0 "D1" V 3600 7000 50  0000 L CNN
 F 1 "1.5kE36A+" V 3700 6800 50  0000 L CNN
 F 2 "" H 3400 6950 50  0001 C CNN
@@
 $EndComp
 $Comp
-L Device:CP1 C?
+L Device:CP1 C4
 U 1 1 61869A3D
 P 3000 6950
-F 0 "C?" H 3115 6996 50  0000 L CNN
+F 0 "C4" H 3115 6996 50  0000 L CNN
 F 1 "470uF" H 3115 6905 50  0000 L CNN
 F 2 "" H 3000 6950 50  0001 C CNN
@@
 $EndComp
 $Comp
-L Device:CP1 C?
+L Device:CP1 C3
 U 1 1 61869513
 P 2550 6950
-F 0 "C?" H 2665 6996 50  0000 L CNN
+F 0 "C3" H 2665 6996 50  0000 L CNN
 F 1 "470uF" H 2665 6905 50  0000 L CNN
 F 2 "" H 2550 6950 50  0001 C CNN
@@
 $EndComp
 $Comp
-L Device:CP1 C?
+L Device:CP1 C2
 U 1 1 61868EEC
 P 2100 6950
-F 0 "C?" H 2215 6996 50  0000 L CNN
+F 0 "C2" H 2215 6996 50  0000 L CNN
 F 1 "470uF" H 2215 6905 50  0000 L CNN
 F 2 "" H 2100 6950 50  0001 C CNN
@@
 $EndComp
 $Comp
-L Device:CP1 C?
+L Device:CP1 C1
 U 1 1 618684BC
 P 1650 6950
-F 0 "C?" H 1765 6996 50  0000 L CNN
+F 0 "C1" H 1765 6996 50  0000 L CNN
 F 1 "470uF" H 1765 6905 50  0000 L CNN
 F 2 "" H 1650 6950 50  0001 C CNN
@@
 $EndComp
 $Comp
-L MRDT_Drill_Holes:BATT_PWR_VIA V?
+L MRDT_Drill_Holes:BATT_PWR_VIA V1
 U 1 1 6186682A
 P 1550 6500
-F 0 "V?" H 1678 6520 60  0000 L CNN
+F 0 "V1" H 1678 6520 60  0000 L CNN
 F 1 "BATT_PWR_VIA" H 1678 6414 60  0000 L CNN
 F 2 "" H 1550 6500 60  0001 C CNN

Commit message: Added MRDT Libraries
Parts:
- V1: symbol MRDT_Drill_Holes:BATT_PWR_VIA -> PowerBoard_2022_Rev1-rescue:BATT_PWR_VIA-MRDT_Drill_Holes
Changed lines of the file:
@@
 Text GLabel 3700 5350 2    50   Input ~ 0
 Current_Sensor_Aux
-Text GLabel 3700 5450 2    50   Input ~ 0
-Current_Sensor_Spare
 Wire Wire Line
 	3700 3300 3600 3300
@@
 Wire Wire Line
 	3700 5250 3600 5250
-Wire Wire Line
-	3600 5450 3700 5450
 Wire Wire Line
 	3700 5350 3600 5350
@@
 $EndComp
 $Comp
-L MRDT_Drill_Holes:BATT_PWR_VIA V1
+L PowerBoard_2022_Rev1-rescue:BATT_PWR_VIA-MRDT_Drill_Holes V1
 U 1 1 6186682A
 P 1550 6500
