File: Hardware/PackVoltage_2022/PowerBoard_2022_Rev1/_autosave-12VSciLog.sch (KiCad schematic (older format))
At the start: 48 parts, among them U17 OKI-78SR-12_1.0-W36-C, U18 OKI-78SR-12_1.0-W36-C, U19 OKI-78SR-12_1.0-W36-C, U20 OKI-78SR-12_1.0-W36-C, U21 OKI-78SR-12_1.0-W36-C, U22 OKI-78SR-12_1.0-W36-C, U23 OKI-78SR-12_1.0-W36-C, U24 OKI-78SR-12_1.0-W36-C

Commit message: Added SciAct to the Board
Changed lines of the file:
@@
 Wire Wire Line
 	3250 4000 3250 5100
+Connection ~ 3550 1350
 $EndSCHEMATC
