File: Hardware/PackVoltage_2022/PowerBoard_2022_Rev1/PowerBoard_2022_Rev1.kicad_pcb (KiCad board)
At the start: 2 copper layers, 330.2 x 177.8 mm, 359 parts, among them Q1 BUK7M8R5-40HX, Q10 BUK7M8R5-40HX, Q11 BUK7M8R5-40HX, Q12 BUK7M8R5-40HX, Q13 BUK7M8R5-40HX, Q14 BUK7M8R5-40HX, Q15 BUK7M8R5-40HX, Q16 BUK7M8R5-40HX, Q17 BUK7M8R5-40HX, Q18 BUK7M8R5-40HX, Q19 BUK7M8R5-40HX, Q2 BUK7M8R5-40HX, Q20 BUK7M8R5-40HX, Q21 BUK7M8R5-40HX, Q22 BUK7M8R5-40HX, Q3 BUK7M8R5-40HX, Q4 BUK7M8R5-40HX, Q5 BUK7M8R5-40HX, Q6 BUK7M8R5-40HX, Q7 BUK7M8R5-40HX, Q8 BUK7M8R5-40HX, Q9 BUK7M8R5-40HX, U1 LT1910, U10 OKI-78SR-12_1.0-W36-C, U11 OKI-78SR-12_1.0-W36-C, U12 OKI-78SR-12_1.0-W36-C, U13 OKI-78SR-12_1.0-W36-C, U14 OKI-78SR-12_1.0-W36-C, U15 OKI-78SR-12_1.0-W36-C, U16 OKI-78SR-12_1.0-W36-C, U17 OKI-78SR-12_1.0-W36-C, U18 OKI-78SR-12_1.0-W36-C, U19 OKI-78SR-12_1.0-W36-C, U2 INA281, U20 OKI-78SR-12_1.0-W36-C, U21 OKI-78SR-12_1.0-W36-C, U22 OKI-78SR-12_1.0-W36-C, U23 OKI-78SR-12_1.0-W36-C, U24 OKI-78SR-12_1.0-W36-C, U25 LT1910, U26 LT1910, U27 LT1910, U28 LT1910, U29 INA281, U3 LT1910, U30 INA281, U31 INA281, U32 INA281, U33 LT1910, U34 LT1910, U35 LT1910, U36 INA281, U37 INA281, U38 INA281, U39 TM4C129E_Launchpad, U4 INA281, U40 LT1910, U41 LT1910, U42 INA281, U43 INA281, U44 LT1910, U45 INA281, U46 LT1910, U47 INA281, U48 LT1910, U49 LT1910, U5 OKI-78SR-5_1.5-W36-C, U50 LT1910, U51 LT1910, U52 INA281, U53 INA281, U54 INA281, U55 INA281, U56 INA281, U57 LT1910, U58 INA281, U59 LT1910, U6 OKI-78SR-3.3_1.5-W36-C, U60 LT1910, U61 LT1910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

Commit message: Rearranged layout to keep actuation next to logic
Parts:
- moved R20 344.8 mm to (69.3, -204.0)
- moved U21 344.8 mm to (76.0, -216.3)
- moved U22 344.8 mm to (87.8, -216.3)
- moved U23 344.8 mm to (111.3, -216.3)
- moved U24 344.8 mm to (99.5, -216.4)
- moved F6 308.1 mm to (82.9, -81.5), turned to 180 degrees
- moved C55 302.3 mm to (83.1, -90.9), turned to 0 degrees
- moved F3 297.2 mm to (374.3, -178.4), turned to 0 degrees
- moved F7 296.6 mm to (81.7, -174.9), turned to 180 degrees
- moved F4 294.7 mm to (373.8, -130.9), turned to 0 degrees
- moved U20 292.2 mm to (90.0, -85.3), turned to 0 degrees
- moved C56 287.1 mm to (91.0, -90.9), turned to 0 degrees
- moved C57 271.9 mm to (98.9, -90.9), turned to 0 degrees
- moved U19 270.0 mm to (101.7, -85.3), turned to 0 degrees
- moved C58 257.5 mm to (106.5, -90.7), turned to 0 degrees
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
Commit message: Started placing GimAct components
Parts:
- moved C63 1019.1 mm to (96.4, -200.2)
- moved C64 1015.5 mm to (92.8, -200.2)
- moved C65 1010.5 mm to (89.3, -200.2)
- moved Q11 1008.9 mm to (46.2, -218.7)
- moved C86 1008.9 mm to (63.5, -195.3)
- moved C88 1008.9 mm to (68.8, -208.5)
- moved D27 1008.9 mm to (58.2, -194.1)
- moved R43 1008.9 mm to (62.7, -207.8)
- moved R45 1008.9 mm to (71.4, -197.6)
- moved R47 1008.9 mm to (64.3, -219.2)
- moved U41 1008.9 mm to (53.6, -206.0)
- moved U43 1008.9 mm to (86.9, -215.4)
- moved C67 1005.7 mm to (84.3, -167.9)
- moved C66 1004.1 mm to (85.7, -200.2)
- moved C70 997.9 mm to (105.9, -167.9)
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Routing:
- added copper zone on B.Cu, net PVAct2

Commit message: Implemented GimAct
Parts:
- moved C22 721.1 mm to (32.5, -128.8)
- moved C24 721.1 mm to (39.6, -128.8)
- moved C35 721.1 mm to (46.7, -129.0)
- moved C36 721.1 mm to (53.8, -129.0)
- moved C100 448.3 mm to (680.5, -177.8)
- moved C105 448.3 mm to (678.2, -302.5)
- moved C107 448.3 mm to (765.3, -310.9)
- moved C108 448.3 mm to (689.1, -311.7)
- moved C109 448.3 mm to (668.3, -91.2)
- moved C89 448.3 mm to (522.7, -316.0)
- moved C95 448.3 mm to (615.7, -170.2)
- moved D28 448.3 mm to (544.1, -312.7)
- moved D30 448.3 mm to (869.7, -183.9)
- moved D34 448.3 mm to (828.3, -305.8)
- moved D38 448.3 mm to (767.3, -298.2)
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Routing:
- net 5V: track 83.2 -> 117.5 mm, vias 8 -> 10
- net Driver_GimAct: track 0.00 -> 32.9 mm, vias 0 -> 2
- net Current_Sense_GimAct: track 0.00 -> 14.8 mm
- net Net-(Q11-Pad4): track 0.00 -> 6.99 mm, vias 0 -> 2
- net Net-(R43-Pad1): track 0.00 -> 2.49 mm
- net Net-(C86-Pad1): track 0.00 -> 2.44 mm
- net GND: track 0.00 -> 2.25 mm, vias 2 -> 3
- net Net-(D27-Pad2): track 0.00 -> 1.66 mm
- added copper zone on F.Cu, net 12VGimAct
- added copper zone on F.Cu, net Anderson_GimAct
- added copper zone on F.Cu, net Net-(Q11-Pad1)

Commit message: Changed a lot, made the whole ass front plane pack, and questioned everything
Parts:
- C1, C2, C21, C3, C34, C4: footprint Capacitor_THT:CP_Radial_D6.3mm_P2.50mm -> Capacitor_THT:CP_Radial_D12.5mm_P5.00mm
- moved R58 774.1 mm to (126.5, -143.5), turned to 270 degrees
- moved U52 770.9 mm to (130.0, -143.5)
- moved U14 762.4 mm to (91.4, -126.0), turned to 90 degrees
- moved C93 760.1 mm to (122.7, -144.5)
- moved R67 759.9 mm to (103.2, -139.4)
- moved R62 759.7 mm to (130.3, -140.7)
- moved R68 757.8 mm to (99.3, -142.6), turned to 270 degrees
- moved Q18 757.5 mm to (100.1, -136.1), turned to 270 degrees
- moved C97 752.6 mm to (132.8, -136.9), turned to 90 degrees
- moved Q14 748.0 mm to (127.5, -137.2), turned to 270 degrees
- moved D34 746.3 mm to (99.3, -146.2), turned to 270 degrees
- moved C101 745.3 mm to (107.2, -135.5), turned to 90 degrees
- moved R66 744.2 mm to (93.1, -143.5), turned to 180 degrees
- moved D30 744.1 mm to (126.5, -147.2), turned to 270 degrees
- moved U56 744.0 mm to (103.3, -142.2)
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Routing:
- net 5V: track 117.5 -> 332.4 mm, vias 10 -> 24
- net Driver_M2: track 0.00 -> 21.7 mm, vias 0 -> 1
- net Driver_M6: track 0.00 -> 19.9 mm, vias 0 -> 1
- net Driver_Aux: track 0.00 -> 19.8 mm, vias 0 -> 1
- net Driver_NetSwitch: track 0.00 -> 19.0 mm, vias 0 -> 2
- net Net-(Q22-Pad4): track 0.00 -> 12.4 mm, vias 0 -> 2
- net Current_Sensor_Aux: track 0.00 -> 11.9 mm, vias 0 -> 1
- net Current_Sensor_M2: track 0.00 -> 11.6 mm, vias 0 -> 1
- net Net-(Q21-Pad4): track 0.00 -> 11.5 mm, vias 0 -> 2
- net Current_Sensor_M6: track 0.00 -> 9.79 mm, vias 0 -> 1
- net Net-(Q14-Pad4): track 0.00 -> 8.68 mm
- net Net-(Q18-Pad4): track 0.00 -> 7.85 mm
- net Net-(Q9-Pad4): track 0.00 -> 7.25 mm
- net Net-(Q2-Pad4): track 0.00 -> 7.21 mm
- net Net-(Q7-Pad4): track 0.00 -> 6.69 mm
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- added copper zone on F.Cu, net 12VDrive
- added copper zone on B.Cu, net 12VGimAct
- added copper zone on F.Cu, net 12VGimbal
- added copper zone on F.Cu, net 12VNetSwitch
- added copper zone on F.Cu, net 12VSciSensor
- added copper zone on F.Cu, net Anderson_Drive
- added copper zone on F.Cu, net Anderson_Gimbal
- added copper zone on F.Cu, net Anderson_NetSwitch
- added copper zone on F.Cu, net Anderson_SciSensor
- added copper zone on F.Cu, net Net-(C76-Pad1)
- added copper zone on F.Cu, net Net-(C8-Pad1)
- added copper zone on F.Cu, net Net-(C82-Pad1)
- added copper zone on F.Cu, net Net-(C84-Pad1)
- added copper zone on F.Cu, net Net-(Q14-Pad1)
- added copper zone on F.Cu, net Net-(Q18-Pad1)
- added copper zone on B.Cu, net Net-(Q2-Pad1)
- added copper zone on F.Cu, net Net-(Q2-Pad1)
- added copper zone on F.Cu, net Net-(Q21-Pad1)
- added copper zone on F.Cu, net Net-(Q22-Pad1)
- added copper zone on F.Cu, net Net-(Q7-Pad1)
- added copper zone on B.Cu, net Net-(Q9-Pad1)
- added copper zone on F.Cu, net Net-(Q9-Pad1)
- added copper zone on F.Cu, net PV
- added copper zone on B.Cu, net PV2
- added copper zone on F.Cu, net PVAct
- added copper zone on F.Cu, net PVAct2
- removed copper zone on F.Cu, net 12VGimAct
- removed copper zone on B.Cu, net PV
- removed copper zone on B.Cu, net PVAct
- removed copper zone on B.Cu, net PVAct2

Commit message: layout changes
Parts:
- moved Conn19 370.2 mm to (311.4, -41.5), turned to 180 degrees
- moved U28 356.7 mm to (309.8, -22.5), turned to 180 degrees
- moved D22 354.2 mm to (312.0, -28.8), turned to 180 degrees
- moved C74 351.8 mm to (315.8, -20.8), turned to 270 degrees
- moved F11 341.0 mm to (303.3, -3.05), turned to 90 degrees
- moved Q6 340.6 mm to (302.0, -27.4), turned to 180 degrees
- moved R24 337.8 mm to (315.8, -24.1), turned to 90 degrees
- moved R31 337.8 mm to (308.6, -28.8), turned to 180 degrees
- moved U32 329.9 mm to (301.4, -33.7), turned to 90 degrees
- moved C78 327.9 mm to (303.3, -21.9), turned to 90 degrees
- moved R32 327.3 mm to (306.8, -33.7), turned to 90 degrees
- moved C71 314.7 mm to (159.8, -22.3)
- moved C75 314.7 mm to (146.0, -23.6)
- moved Conn1 314.7 mm to (156.7, -41.4)
- moved D19 314.7 mm to (153.6, -31.8)
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Routing:
- net 5V: track 332.4 -> 413.4 mm, vias 24 -> 30
- net Driver_M4: track 20.1 -> 0.00 mm, vias 1 -> 0
- net Net-(Q1-Pad1): track 0.00 -> 20.1 mm
- net Driver_M3: track 0.00 -> 19.9 mm, vias 0 -> 1
- net Driver_M7: track 0.00 -> 18.9 mm, vias 0 -> 1
- net Current_Sensor_M4: track 15.9 -> 0.00 mm, vias 1 -> 0
- net GND: track 4.98 -> 20.9 mm, vias 6 -> 7
- net Current_Sensor_M7: track 0.00 -> 14.6 mm, vias 0 -> 1
- net Driver_M5: track 0.00 -> 13.3 mm, vias 0 -> 1
- net Current_Sensor_M5: track 0.00 -> 12.5 mm, vias 0 -> 1
- net Current_Sensor_M3: track 0.00 -> 12.3 mm, vias 0 -> 1
- net Net-(Q4-Pad4): track 0.00 -> 7.96 mm
- net Net-(Q6-Pad4): track 0.00 -> 5.81 mm
- net Net-(C8-Pad1): track 0.00 -> 5.17 mm
- net Net-(C72-Pad1): track 0.00 -> 3.96 mm
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- added copper zone on F.Cu, net Anderson_Aux
- added copper zone on F.Cu, net Anderson_M2
- added copper zone on F.Cu, net Anderson_M3
- added copper zone on F.Cu, net Anderson_M6
- added copper zone on F.Cu, net Anderson_M7
- added copper zone on F.Cu, net Net-(C78-Pad1)
- added copper zone on B.Cu, net Net-(Q4-Pad1)
- added copper zone on F.Cu, net Net-(Q4-Pad1)
- added copper zone on B.Cu, net Net-(Q6-Pad1)
- added copper zone on F.Cu, net Net-(Q6-Pad1)

Commit message: fixed wire issues
Routing:
- net Net-(Q1-Pad1): track 20.1 -> 0.00 mm, vias 2 -> 0
- net Driver_M4: track 0.00 -> 18.1 mm, vias 0 -> 1
- net GND: track 20.9 -> 5.50 mm, vias 7 -> 4
- net Current_Sensor_M4: track 0.00 -> 11.5 mm, vias 0 -> 1
- net Net-(Q5-Pad4): track 7.42 -> 0.00 mm, vias 2 -> 0
- net Net-(Q1-Pad4): track 3.58 -> 8.76 mm
- net Current_Sensor_M3: track 12.3 -> 7.57 mm
- net Net-(C8-Pad1): track 5.17 -> 0.66 mm
- net Current_Sensor_POE: track 15.3 -> 11.1 mm
- net Current_Sensor_M7: track 14.6 -> 10.5 mm
- net Net-(R34-Pad1): track 0.00 -> 3.58 mm
- net Net-(C80-Pad1): track 0.00 -> 3.50 mm, vias 1 -> 0
- net Net-(R1-Pad1): track 0.00 -> 3.37 mm
- net Driver_Aux: track 23.2 -> 19.9 mm
- net Driver_M2: track 21.7 -> 18.8 mm
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- added copper zone on B.Cu, net Net-(Q5-Pad1)
- added copper zone on B.Cu, net Net-(Q7-Pad1)
- removed copper zone on F.Cu, net Net-(C78-Pad1)

Commit message: Organized
Parts:
- moved R16 609.5 mm to (110.5, -135.4), turned to 180 degrees
- moved D8 589.0 mm to (909.1, -78.2)
- moved R11 561.2 mm to (117.7, -118.4), turned to 180 degrees
- moved R15 533.7 mm to (141.2, -108.9), turned to 90 degrees
- moved D10 517.4 mm to (838.8, -112.0)
- moved D16 475.1 mm to (667.5, -292.9)
- moved D15 469.3 mm to (672.6, -278.6)
- moved D7 448.9 mm to (766.1, -75.2)
- moved C41 422.4 mm to (635.7, -240.9)
- moved C42 422.4 mm to (634.2, -237.0)
- moved D12 407.3 mm to (715.8, -72.4)
- moved R18 396.4 mm to (663.1, -292.4)
- moved C46 363.8 mm to (590.1, -280.7)
- moved C45 363.8 mm to (598.4, -280.4)
- moved R17 356.8 mm to (679.5, -277.6)
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Routing:
- net Net-(D13-Pad2): track 0.00 -> 1.95 mm
- net Net-(Q2-Pad1): track 1.86 -> 0.00 mm
- net Net-(D9-Pad2): track 0.00 -> 1.84 mm
- net Net-(D14-Pad2): track 0.00 -> 1.67 mm
- net GND: vias 4 -> 3
- net Net-(Q8-Pad1): vias 0 -> 2

Commit message: Connected GND pads to GND
Routing:
- net GND: track 5.50 -> 160.4 mm, vias 3 -> 11
- net Net-(D18-Pad2): track 0.00 -> 1.69 mm
- added copper zone on F.Cu, net PV2
- removed copper zone on B.Cu, net PV2
