File: Hardware/PackVoltage_2022/PowerBoard_2022_Rev1/PowerBoard_2022_Rev1.kicad_pcb (KiCad board)
At the start: 2 copper layers, 279.4 x 152.4 mm, 261 parts, among them Q1 BUK768R3-60E, Q10 BUK768R3-60E, Q11 BUK768R3-60E, Q12 BUK768R3-60E, Q13 BUK768R3-60E, Q14 BUK768R3-60E, Q15 BUK768R3-60E, Q16 BUK768R3-60E, Q17 BUK768R3-60E, Q18 BUK768R3-60E, Q19 BUK768R3-60E, Q2 BUK768R3-60E, Q20 BUK768R3-60E, Q21 BUK768R3-60E, Q22 BUK768R3-60E, Q3 BUK768R3-60E, Q4 BUK768R3-60E, Q5 BUK768R3-60E, Q6 BUK768R3-60E, Q7 BUK768R3-60E, Q8 BUK768R3-60E, Q9 BUK768R3-60E, U1 LT1910, U2 INA281, U25 LT1910, U26 LT1910, U27 LT1910, U28 LT1910, U29 INA281, U3 LT1910, U30 INA281, U31 INA281, U32 INA281, U33 LT1910, U34 LT1910, U35 LT1910, U36 INA281, U37 INA281, U38 INA281, U39 TM4C129E_Launchpad, U4 INA281, U40 LT1910, U41 LT1910, U42 INA281, U43 INA281, U44 LT1910, U45 INA281, U46 LT1910, U47 INA281, U48 LT1910, U49 LT1910, U5 OKI-78SR-5_1.5-W36-C, U50 LT1910, U51 LT1910, U52 INA281, U53 INA281, U54 INA281, U55 INA281, U56 INA281, U57 LT1910, U58 INA281, U59 LT1910, U6 OKI-78SR-3.3_1.5-W36-C, U60 LT1910, U61 LT1910, U62 LT1910, U63 INA281, U64 INA281, U65 INA281

Commit message: added screw holes
Parts:
- added REF**: 4_40_Hole, MRDT_Drill_Holes:4_40_Hole_Corner, F.Cu at (363.6, 169.8)
- added REF**: 4_40_Hole, MRDT_Drill_Holes:4_40_Hole_Corner, F.Cu at (363.7, 33.4)
- added REF**: 4_40_Hole, MRDT_Drill_Holes:4_40_Hole_Corner, F.Cu at (627.0, 169.8)
- added REF**: 4_40_Hole, MRDT_Drill_Holes:4_40_Hole_Corner, F.Cu at (627.0, 33.4)
Changed lines of the file:
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@@
     (tracks 120)
     (zones 0)
-    (modules 261)
+    (modules 265)
     (nets 239)
   )
@@
     (38 B.Mask user)
     (39 F.Mask user)
-    (40 Dwgs.User user)
+    (40 Dwgs.User user hide)
     (41 Cmts.User user)
     (42 Eco1.User user)
@@
     (add_net PVMulti)
   )
+  (module MRDT_Drill_Holes:4_40_Hole_Corner (layer F.Cu)
+    (at 363.601 169.799 180)
+    (fp_text reference REF** (at 4.00812 -3.50812) (layer F.SilkS) hide
+      (effects (font (size 1 1) (thickness 0.15)))
+    )
+    (fp_text value 4_40_Hole (at 4.00812 -4.50812) (layer F.Fab) hide
+      (effects (font (size 1 1) (thickness 0.15)))
+    )
+    (fp_line (start 0 0) (end 8.0264 0) (layer F.Fab) (width 0.15))
+    (fp_line (start 0 -8.0264) (end 0 0) (layer F.Fab) (width 0.15))
+    (fp_line (start 4.0132 -8.0264) (end 0 -8.0264) (layer F.Fab) (width 0.15))
+    (fp_line (start 8.0264 -4.0132) (end 8.0264 0) (layer F.Fab) (width 0.15))
+    (fp_arc (start 4.0132 -4.0132) (end 4.0132 -8.0264) (angle 90) (layer F.Fab) (width 0.15))
+    (fp_circle (center 4.00812 -4.00812) (end 4.00812 0.00508) (layer F.SilkS) (width 0.15))
+    (pad "" np_thru_hole circle (at 4.00812 -4.00812 180) (size 2.9464 2.9464) (drill 2.9464) (layers *.Cu *.Mask)
+      (clearance 2.5))
+  )
+  (module MRDT_Drill_Holes:4_40_Hole_Corner (layer F.Cu)
+    (at 363.67212 33.401 90)
+    (fp_text reference REF** (at 4.00812 -3.50812 90) (layer F.SilkS) hide
+      (effects (font (size 1 1) (thickness 0.15)))
+    )
+    (fp_text value 4_40_Hole (at 4.00812 -4.50812 90) (layer F.Fab) hide
+      (effects (font (size 1 1) (thickness 0.15)))
+    )
+    (fp_line (start 0 0) (end 8.0264 0) (layer F.Fab) (width 0.15))
+    (fp_line (start 0 -8.0264) (end 0 0) (layer F.Fab) (width 0.15))
+    (fp_line (start 4.0132 -8.0264) (end 0 -8.0264) (layer F.Fab) (width 0.15))
+    (fp_line (start 8.0264 -4.0132) (end 8.0264 0) (layer F.Fab) (width 0.15))
+    (fp_arc (start 4.0132 -4.0132) (end 4.0132 -8.0264) (angle 90) (layer F.Fab) (width 0.15))
+    (fp_circle (center 4.00812 -4.00812) (end 4.00812 0.00508) (layer F.SilkS) (width 0.15))
+    (pad "" np_thru_hole circle (at 4.00812 -4.00812 90) (size 2.9464 2.9464) (drill 2.9464) (layers *.Cu *.Mask)
+      (clearance 2.5))
+  )
+  (module MRDT_Drill_Holes:4_40_Hole_Corner (layer F.Cu)
+    (at 626.999 169.799 270)
+    (fp_text reference REF** (at 4.00812 -3.50812 90) (layer F.SilkS) hide
+      (effects (font (size 1 1) (thickness 0.15)))
+    )
+    (fp_text value 4_40_Hole (at 4.00812 -4.50812 90) (layer F.Fab) hide
+      (effects (font (size 1 1) (thickness 0.15)))
+    )
+    (fp_line (start 0 0) (end 8.0264 0) (layer F.Fab) (width 0.15))
+    (fp_line (start 0 -8.0264) (end 0 0) (layer F.Fab) (width 0.15))
+    (fp_line (start 4.0132 -8.0264) (end 0 -8.0264) (layer F.Fab) (width 0.15))
+    (fp_line (start 8.0264 -4.0132) (end 8.0264 0) (layer F.Fab) (width 0.15))
+    (fp_arc (start 4.0132 -4.0132) (end 4.0132 -8.0264) (angle 90) (layer F.Fab) (width 0.15))
+    (fp_circle (center 4.00812 -4.00812) (end 4.00812 0.00508) (layer F.SilkS) (width 0.15))
+    (pad "" np_thru_hole circle (at 4.00812 -4.00812 270) (size 2.9464 2.9464) (drill 2.9464) (layers *.Cu *.Mask)
+      (clearance 2.5))
+  )
+  (module MRDT_Drill_Holes:4_40_Hole_Corner (layer F.Cu)
+    (at 626.999 33.401)
+    (fp_text reference REF** (at 4.00812 -3.50812) (layer F.SilkS) hide
+      (effects (font (size 1 1) (thickness 0.15)))
+    )
+    (fp_text value 4_40_Hole (at 4.00812 -4.50812) (layer F.Fab) hide
+      (effects (font (size 1 1) (thickness 0.15)))
+    )
+    (fp_line (start 0 0) (end 8.0264 0) (layer F.Fab) (width 0.15))
+    (fp_line (start 0 -8.0264) (end 0 0) (layer F.Fab) (width 0.15))
+    (fp_line (start 4.0132 -8.0264) (end 0 -8.0264) (layer F.Fab) (width 0.15))
+    (fp_line (start 8.0264 -4.0132) (end 8.0264 0) (layer F.Fab) (width 0.15))
+    (fp_arc (start 4.0132 -4.0132) (end 4.0132 -8.0264) (angle 90) (layer F.Fab) (width 0.15))
+    (fp_circle (center 4.00812 -4.00812) (end 4.00812 0.00508) (layer F.SilkS) (width 0.15))
+    (pad "" np_thru_hole circle (at 4.00812 -4.00812) (size 2.9464 2.9464) (drill 2.9464) (layers *.Cu *.Mask)
+      (clearance 2.5))
+  )
   (module MRDT_Shields:TM4C129E_Launchpad_FULL_THT_TOP (layer F.Cu)

Commit message: Organized PV Aux Circuit
Parts:
- moved C8 379.7 mm to (542.2, -38.1), turned to 0 degrees
- moved U3 367.8 mm to (541.7, -44.2)
- moved Conn2 367.6 mm to (543.8, -65.3), turned to 270 degrees
- moved Q2 367.4 mm to (533.7, -43.9), turned to 0 degrees
- moved R4 367.3 mm to (547.4, -45.7)
- moved C7 367.3 mm to (547.4, -41.7)
- moved F2 367.2 mm to (534.7, -24.1)
- moved U4 366.3 mm to (533.0, -56.5), turned to 0 degrees
- moved R6 363.5 mm to (534.9, -50.5), turned to 0 degrees
- moved R5 354.4 mm to (528.7, -53.3), turned to 270 degrees
- moved D4 351.1 mm to (528.7, -57.3), turned to 270 degrees
- moved C72 330.2 mm to (554.0, -118.9)
- moved C74 330.2 mm to (633.1, -118.4)
- moved C75 330.2 mm to (500.5, -116.0)
- moved C76 330.2 mm to (537.6, -114.9)
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Routing:
- net Net-(Q2-Pad4): track 0.00 -> 12.3 mm, vias 0 -> 2
- net Net-(Q2-Pad1): track 0.65 -> 5.02 mm, vias 3 -> 0
- net Net-(C7-Pad1): track 0.00 -> 3.41 mm
- net Anderson_Aux: track 0.00 -> 3.20 mm
- net Net-(R4-Pad1): track 0.00 -> 2.98 mm
- net Net-(C8-Pad1): track 0.66 -> 0.00 mm
- net Net-(D4-Pad2): track 1.73 -> 2.24 mm
- removed copper zone on B.Cu, net Net-(Q2-Pad1)
- removed copper zone on F.Cu, net Net-(Q2-Pad1)
