File: Hardware/PackVoltage_2022/PowerBoard_2022_Rev1/12VSciLog.sch (KiCad schematic (older format))
At the start: 48 parts, among them U17 OKI-78SR-12_1.0-W36-C, U18 OKI-78SR-12_1.0-W36-C, U19 OKI-78SR-12_1.0-W36-C, U20 OKI-78SR-12_1.0-W36-C, U21 OKI-78SR-12_1.0-W36-C, U22 OKI-78SR-12_1.0-W36-C, U23 OKI-78SR-12_1.0-W36-C, U24 OKI-78SR-12_1.0-W36-C

Commit message: Removed redundant LED's in Actuation circuits and final touches on SciAct Layout
Parts:
- removed D18, D19, D20, D22, D23, D24: LED, LED_SMD:LED_0603_1608Metric_Pad1.05x0.95mm_HandSolder, symbol Device:LED
- removed R20, R21, R22, R24, R25, R26: 1000, Resistor_SMD:R_0603_1608Metric_Pad1.05x0.95mm_HandSolder, symbol Device:R
- renumbered D21 to D18, R23 to R20
