File: Hardware/PackVoltage_2022/PowerBoard_2022_Rev1/PackVoltage_2022_Rev1/TIVA.sch (KiCad schematic (older format))
At the start: 8 parts

Commit message: saving
Parts:
- gave numbers to parts that had none: 1
Changed lines of the file:
@@
 	4700 3750 4700 3600
 $Comp
-L power:+3.3V #PWR?
+L power:+3.3V #PWR0144
 U 1 1 620F068D
 P 4700 3600
-F 0 "#PWR?" H 4700 3450 50  0001 C CNN
+F 0 "#PWR0144" H 4700 3450 50  0001 C CNN
 F 1 "+3.3V" H 4715 3773 50  0000 C CNN
 F 2 "" H 4700 3600 50  0001 C CNN
@@
 $EndComp
 $Comp
-L power:GND #PWR?
+L power:GND #PWR0145
 U 1 1 620F0747
 P 5850 3850
-F 0 "#PWR?" H 5850 3600 50  0001 C CNN
+F 0 "#PWR0145" H 5850 3600 50  0001 C CNN
 F 1 "GND" H 5855 3677 50  0000 C CNN
 F 2 "" H 5850 3850 50  0001 C CNN
@@
 Driver_POE
 $Comp
-L MRDT_Shields:TM4C129E_Launchpad U?
+L MRDT_Shields:TM4C129E_Launchpad U19
 U 1 1 6228A2B2
 P 5050 3150
-F 0 "U?" H 5100 3050 60  0000 L CNN
+F 0 "U19" H 5100 3050 60  0000 L CNN
 F 1 "TM4C129E_Launchpad" H 4650 2950 60  0000 L CNN
 F 2 "" H 5050 3150 60  0001 C CNN
@@
 $EndComp
 $Comp
-L MRDT_Shields:TM4C129E_Launchpad U?
+L MRDT_Shields:TM4C129E_Launchpad U19
 U 2 1 6228DC9E
 P 5650 3150
-F 0 "U?" H 5681 4427 60  0000 C CNN
+F 0 "U19" H 5681 4427 60  0000 C CNN
 F 1 "TM4C129E_Launchpad" H 5681 4321 60  0000 C CNN
 F 2 "" H 5650 3150 60  0001 C CNN
@@
 $EndComp
 $Comp
-L MRDT_Shields:TM4C129E_Launchpad U?
+L MRDT_Shields:TM4C129E_Launchpad U19
 U 3 1 62291C19
 P 8050 3150
-F 0 "U?" H 8100 3050 60  0000 L CNN
+F 0 "U19" H 8100 3050 60  0000 L CNN
 F 1 "TM4C129E_Launchpad" H 7650 2900 60  0000 L CNN
 F 2 "" H 8050 3150 60  0001 C CNN
@@
 $EndComp
 $Comp
-L MRDT_Shields:TM4C129E_Launchpad U?
+L MRDT_Shields:TM4C129E_Launchpad U19
 U 6 1 622D3AFF
 P 5650 4700
-F 0 "U?" H 5800 5850 60  0000 C CNN
+F 0 "U19" H 5800 5850 60  0000 C CNN
 F 1 "TM4C129E_Launchpad" H 5700 5950 60  0000 C CNN
 F 2 "" H 5650 4700 60  0001 C CNN
@@
 $EndComp
 $Comp
-L MRDT_Shields:TM4C129E_Launchpad U?
+L MRDT_Shields:TM4C129E_Launchpad U19
 U 7 1 622DC2FB
 P 8050 4800
-F 0 "U?" H 8081 4613 60  0000 C CNN
+F 0 "U19" H 8081 4613 60  0000 C CNN
 F 1 "TM4C129E_Launchpad" H 8081 4719 60  0000 C CNN
 F 2 "" H 8050 4800 60  0001 C CNN
@@
 $EndComp
 $Comp
-L MRDT_Shields:TM4C129E_Launchpad U?
+L MRDT_Shields:TM4C129E_Launchpad U19
 U 8 1 622E4587
 P 8650 4800
-F 0 "U?" H 8750 5950 60  0000 C CNN
+F 0 "U19" H 8750 5950 60  0000 C CNN
 F 1 "TM4C129E_Launchpad" H 8750 6050 60  0000 C CNN
 F 2 "" H 8650 4800 60  0001 C CNN
@@
 $EndComp
 $Comp
-L power:GND #PWR?
+L power:GND #PWR0146
 U 1 1 622EF469
 P 5850 2300
-F 0 "#PWR?" H 5850 2050 50  0001 C CNN
+F 0 "#PWR0146" H 5850 2050 50  0001 C CNN
 F 1 "GND" H 5855 2127 50  0000 C CNN
 F 2 "" H 5850 2300 50  0001 C CNN
@@
 $EndComp
 $Comp
-L power:GND #PWR?
+L power:GND #PWR0147
 U 1 1 622F0EA4
 P 8850 3850
-F 0 "#PWR?" H 8850 3600 50  0001 C CNN
+F 0 "#PWR0147" H 8850 3600 50  0001 C CNN
 F 1 "GND" H 8855 3677 50  0000 C CNN
 F 2 "" H 8850 3850 50  0001 C CNN
@@
 $EndComp
 $Comp
-L power:GND #PWR?
+L power:GND #PWR0148
 U 1 1 622EE8B7
 P 8850 2200
-F 0 "#PWR?" H 8850 1950 50  0001 C CNN
+F 0 "#PWR0148" H 8850 1950 50  0001 C CNN
 F 1 "GND" H 8855 2027 50  0000 C CNN
 F 2 "" H 8850 2200 50  0001 C CNN
@@
 $EndComp
 $Comp
-L MRDT_Shields:TM4C129E_Launchpad U?
+L MRDT_Shields:TM4C129E_Launchpad U19
 U 4 1 6229B428
 P 8650 3150
-F 0 "U?" H 8700 4350 60  0000 L CNN
+F 0 "U19" H 8700 4350 60  0000 L CNN
 F 1 "TM4C129E_Launchpad" H 8300 4450 60  0000 L CNN
 F 2 "" H 8650 3150 60  0001 C CNN
@@
 $EndComp
 $Comp
-L MRDT_Shields:TM4C129E_Launchpad U?
+L MRDT_Shields:TM4C129E_Launchpad U19
 U 5 1 622CEEA6
 P 5050 4700
-F 0 "U?" H 5079 4513 60  0000 C CNN
+F 0 "U19" H 5079 4513 60  0000 C CNN
 F 1 "TM4C129E_Launchpad" H 5079 4619 60  0000 C CNN
 F 2 "" H 5050 4700 60  0001 C CNN
@@
 	4700 2200 4700 2050
 $Comp
-L power:+3.3V #PWR?
+L power:+3.3V #PWR0149
 U 1 1 62371C03
 P 4700 2050
-F 0 "#PWR?" H 4700 1900 50  0001 C CNN
+F 0 "#PWR0149" H 4700 1900 50  0001 C CNN
 F 1 "+3.3V" H 4715 2223 50  0000 C CNN
 F 2 "" H 4700 2050 50  0001 C CNN

Commit message: schematic started
Parts:
- U19: footprint (none) -> MRDT_Shields:TM4C129E_Launchpad_FULL_THT_TOP
Changed lines of the file:
@@
 $Descr A4 11693 8268
 encoding utf-8
-Sheet 2 3
+Sheet 3 3
 Title ""
 Date ""
@@
 F 0 "U19" H 5100 3050 60  0000 L CNN
 F 1 "TM4C129E_Launchpad" H 4650 2950 60  0000 L CNN
-F 2 "" H 5050 3150 60  0001 C CNN
+F 2 "MRDT_Shields:TM4C129E_Launchpad_FULL_THT_TOP" H 5050 3150 60  0001 C CNN
 F 3 "" H 5050 3150 60  0001 C CNN
 	1    5050 3150
@@
 F 0 "U19" H 5681 4427 60  0000 C CNN
 F 1 "TM4C129E_Launchpad" H 5681 4321 60  0000 C CNN
-F 2 "" H 5650 3150 60  0001 C CNN
+F 2 "MRDT_Shields:TM4C129E_Launchpad_FULL_THT_TOP" H 5650 3150 60  0001 C CNN
 F 3 "" H 5650 3150 60  0001 C CNN
 	2    5650 3150
@@
 F 0 "U19" H 8100 3050 60  0000 L CNN
 F 1 "TM4C129E_Launchpad" H 7650 2900 60  0000 L CNN
-F 2 "" H 8050 3150 60  0001 C CNN
+F 2 "MRDT_Shields:TM4C129E_Launchpad_FULL_THT_TOP" H 8050 3150 60  0001 C CNN
 F 3 "" H 8050 3150 60  0001 C CNN
 	3    8050 3150
@@
 F 0 "U19" H 5800 5850 60  0000 C CNN
 F 1 "TM4C129E_Launchpad" H 5700 5950 60  0000 C CNN
-F 2 "" H 5650 4700 60  0001 C CNN
+F 2 "MRDT_Shields:TM4C129E_Launchpad_FULL_THT_TOP" H 5650 4700 60  0001 C CNN
 F 3 "" H 5650 4700 60  0001 C CNN
 	6    5650 4700
@@
 F 0 "U19" H 8081 4613 60  0000 C CNN
 F 1 "TM4C129E_Launchpad" H 8081 4719 60  0000 C CNN
-F 2 "" H 8050 4800 60  0001 C CNN
+F 2 "MRDT_Shields:TM4C129E_Launchpad_FULL_THT_TOP" H 8050 4800 60  0001 C CNN
 F 3 "" H 8050 4800 60  0001 C CNN
 	7    8050 4800
@@
 F 0 "U19" H 8750 5950 60  0000 C CNN
 F 1 "TM4C129E_Launchpad" H 8750 6050 60  0000 C CNN
-F 2 "" H 8650 4800 60  0001 C CNN
+F 2 "MRDT_Shields:TM4C129E_Launchpad_FULL_THT_TOP" H 8650 4800 60  0001 C CNN
 F 3 "" H 8650 4800 60  0001 C CNN
 	8    8650 4800
@@
 F 0 "U19" H 8700 4350 60  0000 L CNN
 F 1 "TM4C129E_Launchpad" H 8300 4450 60  0000 L CNN
-F 2 "" H 8650 3150 60  0001 C CNN
+F 2 "MRDT_Shields:TM4C129E_Launchpad_FULL_THT_TOP" H 8650 3150 60  0001 C CNN
 F 3 "" H 8650 3150 60  0001 C CNN
 	4    8650 3150
@@
 F 0 "U19" H 5079 4513 60  0000 C CNN
 F 1 "TM4C129E_Launchpad" H 5079 4619 60  0000 C CNN
-F 2 "" H 5050 4700 60  0001 C CNN
+F 2 "MRDT_Shields:TM4C129E_Launchpad_FULL_THT_TOP" H 5050 4700 60  0001 C CNN
 F 3 "" H 5050 4700 60  0001 C CNN
 	5    5050 4700
