File: Hardware/PackVoltage_2022/PowerBoard_2022_Rev1/PackVoltage_2022_Rev1/MOTORS.sch (KiCad schematic (older format))
At the start: 83 parts

Commit message: Changed Resistor Values Pt.2
Parts:
- C? (x8): value .1uF -> 0.1uF
- R? (x9): value 3300 -> 2800
Changed lines of the file:
@@
 AR Path="/6219DADC/621D647B" Ref="C?"  Part="1"
 F 0 "C?" H 6765 5946 50  0000 L CNN
-F 1 ".1uF" H 6765 5855 50  0000 L CNN
+F 1 "0.1uF" H 6765 5855 50  0000 L CNN
 F 2 "" H 6688 5750 50  0001 C CNN
 F 3 "~" H 6650 5900 50  0001 C CNN
@@
 AR Path="/6219DADC/621D64B4" Ref="R?"  Part="1"
 F 0 "R?" V 8900 6300 50  0000 C CNN
-F 1 "3300" V 9000 6300 50  0000 C CNN
+F 1 "2800" V 9000 6300 50  0000 C CNN
 F 2 "" V 8930 6300 50  0001 C CNN
 F 3 "~" H 9000 6300 50  0001 C CNN
@@
 AR Path="/6219DADC/621D6D3A" Ref="C?"  Part="1"
 F 0 "C?" H 7065 2996 50  0000 L CNN
-F 1 ".1uF" H 7065 2905 50  0000 L CNN
+F 1 "0.1uF" H 7065 2905 50  0000 L CNN
 F 2 "" H 6988 2800 50  0001 C CNN
 F 3 "~" H 6950 2950 50  0001 C CNN
@@
 AR Path="/6219DADC/621D6D73" Ref="R?"  Part="1"
 F 0 "R?" V 9200 3350 50  0000 C CNN
-F 1 "3300" V 9300 3350 50  0000 C CNN
+F 1 "2800" V 9300 3350 50  0000 C CNN
 F 2 "" V 9230 3350 50  0001 C CNN
 F 3 "~" H 9300 3350 50  0001 C CNN
@@
 AR Path="/6219DADC/621D835C" Ref="C?"  Part="1"
 F 0 "C?" H 6815 1546 50  0000 L CNN
-F 1 ".1uF" H 6815 1455 50  0000 L CNN
+F 1 "0.1uF" H 6815 1455 50  0000 L CNN
 F 2 "" H 6738 1350 50  0001 C CNN
 F 3 "~" H 6700 1500 50  0001 C CNN
@@
 AR Path="/6219DADC/621D8395" Ref="R?"  Part="1"
 F 0 "R?" V 8950 1900 50  0000 C CNN
-F 1 "3300" V 9050 1900 50  0000 C CNN
+F 1 "2800" V 9050 1900 50  0000 C CNN
 F 2 "" V 8980 1900 50  0001 C CNN
 F 3 "~" H 9050 1900 50  0001 C CNN
@@
 AR Path="/6219DADC/621DC704" Ref="C?"  Part="1"
 F 0 "C?" H 1415 1646 50  0000 L CNN
-F 1 ".1uF" H 1415 1555 50  0000 L CNN
+F 1 "0.1uF" H 1415 1555 50  0000 L CNN
 F 2 "" H 1338 1450 50  0001 C CNN
 F 3 "~" H 1300 1600 50  0001 C CNN
@@
 AR Path="/6219DADC/621DC73D" Ref="R?"  Part="1"
 F 0 "R?" V 3550 2000 50  0000 C CNN
-F 1 "3300" V 3650 2000 50  0000 C CNN
+F 1 "2800" V 3650 2000 50  0000 C CNN
 F 2 "" V 3580 2000 50  0001 C CNN
 F 3 "~" H 3650 2000 50  0001 C CNN
@@
 AR Path="/6219DADC/621E2A6B" Ref="C?"  Part="1"
 F 0 "C?" H 1515 3246 50  0000 L CNN
-F 1 ".1uF" H 1515 3155 50  0000 L CNN
+F 1 "0.1uF" H 1515 3155 50  0000 L CNN
 F 2 "" H 1438 3050 50  0001 C CNN
 F 3 "~" H 1400 3200 50  0001 C CNN
@@
 AR Path="/6219DADC/621E2AA4" Ref="R?"  Part="1"
 F 0 "R?" V 3650 3600 50  0000 C CNN
-F 1 "3300" V 3750 3600 50  0000 C CNN
+F 1 "2800" V 3750 3600 50  0000 C CNN
 F 2 "" V 3680 3600 50  0001 C CNN
 F 3 "~" H 3750 3600 50  0001 C CNN
@@
 AR Path="/6219DADC/621ECAEF" Ref="C?"  Part="1"
 F 0 "C?" H 1615 4896 50  0000 L CNN
-F 1 ".1uF" H 1615 4805 50  0000 L CNN
+F 1 "0.1uF" H 1615 4805 50  0000 L CNN
 F 2 "" H 1538 4700 50  0001 C CNN
 F 3 "~" H 1500 4850 50  0001 C CNN
@@
 AR Path="/6219DADC/621ECB28" Ref="R?"  Part="1"
 F 0 "R?" V 3750 5250 50  0000 C CNN
-F 1 "3300" V 3850 5250 50  0000 C CNN
+F 1 "2800" V 3850 5250 50  0000 C CNN
 F 2 "" V 3780 5250 50  0001 C CNN
 F 3 "~" H 3850 5250 50  0001 C CNN
@@
 AR Path="/6219DADC/621FB404" Ref="C?"  Part="1"
 F 0 "C?" H 1765 6746 50  0000 L CNN
-F 1 ".1uF" H 1765 6655 50  0000 L CNN
+F 1 "0.1uF" H 1765 6655 50  0000 L CNN
 F 2 "" H 1688 6550 50  0001 C CNN
 F 3 "~" H 1650 6700 50  0001 C CNN
@@
 AR Path="/6219DADC/621FB43D" Ref="R?"  Part="1"
 F 0 "R?" V 3900 7100 50  0000 C CNN
-F 1 "3300" V 4000 7100 50  0000 C CNN
+F 1 "2800" V 4000 7100 50  0000 C CNN
 F 2 "" V 3930 7100 50  0001 C CNN
 F 3 "~" H 4000 7100 50  0001 C CNN
@@
 AR Path="/6219DADC/624236D3" Ref="R?"  Part="1"
 F 0 "R?" V 6000 7550 50  0000 C CNN
-F 1 "3300" V 6100 7550 50  0000 C CNN
+F 1 "2800" V 6100 7550 50  0000 C CNN
 F 2 "" V 6030 7550 50  0001 C CNN
 F 3 "~" H 6100 7550 50  0001 C CNN
@@
 AR Path="/6219DADC/6211E3C0" Ref="C?"  Part="1"
 F 0 "C?" H 6665 4546 50  0000 L CNN
-F 1 ".1uF" H 6665 4455 50  0000 L CNN
+F 1 "0.1uF" H 6665 4455 50  0000 L CNN
 F 2 "" H 6588 4350 50  0001 C CNN
 F 3 "~" H 6550 4500 50  0001 C CNN
@@
 AR Path="/6219DADC/6211E3F9" Ref="R?"  Part="1"
 F 0 "R?" V 8800 4900 50  0000 C CNN
-F 1 "3300" V 8900 4900 50  0000 C CNN
+F 1 "2800" V 8900 4900 50  0000 C CNN
 F 2 "" V 8830 4900 50  0001 C CNN
 F 3 "~" H 8900 4900 50  0001 C CNN

Commit message: saving
Parts:
- gave numbers to parts that had none: 83

Commit message: schematic started
Parts:
- C11, C12, C13, C14, C15, C16, C17, C18, C19, C20, C21, C22, C23, C24, C25, C26: footprint (none) -> Capacitor_SMD:C_0603_1608Metric_Pad1.08x0.95mm_HandSolder
- D10, D11, D12, D13, D5, D6, D7, D8, D9: footprint (none) -> LED_SMD:LED_0603_1608Metric_Pad1.05x0.95mm_HandSolder
- F1, F2, F3, F4, F5, F6, F7, F8, F9: footprint (none) -> MRDT_Passives:ATC_Fuse_Block
- R10, R13, R15, R16, R17, R18, R19, R20, R21, R22, R26, R3, R4, R5, R6, R7, R8: footprint (none) -> Resistor_SMD:R_0603_1608Metric_Pad0.98x0.95mm_HandSolder
- R11, R12, R14, R23, R24, R25, R27, R9: footprint (none) -> Resistor_SMD:R_2512_6332Metric_Pad1.40x3.35mm_HandSolder
- U11, U12, U13, U14, U3, U4, U5, U6: footprint (none) -> Package_SO:SOIC-8_3.9x4.9mm_P1.27mm

Commit message: Back to TEENSY
Parts:
- Q1, Q2, Q3, Q4, Q5, Q6, Q7, Q8: value BUK7M8R0-40EX -> BUK7S2R0-40HJ
Changed lines of the file:
@@
 AR Path="/6219DADC/621D64AC" Ref="Q?"  Part="1"
 F 0 "Q6" H 8655 5596 50  0000 L CNN
-F 1 "BUK7M8R0-40EX" H 8250 5300 50  0000 L CNN
+F 1 "BUK7S2R0-40HJ" H 8250 5300 50  0000 L CNN
 F 2 "Package_TO_SOT_SMD:LFPAK33" H 8650 5475 50  0001 L CIN
 F 3 "https://assets.nexperia.com/documents/data-sheet/BUK7M8R0-40E.pdf" V 8450 5550 50  0001 L CNN
@@
 AR Path="/6219DADC/621D6D6B" Ref="Q?"  Part="1"
 F 0 "Q8" H 8955 2646 50  0000 L CNN
-F 1 "BUK7M8R0-40EX" H 8550 2350 50  0000 L CNN
+F 1 "BUK7S2R0-40HJ" H 8550 2350 50  0000 L CNN
 F 2 "Package_TO_SOT_SMD:LFPAK33" H 8950 2525 50  0001 L CIN
 F 3 "https://assets.nexperia.com/documents/data-sheet/BUK7M8R0-40E.pdf" V 8750 2600 50  0001 L CNN
@@
 AR Path="/6219DADC/621D838D" Ref="Q?"  Part="1"
 F 0 "Q7" H 8705 1196 50  0000 L CNN
-F 1 "BUK7M8R0-40EX" H 8300 900 50  0000 L CNN
+F 1 "BUK7S2R0-40HJ" H 8300 900 50  0000 L CNN
 F 2 "Package_TO_SOT_SMD:LFPAK33" H 8700 1075 50  0001 L CIN
 F 3 "https://assets.nexperia.com/documents/data-sheet/BUK7M8R0-40E.pdf" V 8500 1150 50  0001 L CNN
@@
 AR Path="/6219DADC/621DC735" Ref="Q?"  Part="1"
 F 0 "Q1" H 3305 1296 50  0000 L CNN
-F 1 "BUK7M8R0-40EX" H 2900 1000 50  0000 L CNN
+F 1 "BUK7S2R0-40HJ" H 2900 1000 50  0000 L CNN
 F 2 "Package_TO_SOT_SMD:LFPAK33" H 3300 1175 50  0001 L CIN
 F 3 "https://assets.nexperia.com/documents/data-sheet/BUK7M8R0-40E.pdf" V 3100 1250 50  0001 L CNN
@@
 AR Path="/6219DADC/621E2A9C" Ref="Q?"  Part="1"
 F 0 "Q2" H 3405 2896 50  0000 L CNN
-F 1 "BUK7M8R0-40EX" H 3000 2600 50  0000 L CNN
+F 1 "BUK7S2R0-40HJ" H 3000 2600 50  0000 L CNN
 F 2 "Package_TO_SOT_SMD:LFPAK33" H 3400 2775 50  0001 L CIN
 F 3 "https://assets.nexperia.com/documents/data-sheet/BUK7M8R0-40E.pdf" V 3200 2850 50  0001 L CNN
@@
 AR Path="/6219DADC/621ECB20" Ref="Q?"  Part="1"
 F 0 "Q3" H 3505 4546 50  0000 L CNN
-F 1 "BUK7M8R0-40EX" H 3100 4250 50  0000 L CNN
+F 1 "BUK7S2R0-40HJ" H 3100 4250 50  0000 L CNN
 F 2 "Package_TO_SOT_SMD:LFPAK33" H 3500 4425 50  0001 L CIN
 F 3 "https://assets.nexperia.com/documents/data-sheet/BUK7M8R0-40E.pdf" V 3300 4500 50  0001 L CNN
@@
 AR Path="/6219DADC/621FB435" Ref="Q?"  Part="1"
 F 0 "Q4" H 3655 6396 50  0000 L CNN
-F 1 "BUK7M8R0-40EX" H 3250 6100 50  0000 L CNN
+F 1 "BUK7S2R0-40HJ" H 3250 6100 50  0000 L CNN
 F 2 "Package_TO_SOT_SMD:LFPAK33" H 3650 6275 50  0001 L CIN
 F 3 "https://assets.nexperia.com/documents/data-sheet/BUK7M8R0-40E.pdf" V 3450 6350 50  0001 L CNN
@@
 AR Path="/6219DADC/6211E3F1" Ref="Q?"  Part="1"
 F 0 "Q5" H 8555 4196 50  0000 L CNN
-F 1 "BUK7M8R0-40EX" H 8150 3900 50  0000 L CNN
+F 1 "BUK7S2R0-40HJ" H 8150 3900 50  0000 L CNN
 F 2 "Package_TO_SOT_SMD:LFPAK33" H 8550 4075 50  0001 L CIN
 F 3 "https://assets.nexperia.com/documents/data-sheet/BUK7M8R0-40E.pdf" V 8350 4150 50  0001 L CNN

Commit message: Somewhat completed schematic
did stuff
Parts:
- U10, U15, U16, U17, U18, U7, U8, U9: symbol MRDT_ICs:INA281 -> PackVoltage_2022_Rev1-rescue:INA281-MRDT_ICs
- U11, U12, U13, U14, U3, U4, U5, U6: symbol MRDT_ICs:LT1910 -> PackVoltage_2022_Rev1-rescue:LT1910-MRDT_ICs
Connections:
- net 5V renamed +5V

Commit message: fixed schematic issues - renamed ports, removed unnecessary ports, corrected footprint assignments; began layout - created circuits for most ports, most components placed
Parts:
- added C25: 0.1uF, Capacitor_SMD:C_0603_1608Metric_Pad1.08x0.95mm_HandSolder, symbol Device:C
- added C26: 10uF, Capacitor_SMD:C_0603_1608Metric_Pad1.08x0.95mm_HandSolder, symbol Device:C
- added D14: LED, LED_SMD:LED_0603_1608Metric_Pad1.05x0.95mm_HandSolder, symbol Device:LED
- added F10: 20, MRDT_Passives:ATC_Fuse_Block, symbol Device:Fuse
- added Q9: BUK7S2R0-40HJ, Package_TO_SOT_SMD:LFPAK33, symbol Transistor_FET:BUK7M8R0-40EX
- added R28: 5.1k, Resistor_SMD:R_0603_1608Metric_Pad0.98x0.95mm_HandSolder, symbol Device:R
- added R29: 2800, Resistor_SMD:R_0603_1608Metric_Pad0.98x0.95mm_HandSolder, symbol Device:R
- added U19: LT1910, Package_SO:SOIC-8_3.9x4.9mm_P1.27mm, symbol MRDT_ICs:LT1910
- R11, R12, R14, R23, R24, R25, R27, R9: value .0025 -> .0015
- U10, U15, U16, U17, U18, U7, U8, U9: symbol PackVoltage_2022_Rev1-rescue:INA281-MRDT_ICs -> MRDT_ICs:INA281
- U11, U12, U13, U14, U3, U4, U5, U6: symbol PackVoltage_2022_Rev1-rescue:LT1910-MRDT_ICs -> MRDT_ICs:LT1910
- renumbered C12 to C10, C13 to C11, C14 to C12, C15 to C13, C16 to C14, C17 to C15, C18 to C16, C19 to C17, C20 to C18, C21 to C19, C22 to C20, C23 to C21, C24 to C22, C25 to C23, C26 to C24, C11 to C9
Connections:
- net +5V: now also R28.2
- net Anderson_Spare: now also Q9.1 (S), Q9.2 (S), Q9.3 (S), R29.2; no longer R24.2, U16.4 (-)
- net Driver_Spare: now also U19.4 (IN); no longer U12.4 (IN)
- net GND: now also C25.2, C26.2, D14.1 (K), U19.1 (GND)
- net PV: now also F10.1
- net Current_Sensor_Spare renamed Current_Sensor_SpareMotor
- new net: R28.1, U19.3 (FAULT)
- new net: C25.1, U19.2 (TIMER)
- new net: Q9.4 (G), U19.5 (GATE)
- new net: C26.1, F10.2, Q9.5 (D), U19.6 (SENSE), U19.8 (V+)
- new net: D14.2 (A), R29.1
- new net Anderson_SpareMotor: R24.2, U16.4 (-)
- new net Driver_SpareMotor: U12.4 (IN)
