File: Hardware/2023 Powerboard/2023 Powerboard.kicad_pcb (KiCad board)
At the start: 2 copper layers, 153 parts, among them J1 RJ45_LED_Shielded, J2 6P6C, Q1 BSS138, Q10 BSS138, Q11 QM6015D, Q12 IRF7606PBF, Q13 BSS138, Q14 QM6015D, Q15 BSS138, Q16 IRF7606PBF, Q17 BSS138, Q18 QM6015D, Q19 BSS138, Q2 BSS138, Q20 BSS138, Q21 IRF7606PBF, Q22 QM6015D, Q23 BSS138, Q24 BSS138, Q25 IRF7606PBF, Q26 QM6015D, Q27 BSS138, Q28 BSS138, Q29 IRF7606PBF, Q3 QM6015D, Q30 QM6015D, Q31 BSS138, Q32 QM6015D, Q4 IRF7606PBF, Q5 BSS138, Q6 BSS138, Q7 QM6015D, Q8 IRF7606PBF, Q9 BSS138, U1 3V3, U2 Teensy4.1_DEV-16771

Commit message: Added Fuses, Potential Layout for Connector 1
Parts:
- added F17: 5, MRDT_Passives:ATC_Fuse_Block, F.Cu at (341.2, 91.8)
- added F18: 1, MRDT_Passives:ATC_Fuse_Block, F.Cu at (357.1, 91.8)
- moved D2 58.6 mm to (66.5, 61.7), turned to 90 degrees
- moved R2 48.0 mm to (68.8, 64.0), turned to -90 degrees
- moved R1 42.0 mm to (71.6, 63.1), turned to 180 degrees
- moved R6 41.3 mm to (66.5, 58.2), turned to -90 degrees
- moved F14 13.4 mm to (324.0, 91.4), turned to 90 degrees
- moved Q1 12.4 mm to (68.8, 67.8), turned to 90 degrees
- moved F1 11.6 mm to (73.5, 81.9)
- moved Q3 8.38 mm to (71.1, 56.6), turned to 90 degrees
- moved Conn1 3.75 mm to (71.8, 46.4), turned to -90 degrees
Connections:
- Conn17 pad 4: PV -> POE
- Conn18 pad 4: PV -> Net Switch
Routing:
- net Net-(Q3-Pad1): track 0.00 -> 4.15 mm
- net Net-(Q1-Pad3): track 0.00 -> 1.96 mm
- net Net-(D2-Pad2): track 0.00 -> 1.77 mm

Commit message: Placed Power Vias, Set Up Oki and Power Filter
Parts:
- moved C2 482.9 mm to (27.7, 120.9), turned to 180 degrees
- moved C3 482.8 mm to (27.7, 76.7), turned to 180 degrees
- moved C5 481.9 mm to (27.7, 106.2), turned to 180 degrees
- moved C1 477.5 mm to (27.9, 91.4), turned to 180 degrees
- moved D4 471.1 mm to (22.7, 59.4)
- moved D5 466.5 mm to (22.7, 67.1)
- moved V1 445.1 mm to (31.6, 42.2)
- moved D1 435.1 mm to (31.0, 137.7), turned to 90 degrees
- moved R5 434.4 mm to (31.0, 134.1), turned to 90 degrees
- moved C4 432.1 mm to (33.0, 134.1), turned to -90 degrees
- moved C6 425.7 mm to (45.2, 134.1), turned to -90 degrees
- moved D7 423.9 mm to (47.2, 137.7), turned to 90 degrees
- moved R12 423.6 mm to (47.2, 134.1), turned to -90 degrees
- moved U1 416.0 mm to (36.6, 133.6)
- moved V2 140.0 mm to (391.2, 47.2)
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
Commit message: MOSFET Layouts
Parts:
- Conn1, Conn10, Conn11, Conn12, Conn13, Conn14, Conn15, Conn16, Conn17, Conn18, Conn2, Conn3, Conn4, Conn5, Conn6, Conn7, Conn8, Conn9: moved to B.Cu
- moved V5 432.4 mm to (24.9, 30.7), turned to 90 degrees
- moved V3 417.1 mm to (24.9, 130.9), turned to 180 degrees
- moved V6 166.3 mm to (347.4, 30.7)
- moved V4 112.0 mm to (347.4, 130.9), turned to -90 degrees
- moved U2 84.4 mm to (170.7, 115.8)
- moved D12 80.2 mm to (225.3, 56.6), turned to 90 degrees
- moved D18 80.0 mm to (269.0, 56.4), turned to 90 degrees
- moved D16 76.4 mm to (254.5, 56.6), turned to 90 degrees
- moved D10 75.7 mm to (212.1, 56.4), turned to 90 degrees
- moved C7 75.4 mm to (304.3, 58.2), turned to -90 degrees
- moved D14 74.7 mm to (239.8, 56.6), turned to 90 degrees
- moved D20 74.2 mm to (153.2, 61.2), turned to 90 degrees
- moved J1 72.0 mm to (310.4, 32.2), turned to 180 degrees
- moved D8 71.2 mm to (199.6, 56.4), turned to 90 degrees
- moved R34 70.6 mm to (239.8, 53.1), turned to -90 degrees
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Other:
- board outline added: 338.6 x 116.4 mm

Commit message: stuff
Parts:
- moved F17 14.6 mm to (279.5, 67.4)
- moved F8 14.6 mm to (218.8, 67.4)
- moved F6 14.6 mm to (204.5, 67.4)
- moved F10 14.6 mm to (233.5, 67.4)
- moved F14 14.5 mm to (262.6, 67.5)
- moved F18 14.5 mm to (292.3, 67.5)
- moved F4 14.5 mm to (190.9, 67.5)
- moved F12 14.5 mm to (248.2, 67.5)
- moved F2 14.4 mm to (177.0, 67.5)
- moved D9 13.4 mm to (80.8, 48.7)
- moved R19 13.4 mm to (80.8, 45.2)
- moved D6 13.4 mm to (67.9, 48.7)
- moved R13 13.4 mm to (67.9, 45.0)
- moved D2 13.3 mm to (55.8, 48.6)
- moved R6 13.3 mm to (55.8, 45.1)
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Routing:
- net M2: track 0.00 -> 5.31 mm
- net M5: track 0.00 -> 5.30 mm
- net M1: track 0.00 -> 5.29 mm
- net Spare: track 0.00 -> 5.28 mm
- net MS: track 0.00 -> 5.27 mm
- net Aux: track 0.00 -> 5.26 mm
- net M4: track 0.00 -> 5.25 mm
- net M3: track 0.00 -> 5.23 mm
- net M6: track 0.00 -> 5.22 mm
- net Net-(Q29-Pad4): track 0.00 -> 4.46 mm
- net Net-(Q11-Pad1): track 0.00 -> 4.29 mm
- net Net-(Q22-Pad1): track 0.00 -> 4.29 mm
- net Net-(Q25-Pad4): track 0.00 -> 4.24 mm
- net Net-(Q21-Pad4): track 0.00 -> 4.24 mm
- net Net-(Q4-Pad4): track 0.00 -> 4.24 mm
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- added copper zone on F.Cu, net Aux
- added copper zone on F.Cu, net BB
- added copper zone on F.Cu, net Cam
- added copper zone on F.Cu, net Drive
- added copper zone on F.Cu, net Gimbal
- added copper zone on F.Cu, net LCSpare
- added copper zone on F.Cu, net M1
- added copper zone on F.Cu, net M2
- added copper zone on F.Cu, net M3
- added copper zone on F.Cu, net M4
- added copper zone on F.Cu, net M5
- added copper zone on F.Cu, net M6
- added copper zone on F.Cu, net MM
- added copper zone on F.Cu, net MS
- added copper zone on F.Cu, net Nav
- added copper zone on F.Cu, net Net Switch
- added copper zone on F.Cu, net Net-(F1-Pad2)
- added copper zone on F.Cu, net Net-(F10-Pad2)
- added copper zone on F.Cu, net Net-(F11-Pad2)
- added copper zone on F.Cu, net Net-(F12-Pad2)
- added copper zone on F.Cu, net Net-(F13-Pad2)
- added copper zone on F.Cu, net Net-(F14-Pad2)
- added copper zone on F.Cu, net Net-(F15-Pad2)
- added copper zone on F.Cu, net Net-(F2-Pad2)
- added copper zone on F.Cu, net Net-(F3-Pad2)
- added copper zone on F.Cu, net Net-(F4-Pad2)
- added copper zone on F.Cu, net Net-(F5-Pad2)
- added copper zone on F.Cu, net Net-(F6-Pad2)
- added copper zone on F.Cu, net Net-(F7-Pad2)
- added copper zone on F.Cu, net Net-(F8-Pad2)
- added copper zone on F.Cu, net Net-(F9-Pad2)
- added copper zone on F.Cu, net POE
- added copper zone on F.Cu, net Spare

Commit message: Traces and silkscreen
Parts:
- added G***: LOGO, MRDT_Silkscreens:0_MRDT_Logo_60mm, F.Cu at (323.6, 81.8)
- moved D1 161.4 mm to (238.1, 118.9), turned to 180 degrees
- moved R5 158.0 mm to (234.5, 118.9), turned to 180 degrees
- moved C4 155.9 mm to (234.5, 116.9), turned to 0 degrees
- moved U1 151.8 mm to (234.0, 113.3), turned to 90 degrees
- moved D7 145.7 mm to (238.1, 102.7), turned to 180 degrees
- moved C6 143.8 mm to (234.5, 104.7), turned to 0 degrees
- moved R12 141.9 mm to (234.5, 102.7), turned to 0 degrees
- moved U2 10.4 mm to (170.4, 105.4)
- moved V2 5.14 mm to (339.3, 42.1)
Routing:
- net CTLM1: track 0.00 -> 187.8 mm, vias 0 -> 2
- net CTLM2: track 0.00 -> 172.1 mm, vias 0 -> 2
- net CTLM3: track 0.00 -> 156.8 mm, vias 0 -> 2
- net CTLLCSpare: track 0.00 -> 146.5 mm, vias 0 -> 2
- net CTLM4: track 0.00 -> 141.1 mm, vias 0 -> 2
- net CTLBB: track 0.00 -> 129.5 mm, vias 0 -> 2
- net CTLDrive: track 0.00 -> 128.1 mm, vias 0 -> 2
- net CTLM5: track 0.00 -> 123.8 mm, vias 0 -> 2
- net CTLCam: track 0.00 -> 122.4 mm, vias 0 -> 4
- net CTLNav: track 0.00 -> 112.2 mm, vias 0 -> 2
- net CTLGimbal: track 0.00 -> 112.1 mm, vias 0 -> 2
- net CTLMM: track 0.00 -> 111.3 mm, vias 0 -> 4
- net CTLM6: track 0.00 -> 108.6 mm, vias 0 -> 2
- net CTLSpare: track 0.00 -> 108.2 mm, vias 0 -> 4
- net +3V3: track 0.00 -> 105.7 mm
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- added copper zone on F.Cu, net GND
- added copper zone on F.Cu, net Net-(F16-Pad2)
- added copper zone on B.Cu, net PV
Other:
- board text added: "Power Board, Rev 1.0 Mars Rover Design Team Missouri S&T, 2023 Natasha Cox, Garrett McEntire, Sophia Strathman"

Commit message: Layout edits
Parts:
- removed G***: LOGO, MRDT_Silkscreens:0_MRDT_Logo_60mm
- moved Conn17 236.1 mm to (43.9, 34.5)
- moved Conn18 236.1 mm to (57.1, 34.5)
- moved F17 236.1 mm to (43.4, 67.6)
- moved F18 236.1 mm to (56.3, 67.6)
- moved Conn1 220.3 mm to (280.2, 34.5)
- moved D2 220.3 mm to (276.2, 48.6)
- moved Q1 220.3 mm to (278.6, 56.0)
- moved Q3 220.3 mm to (280.9, 44.8)
- moved R2 220.3 mm to (278.6, 52.2)
- moved R6 220.3 mm to (276.2, 45.1)
- moved F1 220.3 mm to (283.2, 70.7)
- moved R1 220.3 mm to (281.4, 51.3)
- moved Q7 194.2 mm to (266.8, 44.9)
- moved R8 194.2 mm to (267.2, 51.4)
- moved Conn2 194.2 mm to (266.2, 34.5)
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Routing:
- net CTLCam: track 122.4 -> 34.4 mm, vias 4 -> 0
- net CTLSpare: track 108.2 -> 31.7 mm, vias 4 -> 0
- net CTLMM: track 111.3 -> 44.2 mm, vias 4 -> 2
- net CTLM1: track 187.8 -> 123.0 mm
- net CTLDrive: track 128.1 -> 67.3 mm
- net CTLM2: track 172.1 -> 111.4 mm
- net CTLM3: track 156.8 -> 99.8 mm
- net CTLGimbal: track 112.1 -> 55.9 mm
- net CTLAux: track 98.3 -> 42.9 mm, vias 4 -> 2
- net CTLM4: track 141.1 -> 88.6 mm
- net CTLM5: track 123.8 -> 77.1 mm
- net CTLM6: track 108.6 -> 65.8 mm
- net CTLMS: track 92.7 -> 54.4 mm
- net GND: track 0.00 -> 35.7 mm
- net CTLLCSpare: track 146.5 -> 111.9 mm
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- added copper zone on B.Cu, net GND
- removed copper zone on B.Cu, net PV
Other:
- board text added: "Multimedia"

Commit message: Finished Layout
Parts:
- moved U2 108.4 mm to (238.6, 168.4)
- moved C1 94.3 mm to (56.4, 146.1)
- moved C2 94.3 mm to (85.9, 146.3)
- moved C3 94.3 mm to (41.7, 146.3)
- moved C5 94.3 mm to (71.1, 146.3)
- moved D4 94.3 mm to (24.4, 151.3)
- moved D5 94.3 mm to (32.0, 151.3)
- moved D7 89.0 mm to (197.6, 175.8), turned to 0 degrees
- moved R12 88.6 mm to (201.2, 175.8), turned to 180 degrees
- moved C6 84.6 mm to (201.2, 173.7), turned to 180 degrees
- moved V4 73.8 mm to (343.9, 170.0)
- moved U1 67.3 mm to (202.1, 165.1), turned to -90 degrees
- moved C7 67.1 mm to (327.1, 152.9), turned to 0 degrees
- moved J1 67.1 mm to (353.0, 159.0)
- moved J2 67.1 mm to (326.1, 165.1)
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Routing:
- net CTLLCSpare: track 111.9 -> 259.4 mm
- net CTLCam: track 34.4 -> 175.6 mm, vias 0 -> 1
- net CTLSpare: track 31.7 -> 171.8 mm, vias 0 -> 1
- net CTLDrive: track 67.3 -> 204.9 mm, vias 2 -> 1
- net CTLBB: track 126.8 -> 264.3 mm
- net CTLMM: track 44.2 -> 181.7 mm, vias 2 -> 1
- net CTLGimbal: track 55.9 -> 193.2 mm, vias 2 -> 1
- net CTLNav: track 143.1 -> 277.1 mm
- net CTLAux: track 42.9 -> 156.7 mm, vias 2 -> 1
- net CTLMS: track 54.4 -> 140.9 mm, vias 2 -> 1
- net CTLM6: track 65.8 -> 134.5 mm, vias 2 -> 1
- net CTLM5: track 77.1 -> 118.5 mm, vias 2 -> 1
- net Net-(C7-Pad2): track 0.00 -> 36.7 mm
- net GND: track 35.7 -> 0.00 mm
- net PV: track 5.76 -> 27.4 mm
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- added copper zone on F.Cu, net PV
Other:
- board size 338.6 x 116.4 mm -> 336.6 x 163.8 mm
- board text added: "AUX"
- board text added: "BB"
- board text added: "CAM"
- board text added: "DRV"
- board text added: "GIM"
- board text added: "GND"
- board text added: "M1"
- board text added: "M2"
- board text added: "M3"
- board text added: "M4"
- board text added: "M5"
- board text added: "M6"
- board text added: "MM"
- board text added: "MS"
- board text added: "NAV"
- board text added: "NET"
- board text added: "POE"
- board text added: "PV"
- board text added: "S1A"
- board text added: "S20A"
- board text removed: "Multimedia"

Commit message: Layout Review Changes
Parts:
- added D21: Green, LED_SMD:LED_0603_1608Metric_Pad1.05x0.95mm_HandSolder, F.Cu at (49.9, 43.0)
- added D22: Green, LED_SMD:LED_0603_1608Metric_Pad1.05x0.95mm_HandSolder, F.Cu at (62.6, 43.0)
- added R51: 3k, Resistor_SMD:R_0603_1608Metric_Pad0.98x0.95mm_HandSolder, F.Cu at (49.0, 40.4)
- added R52: 3k, Resistor_SMD:R_0603_1608Metric_Pad0.98x0.95mm_HandSolder, F.Cu at (61.7, 40.4)
- R12: value 130 -> 120
- moved D7 17.6 mm to (195.6, 158.2)
- moved R12 17.6 mm to (199.1, 158.2)
- moved C6 17.6 mm to (199.1, 156.2)
- moved U1 17.6 mm to (200.0, 147.6)
- moved C4 13.3 mm to (203.7, 148.5), turned to -90 degrees
- moved R5 11.8 mm to (205.5, 148.5), turned to 90 degrees
- moved D1 10.9 mm to (205.5, 152.0), turned to 90 degrees
- moved U2 10.2 mm to (238.6, 158.2)
Connections:
- U2 pad 13: CTLNav -> unconnected-(U2-Pad13)
- U2 pad 14: CTLBB -> unconnected-(U2-Pad14)
- U2 pad 15: CTLLCSpare -> unconnected-(U2-Pad15)
- U2 pad 24: unconnected-(U2-Pad24) -> CTLLCSpare
- U2 pad 25: unconnected-(U2-Pad25) -> CTLBB
- U2 pad 26: unconnected-(U2-Pad26) -> CTLNav
Routing:
- net CTLNav: track 277.1 -> 3.08 mm, vias 2 -> 1
- net CTLBB: track 264.3 -> 3.32 mm, vias 2 -> 1
- net CTLLCSpare: track 259.4 -> 3.56 mm, vias 2 -> 1
- net PV: track 27.4 -> 5.53 mm
- net CTLDrive: track 204.9 -> 194.7 mm
- net CTLSpare: track 171.8 -> 161.6 mm
- net CTLM5: track 118.5 -> 108.4 mm
- net CTLM4: track 106.9 -> 96.7 mm
- net CTLM3: track 115.8 -> 105.6 mm
- net CTLM2: track 121.1 -> 110.9 mm
- net CTLGimbal: track 193.2 -> 183.0 mm
- net CTLCam: track 175.6 -> 165.5 mm
- net CTLM6: track 134.5 -> 124.3 mm
- net CTLM1: track 136.1 -> 125.9 mm
- net CTLMS: track 140.9 -> 130.7 mm
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Other:
- board text added: "3V3"
