File: Hardware/2023 Powerboard/2023 Powerboard.kicad_sch (KiCad schematic)
At the start: 17 parts

Commit message: finished schematic
Parts:
- added Conn1, Conn10, Conn11, Conn12, Conn13, Conn14, Conn15, Conn16, Conn17, Conn18, Conn2, Conn3, Conn4, Conn5, Conn6, Conn7, Conn8, Conn9: AndersonPP, symbol MRDT_Connectors:AndersonPP
- added D1, D10, D11, D12, D13, D14, D15, D16, D17, D18, D19, D2, D20, D3, D6, D8, D9: Green, symbol Device:LED
- added Q1, Q10, Q13, Q15, Q17, Q19, Q2, Q20, Q23, Q24, Q27, Q28, Q31, Q5, Q6, Q9: BSS138, Package_TO_SOT_SMD:SOT-23, symbol Transistor_FET:BSS138
- added Q11, Q14, Q18, Q22, Q26, Q3, Q30, Q32, Q7: QM6015D, Package_TO_SOT_SMD:TO-252-2, symbol Transistor_FET:QM6015D
- added Q12, Q16, Q21, Q25, Q29, Q4, Q8: IRF7606PBF, Package_SO:MSOP-8_3x3mm_P0.65mm, symbol Transistor_FET:IRF7606PBF
- added R1, R10, R15, R17, R21, R23, R26, R3, R30, R32, R36, R38, R42, R44, R48, R8: 3.3k, symbol Device:R
- added R11, R16, R18, R2, R22, R24, R27, R31, R33, R37, R39, R4, R43, R45, R49, R9: 6.8k, symbol Device:R
- added R13, R14, R19, R20, R25, R28, R29, R34, R35, R40, R41, R46, R47, R5, R50, R6, R7: 3k, symbol Device:R
- gave numbers to parts that had none: 17
Connections:
- net GND: now also Conn1.1 (GND), Conn10.1 (GND), Conn11.1 (GND), Conn12.1 (GND), Conn13.1 (GND), Conn14.1 (GND), Conn15.1 (GND), Conn16.1 (GND), Conn17.1 (GND), Conn18.1 (GND), Conn2.1 (GND), Conn3.1 (GND), Conn4.1 (GND), Conn5.1 (GND), Conn6.1 (GND), Conn7.1 (GND), Conn8.1 (GND), Conn9.1 (GND), D1.1 (K), D10.1 (K), D11.1 (K), D12.1 (K), D13.1 (K), D14.1 (K), D15.1 (K), D16.1 (K), D17.1 (K), D18.1 (K), D19.1 (K), D2.1 (K), D20.1 (K), D3.1 (K), D6.1 (K), D8.1 (K), D9.1 (K), Q1.2 (S), Q10.2 (S), Q13.2 (S), Q15.2 (S), Q17.2 (S), Q19.2 (S), Q2.2 (S), Q20.2 (S), Q23.2 (S), Q24.2 (S), Q27.2 (S), Q28.2 (S), Q31.2 (S), Q5.2 (S), Q6.2 (S), Q9.2 (S)
- net PV: now also Conn17.4 (PV+), Conn18.4 (PV+), Q11.3 (S), Q12.1 (S), Q12.2 (S), Q12.3 (S), Q14.3 (S), Q16.1 (S), Q16.2 (S), Q16.3 (S), Q18.3 (S), Q21.1 (S), Q21.2 (S), Q21.3 (S), Q22.3 (S), Q25.1 (S), Q25.2 (S), Q25.3 (S), Q26.3 (S), Q29.1 (S), Q29.2 (S), Q29.3 (S), Q3.3 (S), Q30.3 (S), Q32.3 (S), Q4.1 (S), Q4.2 (S), Q4.3 (S), Q7.3 (S), Q8.1 (S), Q8.2 (S), Q8.3 (S), R1.1, R10.1, R15.1, R17.1, R21.1, R23.1, R26.1, R3.1, R30.1, R32.1, R36.1, R38.1, R42.1, R44.1, R48.1, R5.2, R8.1
- net TM1: now reaches U2.0 (RX1)
- net TM1: now also Q1.1 (G)
- net TM2: now reaches U2.1 (TX1)
- net TM2: now also Q5.1 (G)
- net TMM: now reaches U2.10 (CS1)
- net TMM: now also Q6.1 (G)
- net TGimbal: now reaches U2.11 (MOSI)
- net TGimbal: now also Q10.1 (G)
- net TDrive: now reaches U2.12 (MISO)
- net TDrive: now also Q15.1 (G)
- net TNav: now reaches U2.13 (SCK)
- net TNav: now also Q19.1 (G)
- net TBB: now reaches U2.14 (A0)
- net TBB: now also Q23.1 (G)
- net TLSpare: now reaches U2.15 (A1)
- net TLSpare: now also Q27.1 (G)
- net TM3: now reaches U2.2 (OUT2)
- net TM3: now also Q9.1 (G)
- net TM4: now reaches U2.3 (LRCLK2)
- net TM4: now also Q13.1 (G)
- net TM5: now reaches U2.4 (BCLK2)
- net TM5: now also Q17.1 (G)
- net TM6: now reaches U2.5 (IN2)
- net TM6: now also Q20.1 (G)
- net TMS: now reaches U2.6 (OUT1D)
- net TMS: now also Q24.1 (G)
- net TAux: now reaches U2.7 (RX2)
- net TAux: now also Q28.1 (G)
- net TSpare: now reaches U2.8 (TX2)
- net TSpare: now also Q31.1 (G)
- net TCam: now reaches U2.9 (OUT1C)
- net TCam: now also Q2.1 (G)
- new net: Q22.1 (G), R32.2, R33.1
- new net: Q20.3 (D), R33.2
- new net: D2.2 (A), R6.2
- new net: D6.2 (A), R13.2
- new net: Q16.4 (G), R23.2, R24.1
- new net: Q30.1 (G), R44.2, R45.1
- new net: Q2.3 (D), R4.2
- new net: Q8.4 (G), R10.2, R11.1
- new net: Q23.3 (D), R37.2
- new net: Q29.4 (G), R42.2, R43.1
- new net: Q27.3 (D), R43.2
- new net: Q32.1 (G), R48.2, R49.1
- new net: Q3.1 (G), R1.2, R2.1
- new net: D1.2 (A), R5.1
- new net: D10.2 (A), R20.2
- new net: D15.2 (A), R35.2
- new net: D16.2 (A), R40.2
- new net: Q11.1 (G), R15.2, R16.1
- new net: D14.2 (A), R34.2
- new net: Q28.3 (D), R45.2
- new net: D12.2 (A), R28.2
- new net: Q14.1 (G), R21.2, R22.1
- new net: Q13.3 (D), R22.2
- new net: Q12.4 (G), R17.2, R18.1
- new net: Q31.3 (D), R49.2
- new net: Q7.1 (G), R8.2, R9.1
- new net: D20.2 (A), R50.2
- new net: Q17.3 (D), R27.2
- new net: Q10.3 (D), R18.2
- new net: Q24.3 (D), R39.2
- new net: Q19.3 (D), R31.2
- new net: D19.2 (A), R47.2
- new net: Q15.3 (D), R24.2
- new net: D11.2 (A), R25.2
- new net: Q26.1 (G), R38.2, R39.1
- new net: Q4.4 (G), R3.2, R4.1
- new net: D17.2 (A), R41.2
- new net: Q5.3 (D), R9.2
- new net: D18.2 (A), R46.2
- new net: Q18.1 (G), R26.2, R27.1
- new net: Q25.4 (G), R36.2, R37.1
- new net: D13.2 (A), R29.2
- new net: D8.2 (A), R14.2
- new net: D3.2 (A), R7.2
- new net: D9.2 (A), R19.2
- new net: Q6.3 (D), R11.2
- new net: Q21.4 (G), R30.2, R31.1
- new net: Q1.3 (D), R2.2
- new net: Q9.3 (D), R16.2
- new net Aux: Conn8.4 (PV+), Q30.2 (D), R47.1
- new net BB: Conn15.4 (PV+), Q25.5 (D), Q25.6 (D), Q25.7 (D), Q25.8 (D), R40.1
- new net Cam: Conn10.4 (PV+), Q4.5 (D), Q4.6 (D), Q4.7 (D), Q4.8 (D), R7.1
- new net Drive: Conn13.4 (PV+), Q16.5 (D), Q16.6 (D), Q16.7 (D), Q16.8 (D), R28.1
- new net Gimbal: Conn12.4 (PV+), Q12.5 (D), Q12.6 (D), Q12.7 (D), Q12.8 (D), R20.1
- new net LSpare: Conn16.4 (PV+), Q29.5 (D), Q29.6 (D), Q29.7 (D), Q29.8 (D), R46.1
- new net M1: Conn1.4 (PV+), Q3.2 (D), R6.1
- new net M2: Conn2.4 (PV+), Q7.2 (D), R13.1
- new net M3: Conn3.4 (PV+), Q11.2 (D), R19.1
- new net M4: Conn4.4 (PV+), Q14.2 (D), R25.1
- new net M5: Conn5.4 (PV+), Q18.2 (D), R29.1
- new net M6: Conn6.4 (PV+), Q22.2 (D), R35.1
- new net MM: Conn11.4 (PV+), Q8.5 (D), Q8.6 (D), Q8.7 (D), Q8.8 (D), R14.1
- new net MS: Conn7.4 (PV+), Q26.2 (D), R41.1
- new net Nav: Conn14.4 (PV+), Q21.5 (D), Q21.6 (D), Q21.7 (D), Q21.8 (D), R34.1
- new net Spare: Conn9.4 (PV+), Q32.2 (D), R50.1
- no-connect marks 3 -> 42
Other:
- note added: "3V3 Oki"
- note added: ";)"
- note added: "Andersons"
- note added: "High Current"
- note added: "Label?"
- note added: "Medium/Low Current"
- note added: "Teensy"
- moved on the sheet: C1, C2, C3, C4, C5, C6, C7, D4, D5, D7, J1, J2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

Commit message: Added Fuses
Parts:
- added F1, F11, F13, F15, F16, F3, F5, F7, F9: 20, symbol Device:Fuse
- added F10, F12, F14, F8: 1, symbol Device:Fuse
- added F2, F4, F6: 5, symbol Device:Fuse
Connections:
- net PV: now also F1.1, F10.1, F11.1, F12.1, F13.1, F14.1, F15.1, F16.1, F2.1, F3.1, F4.1, F5.1, F6.1, F7.1, F8.1, F9.1; no longer Q11.3 (S), Q12.1 (S), Q12.2 (S), Q12.3 (S), Q14.3 (S), Q16.1 (S), Q16.2 (S), Q16.3 (S), Q18.3 (S), Q21.1 (S), Q21.2 (S), Q21.3 (S), Q22.3 (S), Q25.1 (S), Q25.2 (S), Q25.3 (S), Q26.3 (S), Q29.1 (S), Q29.2 (S), Q29.3 (S), Q3.3 (S), Q30.3 (S), Q32.3 (S), Q4.1 (S), Q4.2 (S), Q4.3 (S), Q7.3 (S), Q8.1 (S), Q8.2 (S), Q8.3 (S), R1.1, R10.1, R15.1, R17.1, R21.1, R23.1, R26.1, R3.1, R30.1, R32.1, R36.1, R38.1, R42.1, R44.1, R48.1, R8.1
- new net: F12.2, Q25.1 (S), Q25.2 (S), Q25.3 (S), R36.1
- new net: F11.2, Q22.3 (S), R32.1
- new net: F3.2, Q7.3 (S), R8.1
- new net: F4.2, Q8.1 (S), Q8.2 (S), Q8.3 (S), R10.1
- new net: F8.2, Q16.1 (S), Q16.2 (S), Q16.3 (S), R23.1
- new net: F15.2, Q30.3 (S), R44.1
- new net: F16.2, Q32.3 (S), R48.1
- new net: F1.2, Q3.3 (S), R1.1
- new net: F6.2, Q12.1 (S), Q12.2 (S), Q12.3 (S), R17.1
- new net: F5.2, Q11.3 (S), R15.1
- new net: F10.2, Q21.1 (S), Q21.2 (S), Q21.3 (S), R30.1
- new net: F7.2, Q14.3 (S), R21.1
- new net: F9.2, Q18.3 (S), R26.1
- new net: F2.2, Q4.1 (S), Q4.2 (S), Q4.3 (S), R3.1
- new net: F13.2, Q26.3 (S), R38.1
- new net: F14.2, Q29.1 (S), Q29.2 (S), Q29.3 (S), R42.1

Commit message: Made Most of the Review Changes
Parts:
- added V3, V4, V5, V6: Via, symbol MRDT_Drill_Holes:Via
Connections:
- net LSpare renamed LCSpare
- net TLSpare renamed TLCSpare
Other:
- note added: "Capacitor Bank"
- note added: "Mounting Vias"
- note removed: "Label?"
Changed lines of the file:
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@@
     (stroke (width 0) (type default) (color 0 0 0 0))
   )
+  (polyline (pts (xy 59.69 107.95) (xy 59.69 146.05))
+    (stroke (width 0) (type default) (color 0 0 0 0))
+  )
   (wire (pts (xy 113.03 251.46) (xy 113.03 252.73))
     (stroke (width 0) (type default) (color 0 0 0 0))
@@
     (stroke (width 0) (type default) (color 0 0 0 0))
   )
+  (text "Mounting Vias" (at 13.97 116.84 0)
+    (effects (font (size 4 4) (thickness 0.8) bold) (justify left bottom))
+  )
   (text "Teensy" (at 151.13 24.13 0)
     (effects (font (size 4 4) (thickness 0.8) bold) (justify left bottom))
@@
     (effects (font (size 4 4) (thickness 0.8) bold) (justify left bottom))
   )
-  (text ";)" (at 44.45 129.54 0)
+  (text ";)" (at 72.39 129.54 0)
     (effects (font (size 5 5) (thickness 1) bold) (justify left bottom))
   )
@@
     (effects (font (size 4 4) (thickness 0.8) bold) (justify left bottom))
   )
-  (text "Label?" (at 13.97 20.32 0)
+  (text "Capacitor Bank" (at 13.97 20.32 0)
     (effects (font (size 4 4) bold) (justify left bottom))
   )
@@
     )
   )
-  (global_label "TLSpare" (shape input) (at 224.79 262.89 90) (fields_autoplaced)
+  (global_label "TLCSpare" (shape input) (at 224.79 262.89 90) (fields_autoplaced)
     (effects (font (size 1.27 1.27)) (justify left))
-    (property "Intersheet References" "${INTERSHEET_REFS}" (id 0) (at 224.8694 253.0988 90)
+    (property "Intersheet References" "${INTERSHEET_REFS}" (id 0) (at 224.7106 251.8288 90)
       (effects (font (size 1.27 1.27)) (justify left) hide)
     )
@@
     )
   )
-  (global_label "TLSpare" (shape output) (at 179.07 106.68 180) (fields_autoplaced)
+  (global_label "TLCSpare" (shape output) (at 179.07 106.68 180) (fields_autoplaced)
     (effects (font (size 1.27 1.27)) (justify right))
-    (property "Intersheet References" "${INTERSHEET_REFS}" (id 0) (at 169.2788 106.6006 0)
+    (property "Intersheet References" "${INTERSHEET_REFS}" (id 0) (at 168.0088 106.6006 0)
       (effects (font (size 1.27 1.27)) (justify right) hide)
     )
@@
     )
   )
-  (global_label "LSpare" (shape input) (at 360.68 93.98 0) (fields_autoplaced)
+  (global_label "LCSpare" (shape input) (at 360.68 93.98 0) (fields_autoplaced)
     (effects (font (size 1.27 1.27)) (justify left))
-    (property "Intersheet References" "${INTERSHEET_REFS}" (id 0) (at 369.5036 93.9006 0)
+    (property "Intersheet References" "${INTERSHEET_REFS}" (id 0) (at 370.7736 93.9006 0)
       (effects (font (size 1.27 1.27)) (justify left) hide)
     )
@@
     )
   )
-  (global_label "LSpare" (shape output) (at 246.38 252.73 270) (fields_autoplaced)
+  (global_label "LCSpare" (shape output) (at 246.38 252.73 270) (fields_autoplaced)
     (effects (font (size 1.27 1.27)) (justify right))
-    (property "Intersheet References" "${INTERSHEET_REFS}" (id 0) (at 246.3006 261.5536 90)
+    (property "Intersheet References" "${INTERSHEET_REFS}" (id 0) (at 246.3006 262.8236 90)
       (effects (font (size 1.27 1.27)) (justify right) hide)
     )
@@
     (pin "3")
   )
+  (symbol (lib_id "MRDT_Drill_Holes:Via") (at 19.05 127 0) (unit 1)
+    (in_bom yes) (on_board yes) (fields_autoplaced)
+    (property "Reference" "V4" (id 0) (at 24.765 126.0238 0)
+      (effects (font (size 1.524 1.524)) (justify left))
+    )
+    (property "Value" "Via" (id 1) (at 24.765 129.0172 0)
+      (effects (font (size 1.524 1.524)) (justify left))
+    )
+    (property "Footprint" "" (id 2) (at 19.05 127 0)
+      (effects (font (size 1.524 1.524)) hide)
+    )
+    (property "Datasheet" "" (id 3) (at 19.05 127 0)
+      (effects (font (size 1.524 1.524)) hide)
+    )
+    (pin "1")
+  )
   (symbol (lib_id "Device:LED") (at 24.13 85.09 0) (unit 1)
     (in_bom yes) (on_board yes)
@@
     (pin "2")
   )
+  (symbol (lib_id "MRDT_Drill_Holes:Via") (at 19.05 139.7 0) (unit 1)
+    (in_bom yes) (on_board yes) (fields_autoplaced)
+    (property "Reference" "V6" (id 0) (at 24.765 138.7238 0)
+      (effects (font (size 1.524 1.524)) (justify left))
+    )
+    (property "Value" "Via" (id 1) (at 24.765 141.7172 0)
+      (effects (font (size 1.524 1.524)) (justify left))
+    )
+    (property "Footprint" "" (id 2) (at 19.05 139.7 0)
+      (effects (font (size 1.524 1.524)) hide)
+    )
+    (property "Datasheet" "" (id 3) (at 19.05 139.7 0)
+      (effects (font (size 1.524 1.524)) hide)
+    )
+    (pin "1")
+  )
   (symbol (lib_id "Device:Fuse") (at 219.71 167.64 0) (unit 1)
     (in_bom yes) (on_board yes)
@@
     (pin "1")
   )
+  (symbol (lib_id "MRDT_Drill_Holes:Via") (at 19.05 120.65 0) (unit 1)
+    (in_bom yes) (on_board yes) (fields_autoplaced)
+    (property "Reference" "V3" (id 0) (at 24.765 119.6738 0)
+      (effects (font (size 1.524 1.524)) (justify left))
+    )
+    (property "Value" "Via" (id 1) (at 24.765 122.6672 0)
+      (effects (font (size 1.524 1.524)) (justify left))
+    )
+    (property "Footprint" "" (id 2) (at 19.05 120.65 0)
+      (effects (font (size 1.524 1.524)) hide)
+    )
+    (property "Datasheet" "" (id 3) (at 19.05 120.65 0)
+      (effects (font (size 1.524 1.524)) hide)
+    )
+    (pin "1")
+  )
   (symbol (lib_id "power:GND") (at 87.63 86.36 0) (unit 1)
     (in_bom yes) (on_board yes) (fields_autoplaced)
@@
     (pin "2")
   )
+  (symbol (lib_id "MRDT_Drill_Holes:Via") (at 19.05 133.35 0) (unit 1)
+    (in_bom yes) (on_board yes) (fields_autoplaced)
+    (property "Reference" "V5" (id 0) (at 24.765 132.3738 0)
+      (effects (font (size 1.524 1.524)) (justify left))
+    )
+    (property "Value" "Via" (id 1) (at 24.765 135.3672 0)
+      (effects (font (size 1.524 1.524)) (justify left))
+    )
+    (property "Footprint" "" (id 2) (at 19.05 133.35 0)
+      (effects (font (size 1.524 1.524)) hide)
+    )
+    (property "Datasheet" "" (id 3) (at 19.05 133.35 0)
+      (effects (font (size 1.524 1.524)) hide)
+    )
+    (pin "1")
+  )
   (symbol (lib_id "Device:R") (at 82.55 255.27 0) (unit 1)
     (in_bom yes) (on_board yes)
@@
       (reference "V2") (unit 1) (value "GND1") (footprint "")
     )
+    (path "/98225fd9-e0e2-4ffa-94bd-d5a731be807e"
+      (reference "V3") (unit 1) (value "Via") (footprint "")
+    )
+    (path "/218c2f2a-02f7-4ac5-8960-c2185b7d605e"
+      (reference "V4") (unit 1) (value "Via") (footprint "")
+    )
+    (path "/9bef0ffa-3c3a-4e71-9c08-490f16189f09"
+      (reference "V5") (unit 1) (value "Via") (footprint "")
+    )
+    (path "/70b4c972-b782-4ed1-b71a-f083beb5f3b8"
+      (reference "V6") (unit 1) (value "Via") (footprint "")
+    )
   )

Commit message: Finished Review Changes, Created PDF, Cleaned Out Old Files
Connections:
- net TAux renamed CTLAux
- net TBB renamed CTLBB
- net TCam renamed CTLCam
- net TDrive renamed CTLDrive
- net TGimbal renamed CTLGimbal
- net TLCSpare renamed CTLLCSpare
- net TM1 renamed CTLM1
- net TM2 renamed CTLM2
- net TM3 renamed CTLM3
- net TM4 renamed CTLM4
- net TM5 renamed CTLM5
- net TM6 renamed CTLM6
- net TMM renamed CTLMM
- net TMS renamed CTLMS
- net TNav renamed CTLNav
- net TSpare renamed CTLSpare

Commit message: Assigned Footprints
Parts:
- C1, C2, C3, C5: footprint (none) -> Capacitor_THT:CP_Radial_D12.5mm_P5.00mm
- C4, C6, C7: footprint (none) -> Capacitor_SMD:C_0603_1608Metric_Pad1.08x0.95mm_HandSolder
- Conn1, Conn10, Conn11, Conn12, Conn13, Conn14, Conn15, Conn16, Conn17, Conn18, Conn2, Conn3, Conn4, Conn5, Conn6, Conn7, Conn8, Conn9: footprint (none) -> MRDT_Connectors:Square_Anderson_2_V_Side_By_Side_PV
- D1, D10, D11, D12, D13, D14, D15, D16, D17, D18, D19, D2, D20, D3, D6, D7, D8, D9: footprint (none) -> LED_SMD:LED_0603_1608Metric_Pad1.05x0.95mm_HandSolder
- D4, D5: footprint (none) -> Diode_THT:D_DO-201_P5.08mm_Vertical_KathodeUp
- F1, F10, F11, F12, F13, F14, F15, F16, F2, F3, F4, F5, F6, F7, F8, F9: footprint (none) -> MRDT_Passives:ATC_Fuse_Block
- J1: footprint (none) -> MRDT_Connectors:RJ45_Teensy
- J2: footprint (none) -> Connector_PinSocket_2.00mm:PinSocket_2x03_P2.00mm_Vertical
- Q12, Q16, Q21, Q25, Q29, Q4, Q8: footprint Package_SO:MSOP-8_3x3mm_P0.65mm -> Package_SO:SOP-8_3.9x4.9mm_P1.27mm
- R1, R10, R11, R12, R13, R14, R15, R16, R17, R18, R19, R2, R20, R21, R22, R23, R24, R25, R26, R27, R28, R29, R3, R30, R31, R32, R33, R34, R35, R36, R37, R38, R39, R4, R40, R41, R42, R43, R44, R45, R46, R47, R48, R49, R5, R50, R6, R7, R8, R9: footprint (none) -> Resistor_SMD:R_0603_1608Metric_Pad0.98x0.95mm_HandSolder
- U1: footprint (none) -> MRDT_Devices:OKI_Horizontal
- U2: footprint MODULE_DEV-16771 -> MRDT_Shields:MODULE_DEV-16771
- V1, V2: footprint (none) -> MRDT_Drill_Holes:BATT_PWR_VIA
- V3, V4, V5, V6: footprint (none) -> MRDT_Drill_Holes:4_40_Hole_Corner
