File: Hardware/PowerBoard_2024/PowerBoard_2024.kicad_pcb (KiCad board)
At the start: 2 copper layers, 218 parts, among them J1 RJ45_LED_Shielded, Q1 BSS138, Q10 BSS138, Q11 BSS138, Q12 IRF7606PBF, Q13 IRF7606PBF, Q14 SPD30P06PGBTMA1, Q15 BSS138, Q16 SPD30P06PGBTMA1, Q17 BSS138, Q18 BSS138, Q19 BSS138, Q2 IRF7606PBF, Q20 IRF7606PBF, Q21 IRF7606PBF, Q22 SPD30P06PGBTMA1, Q23 BSS138, Q24 SPD30P06PGBTMA1, Q25 BSS138, Q26 SPD30P06PGBTMA1, Q27 BSS138, Q28 SPD30P06PGBTMA1, Q29 BSS138, Q3 BSS138, Q30 SPD30P06PGBTMA1, Q4 IRF7606PBF, Q5 BSS138, Q6 SPD30P06PGBTMA1, Q7 BSS138, Q8 SPD30P06PGBTMA1, Q9 BSS138, U1 3V3, U10 ACS725xLCTR-20AB, U11 ACS725xLCTR-20AB, U12 ACS725xLCTR-20AB, U13 ACS725xLCTR-20AB, U14 ACS725xLCTR-20AB, U15 Teensy4.1_DEV-16771, U16 ACS725xLCTR-20AB, U17 ACS725xLCTR-20AB, U18 ACS725xLCTR-20AB, U19 ACS725xLCTR-20AB, U2 ACS725xLCTR-20AB, U20 PKE3316ZPI, U21 ACS725xLCTR-20AB, U22 PKE3316ZPI, U23 ACS725xLCTR-20AB, U3 ACS725xLCTR-20AB, U4 ACS725xLCTR-20AB, U5 ACS725xLCTR-20AB, U6 ACS725xLCTR-20AB, U7 ACS725xLCTR-20AB, U8 ACS725xLCTR-20AB, U9 ACS725xLCTR-20AB

Commit message: Layout Started
Fixed footprints
Started Layout
Lots of work left to be done
Parts:
- C8: footprint Capacitor_THT:CP_Radial_D16.0mm_P7.50mm -> Capacitor_THT:CP_Radial_D6.3mm_P2.50mm
- Conn1, Conn10, Conn11, Conn12, Conn13, Conn14, Conn15, Conn16, Conn17, Conn18, Conn19, Conn2, Conn3, Conn4, Conn5, Conn6, Conn7, Conn8, Conn9: footprint MRDT_Connectors:Anderson_2_Horizontal_Side_by_Side_PV -> MRDT_Connectors:Square_Anderson_2_H_Stacked
- moved Q14 318.8 mm to (452.2, 108.3)
- moved Q16 318.8 mm to (452.2, 116.3)
- moved Q22 318.8 mm to (452.2, 124.4)
- moved Q24 318.8 mm to (452.2, 132.4)
- moved Q26 318.8 mm to (452.2, 140.5)
- moved Q28 318.8 mm to (452.2, 148.5)
- moved Q30 318.8 mm to (452.2, 156.6)
- moved Q6 318.8 mm to (452.2, 92.2)
- moved Q8 318.8 mm to (452.2, 100.2)
- moved C35 246.4 mm to (274.3, 82.8)
- moved C36 246.4 mm to (274.3, 85.3)
- moved C37 246.4 mm to (274.3, 87.9)
- moved C38 246.4 mm to (274.3, 90.4)
- moved C39 246.4 mm to (274.3, 92.9)
- moved C40 246.4 mm to (274.3, 95.4)
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Other:
- board outline added: 160.5 x 160.5 mm

Commit message: Fill gnd plane
discussed stuff & goofed
Parts:
- C11, C53, U23: moved to B.Cu
- moved U23 320.7 mm to (77.2, 75.2), turned to 90 degrees
- moved C11 257.8 mm to (74.7, 81.8), turned to -90 degrees
- moved C10 253.0 mm to (79.3, 82.3)
- moved U1 229.6 mm to (176.9, 179.6), turned to 90 degrees
- moved C53 203.6 mm to (76.7, 69.2), turned to -90 degrees
- moved C52 132.5 mm to (146.1, 97.0)
- moved C22 88.0 mm to (177.6, 107.2)
- moved Q4 64.3 mm to (313.8, 149.1)
- moved D8 64.3 mm to (334.4, 156.5)
- moved Q3 64.3 mm to (320.0, 148.9)
- moved C15 30.8 mm to (268.4, 123.6)
- moved R11 30.8 mm to (285.8, 123.6)
- moved R9 30.8 mm to (285.8, 118.6)
- moved C16 30.8 mm to (268.4, 126.1)
- moved R10 30.8 mm to (285.8, 121.1)
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Routing:
- added copper zone on B.Cu, net GND
- added copper zone on F.Cu, net GND

Commit message: Layout
Progress
4 Layer Board
Parts:
- Conn1, Conn10, Conn11, Conn12, Conn13, Conn14, Conn15, Conn16, Conn17, Conn18, Conn19, Conn2, Conn3, Conn4, Conn5, Conn6, Conn7, Conn8, Conn9: moved to B.Cu
- moved Q8 327.2 mm to (129.3, 153.3), turned to 90 degrees
- moved Q16 316.7 mm to (137.7, 153.3), turned to 90 degrees
- moved Q24 306.1 mm to (146.8, 153.3), turned to 90 degrees
- moved Q28 296.3 mm to (156.0, 153.2), turned to 90 degrees
- moved Q30 287.1 mm to (165.1, 153.3), turned to 90 degrees
- moved C10 280.1 mm to (359.3, 75.8)
- moved C11 280.1 mm to (354.7, 75.3)
- moved C53 280.1 mm to (356.7, 62.8)
- moved Q26 278.2 mm to (174.2, 153.2), turned to 90 degrees
- moved U23 270.6 mm to (347.7, 67.5)
- moved Q22 270.6 mm to (183.1, 153.2), turned to 90 degrees
- moved Q14 263.7 mm to (192.3, 153.2), turned to 90 degrees
- moved U5 259.9 mm to (106.2, 128.0)
- moved Q6 258.1 mm to (201.4, 153.3), turned to 90 degrees
- moved U9 254.8 mm to (119.6, 127.8)
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Connections:
- C17 pad 1: GND -> Net-(U4-FILTER)
- C17 pad 2: Net-(U4-FILTER) -> GND
- C18 pad 1: +3V3 -> GND
- C18 pad 2: GND -> +3V3
- C19 pad 1: GND -> Net-(U5-FILTER)
- C19 pad 2: Net-(U5-FILTER) -> GND
- C20 pad 1: +3V3 -> GND
- C20 pad 2: GND -> +3V3
- C25 pad 1: GND -> Net-(U8-FILTER)
- C25 pad 2: Net-(U8-FILTER) -> GND
- C26 pad 1: +3V3 -> GND
- C26 pad 2: GND -> +3V3
- C27 pad 1: GND -> Net-(U9-FILTER)
- C27 pad 2: Net-(U9-FILTER) -> GND
- C28 pad 1: +3V3 -> GND
- C28 pad 2: GND -> +3V3
- C33 pad 1: GND -> Net-(U12-FILTER)
- C33 pad 2: Net-(U12-FILTER) -> GND
- C34 pad 1: +3V3 -> GND
- C34 pad 2: GND -> +3V3
- C35 pad 1: GND -> Net-(U13-FILTER)
- C35 pad 2: Net-(U13-FILTER) -> GND
- C36 pad 1: +3V3 -> GND
- C36 pad 2: GND -> +3V3
- C37 pad 1: GND -> Net-(U14-FILTER)
- C37 pad 2: Net-(U14-FILTER) -> GND
- C38 pad 1: +3V3 -> GND
- C38 pad 2: GND -> +3V3
- C40 pad 1: GND -> Net-(U16-FILTER)
- C40 pad 2: Net-(U16-FILTER) -> GND
- C41 pad 1: +3V3 -> GND
- C41 pad 2: GND -> +3V3
- C42 pad 1: GND -> Net-(U17-FILTER)
- C42 pad 2: Net-(U17-FILTER) -> GND
- C43 pad 1: +3V3 -> GND
- C43 pad 2: GND -> +3V3
Routing:
- net +3V3: track 0.00 -> 27.9 mm
- net Net-(Q8-D): track 0.00 -> 9.46 mm
- net Net-(Q16-D): track 0.00 -> 9.30 mm
- net Net-(Q26-D): track 0.00 -> 9.18 mm
- net Net-(Q14-D): track 0.00 -> 9.01 mm
- net Net-(Q6-D): track 0.00 -> 8.89 mm
- net Net-(Q22-D): track 0.00 -> 8.89 mm
- net Net-(Q24-D): track 0.00 -> 8.84 mm
- net Net-(Q30-D): track 0.00 -> 8.68 mm
- net Net-(Q28-D): track 0.00 -> 8.47 mm
- net CTL_M6: track 0.00 -> 3.36 mm
- net CTL_M1: track 0.00 -> 3.25 mm
- net Net-(U8-FILTER): track 0.00 -> 3.24 mm
- net Net-(U9-FILTER): track 0.00 -> 3.23 mm
- net CTL_M3: track 0.00 -> 3.22 mm
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- added copper zone on In2.Cu, net GND
- added copper zone on F.Cu, net PV
- added copper zone on In1.Cu, net PV
- removed copper zone on B.Cu, net GND
- removed copper zone on F.Cu, net GND
Other:
- board size 160.5 x 160.5 mm -> 211.3 x 160.5 mm
- copper layers 2 -> 4

Commit message: Layout Stuff Rev1
Parts:
- C11, C53, U23: moved to F.Cu
- C49: footprint Capacitor_SMD:C_0603_1608Metric_Pad1.08x0.95mm_HandSolder -> Capacitor_SMD:C_1206_3216Metric_Pad1.33x1.80mm_HandSolder
- moved U21 307.4 mm to (178.7, 115.9), turned to 90 degrees
- moved Conn12 273.5 mm to (358.6, 186.5), turned to 180 degrees
- moved Conn14 268.3 mm to (358.4, 169.2), turned to 180 degrees
- moved Conn15 268.2 mm to (358.4, 133.2), turned to 180 degrees
- moved Conn13 268.0 mm to (358.4, 151.4), turned to 180 degrees
- moved Conn7 265.8 mm to (329.1, 241.8), turned to 90 degrees
- moved U19 263.0 mm to (222.6, 115.8), turned to 90 degrees
- moved D4 251.6 mm to (172.1, 112.5), turned to -90 degrees
- moved U18 244.1 mm to (240.9, 115.9), turned to 90 degrees
- moved Conn6 243.2 mm to (310.1, 241.8), turned to 90 degrees
- moved C48 239.3 mm to (177.7, 132.2)
- moved C35 232.0 mm to (341.0, 241.5)
- moved C36 232.0 mm to (341.0, 237.1)
- moved U13 232.0 mm to (335.7, 239.9)
- moved Conn5 222.2 mm to (291.0, 241.8), turned to 90 degrees
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Connections:
- C19 pad 1: Net-(U5-FILTER) -> GND
- C19 pad 2: GND -> Net-(U5-FILTER)
- C20 pad 1: GND -> +3V3
- C20 pad 2: +3V3 -> GND
- C27 pad 1: Net-(U9-FILTER) -> GND
- C27 pad 2: GND -> Net-(U9-FILTER)
- C28 pad 1: GND -> +3V3
- C28 pad 2: +3V3 -> GND
- U15 pad 10: unconnected-(U15-CS1-Pad10) -> CTL_DiffGPS
- U15 pad 11: CTL_DiffGPS -> CTL_Core
- U15 pad 14: CS_HC_Spare -> CS_M5
- U15 pad 15: CS_Cam -> CS_M6
- U15 pad 16: CS_Net Switch_3 -> CS_MS
- U15 pad 17: CS_Aux -> CS_Cam
- U15 pad 18: CS_M1 -> CS_HC_Spare
- U15 pad 19: CS_M2 -> CS_Aux
- U15 pad 20: CS_M3 -> CS_LC_Spare
- U15 pad 21: CS_M4 -> CS_Core
- U15 pad 22: CS_M5 -> CS_DiffGPS
- U15 pad 23: CS_M6 -> CS_RouterPi
- U15 pad 24: CS_Core -> CS_Net Switch_1
- U15 pad 25: CS_RouterPi -> CS_Net Switch_2
- U15 pad 26: CS_Net Switch_1 -> CS_Net Switch_3
- U15 pad 27: CS_DiffGPS -> CS_POE
- U15 pad 29: CTL_HC_Spare -> CTL_M6
- U15 pad 30: CTL_Cam -> CTL_M5
- U15 pad 34: CTL_Aux -> CTL_M4
- U15 pad 35: CTL_M1 -> CTL_M3
- U15 pad 37: CTL_M3 -> CTL_M1
- U15 pad 38: CS_Net Switch_2 -> CS_M1
- U15 pad 39: CS_POE -> CS_M2
- U15 pad 40: CS_LC_Spare -> CS_M3
- U15 pad 41: CS_MS -> CS_M4
- U15 pad 5: CTL_M6 -> CTL_Aux
- U15 pad 6: CTL_M5 -> CTL_HC_Spare
- U15 pad 7: CTL_M4 -> CTL_Cam
- U15 pad 8: CTL_Core -> unconnected-(U15-TX2-Pad8)
Routing:
- net +3V3: track 27.9 -> 726.8 mm, vias 0 -> 20
- net CS_POE: track 0.00 -> 225.5 mm, vias 0 -> 1
- net CS_Net Switch_3: track 0.00 -> 215.3 mm, vias 0 -> 1
- net CS_Net Switch_2: track 0.00 -> 198.5 mm, vias 0 -> 1
- net CS_Cam: track 0.00 -> 190.1 mm, vias 0 -> 1
- net CS_Net Switch_1: track 0.00 -> 181.4 mm, vias 0 -> 1
- net CTL_Cam: track 0.00 -> 162.8 mm, vias 0 -> 1
- net CS_HC_Spare: track 0.00 -> 147.2 mm, vias 0 -> 1
- net CS_Aux: track 0.00 -> 125.4 mm, vias 0 -> 1
- net Net-(Q13-D-Pad5): track 0.00 -> 122.2 mm, vias 0 -> 2
- net CS_M1: track 0.00 -> 115.5 mm, vias 0 -> 1
- net CTL_HC_Spare: track 3.14 -> 116.6 mm, vias 0 -> 1
- net CS_LC_Spare: track 0.00 -> 106.4 mm, vias 0 -> 1
- net CS_M2: track 0.00 -> 98.5 mm, vias 0 -> 1
- net Net-(Q20-D-Pad5): track 0.00 -> 95.4 mm, vias 0 -> 2
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- added copper zone on F.Cu, net +12V
- added copper zone on F.Cu, net +24V
- added copper zone on F.Cu, net 12V_Spare
- added copper zone on F.Cu, net Aux
- added copper zone on F.Cu, net Cam
- added copper zone on F.Cu, net Core
- added copper zone on F.Cu, net DiffGPS
- added copper zone on B.Cu, net GND
- added copper zone on F.Cu, net GND
- added copper zone on In1.Cu, net GND
- added copper zone on F.Cu, net HC_Spare
- added copper zone on F.Cu, net LC_Spare
- added copper zone on F.Cu, net M1
- added copper zone on F.Cu, net M2
- added copper zone on F.Cu, net M3
- added copper zone on F.Cu, net M4
- added copper zone on F.Cu, net M5
- added copper zone on F.Cu, net M6
- added copper zone on F.Cu, net MS
- added copper zone on F.Cu, net Net Switch_1
- added copper zone on F.Cu, net Net Switch_2
- added copper zone on F.Cu, net Net Switch_3
- added copper zone on F.Cu, net Net-(Q12-D-Pad5)
- added copper zone on F.Cu, net Net-(Q13-D-Pad5)
- added copper zone on F.Cu, net Net-(Q2-D-Pad5)
- added copper zone on F.Cu, net Net-(Q20-D-Pad5)
- added copper zone on F.Cu, net Net-(Q21-D-Pad5)
- added copper zone on F.Cu, net Net-(Q4-D-Pad5)
- added copper zone on F.Cu, net POE
- added copper zone on F.Cu, net RouterPi
- added copper zone on F.Cu, net Switch_3 24V
- removed copper zone on In1.Cu, net PV

Commit message: Layout Changes
Changed the layout
Parts:
- moved C9 101.5 mm to (359.7, 124.5), turned to 0 degrees
- moved J1 100.4 mm to (377.8, 139.6)
- moved C39 100.4 mm to (351.5, 133.4)
- moved D3 100.2 mm to (363.7, 126.0), turned to -90 degrees
- moved R1 97.9 mm to (359.7, 127.0), turned to 180 degrees
- moved C12 88.0 mm to (360.2, 106.7), turned to 0 degrees
- moved D6 87.1 mm to (364.2, 108.2)
- moved R4 85.0 mm to (360.2, 109.7), turned to 0 degrees
- moved U1 79.5 mm to (359.3, 119.9), turned to 90 degrees
- moved R31 75.0 mm to (365.6, 163.1), turned to 0 degrees
- moved D12 74.2 mm to (365.6, 166.1), turned to 0 degrees
- moved R50 71.7 mm to (364.7, 230.6)
- moved D16 69.3 mm to (365.3, 219.5), turned to 0 degrees
- moved D15 67.3 mm to (365.3, 184.4), turned to 0 degrees
- moved R46 66.1 mm to (365.4, 181.4), turned to 0 degrees
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Connections:
- U15 pad 10: CTL_DiffGPS -> CTL_Core
- U15 pad 11: CTL_Core -> CTL_DiffGPS
- U15 pad 12: CTL_LC_Spare -> CTL_RouterPi
- U15 pad 34: CTL_M4 -> CTL_M1
- U15 pad 35: CTL_M3 -> CTL_M2
- U15 pad 36: CTL_M2 -> CTL_M3
- U15 pad 37: CTL_M1 -> CTL_M4
- U15 pad 9: CTL_RouterPi -> CTL_LC_Spare
Routing:
- net +3V3: track 726.8 -> 0.00 mm, vias 20 -> 0
- net Net-(Q13-D-Pad5): track 122.2 -> 0.00 mm, vias 2 -> 0
- net CTL_MS: track 35.7 -> 148.0 mm
- net Net-(Q20-D-Pad5): track 95.4 -> 0.00 mm, vias 2 -> 0
- net Net-(Q8-G): track 85.4 -> 0.00 mm
- net CS_Cam: track 190.1 -> 105.8 mm
- net CS_MS: track 23.1 -> 107.3 mm
- net CTL_M6: track 44.8 -> 128.8 mm
- net Net-(Q8-D): track 82.9 -> 0.00 mm
- net CTL_Cam: track 162.8 -> 89.9 mm
- net Net-(Q16-G): track 71.8 -> 0.00 mm
- net CS_Net Switch_2: track 198.5 -> 128.5 mm
- net Net-(Q12-D-Pad5): track 69.1 -> 0.00 mm, vias 2 -> 0
- net Net-(Q16-D): track 69.0 -> 0.00 mm
- net CS_Net Switch_3: track 215.3 -> 146.7 mm
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- added copper zone on F.Cu, net Net-(Q14-D)
- added copper zone on F.Cu, net Net-(Q16-D)
- added copper zone on F.Cu, net Net-(Q22-D)
- added copper zone on F.Cu, net Net-(Q24-D)
- added copper zone on F.Cu, net Net-(Q26-D)
- added copper zone on F.Cu, net Net-(Q28-D)
- added copper zone on F.Cu, net Net-(Q30-D)
- added copper zone on F.Cu, net Net-(Q6-D)
- added copper zone on F.Cu, net Net-(Q8-D)

Commit message: Layout Review Ready
Made the traces pretty
Parts:
- moved C6 129.3 mm to (200.2, 225.0), turned to -90 degrees
- moved C4 124.6 mm to (203.2, 225.0), turned to -90 degrees
- moved C2 115.5 mm to (208.3, 224.0), turned to -90 degrees
- moved D5 62.7 mm to (218.4, 122.4), turned to -90 degrees
- moved R3 56.7 mm to (219.5, 126.5), turned to 180 degrees
- moved C8 49.4 mm to (220.1, 132.1), turned to 180 degrees
- moved D8 19.2 mm to (299.7, 111.8), turned to 90 degrees
- moved D7 18.7 mm to (275.3, 111.8), turned to 90 degrees
- moved D4 16.9 mm to (189.0, 111.8)
- moved R12 16.4 mm to (296.7, 111.8)
- moved R8 15.9 mm to (272.3, 111.8)
- moved R2 14.8 mm to (185.9, 111.8), turned to -90 degrees
- moved R20 3.07 mm to (321.6, 111.8), turned to 90 degrees
- moved D10 3.07 mm to (324.6, 111.8), turned to 90 degrees
- moved D6 2.03 mm to (364.2, 110.2)
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Connections:
- U15 pad 20: CS_LC_Spare -> CS_RouterPi
- U15 pad 21: CS_Core -> CS_DiffGPS
- U15 pad 22: CS_DiffGPS -> CS_Core
- U15 pad 23: CS_RouterPi -> CS_LC_Spare
Routing:
- net +3V3: track 0.00 -> 784.0 mm, vias 0 -> 20
- net CTL_MS: track 148.0 -> 243.6 mm
- net CTL_M6: track 128.8 -> 222.5 mm
- net LED: track 0.00 -> 93.0 mm
- net CTL_M5: track 110.8 -> 202.2 mm
- net CTL_M4: track 70.9 -> 160.8 mm
- net CTL_LC_Spare: track 49.1 -> 131.5 mm
- net CS_M1: track 108.2 -> 189.8 mm
- net TX+: track 0.00 -> 81.5 mm
- net TX-: track 0.00 -> 81.4 mm
- net CS_M2: track 89.3 -> 168.1 mm
- net CTL_M3: track 60.6 -> 139.3 mm
- net CS_M3: track 68.2 -> 146.4 mm
- net CTL_Core: track 45.2 -> 118.0 mm
- net CS_M4: track 58.9 -> 125.3 mm
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